File: hardware/kicad/bwlc1a.kicad_pcb (KiCad board)
At the start: 4 copper layers, 80 x 50 mm, 107 parts, among them J1 JST-2PH, J2 USB_C_Receptacle_USB2.0, J4 Nano SIM, J5 RSP-122811-02, Q1 DMG3415UQ-7, Q2 NPN, Q3 NPN, Q4 NPN, Q5 NPN, Q6 NPN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

Commit message: Update on PCB Layout
Parts:
- added C38: 100n, Capacitor_SMD:C_0402_1005Metric, F.Cu at (142.8, 102.9)
- C19, C31, C32: footprint Capacitor_SMD:C_0402_1005Metric -> Capacitor_SMD:C_0603_1608Metric
- C21: footprint Capacitor_SMD:C_0402_1005Metric -> Capacitor_SMD:C_0805_2012Metric
- moved TP1 142.7 mm to (197.8, 111.8), turned to 180 degrees
- moved C25 140.0 mm to (168.7, 126.5), turned to 180 degrees
- moved C24 139.9 mm to (168.7, 124.4)
- moved C23 139.7 mm to (168.7, 122.2)
- moved C22 139.6 mm to (168.7, 120.1)
- moved C26 139.4 mm to (168.7, 127.6), turned to 180 degrees
- moved TP2 139.2 mm to (197.8, 108.3), turned to 180 degrees
- moved R16 136.3 mm to (168.7, 125.4)
- moved TP3 136.1 mm to (197.8, 104.7), turned to 180 degrees
- moved R17 133.4 mm to (168.7, 123.3)
- moved TP4 133.2 mm to (197.8, 101.2), turned to 180 degrees
- moved R20 127.8 mm to (168.7, 121.2)
- moved Q3 108.3 mm to (141.7, 96.0), turned to 180 degrees
- moved D4 107.9 mm to (168.4, 117.8)
- moved Q4 107.6 mm to (141.8, 99.6)
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Routing:
- net VDD_BAT: track 0.00 -> 53.8 mm
- net GND: track 0.00 -> 43.2 mm, vias 0 -> 16
- net IMU_VDD: track 0.00 -> 10.6 mm
- net A7670_UART_RX: track 0.00 -> 8.17 mm
- net A7670_TX: track 0.00 -> 7.50 mm
- net USB_D-: track 0.00 -> 6.03 mm
- net /TPS_FB: track 0.00 -> 5.30 mm
- net Net-(U8-ADJ): track 0.00 -> 5.23 mm
- net ESP_32K_P: track 0.00 -> 4.91 mm
- net ESP_32K_N: track 0.00 -> 4.85 mm
- net RESET: track 0.00 -> 4.82 mm
- net A7670_UART_TX: track 0.00 -> 4.66 mm
- net Net-(Q6-B): track 0.00 -> 4.29 mm
- net Net-(Q5-B): track 0.00 -> 4.12 mm
- net Net-(JP2-A): track 0.00 -> 3.68 mm
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- added copper zone on F.Cu, net GND
- added copper zone on In1.Cu, net GND
- added copper zone on F.Cu, net Net-(C27-Pad1)
- added copper zone on F.Cu, net Net-(JP2-A)

Commit message: Update on routing
Parts:
- removed C22, C23, C24: 22p (N.C.), Capacitor_SMD:C_0402_1005Metric
- removed C26: 33p, Capacitor_SMD:C_0402_1005Metric
- removed R15: N.C, Resistor_SMD:R_0402_1005Metric
- C20: footprint Capacitor_SMD:CP_Elec_8x10.5 -> Capacitor_SMD:CP_Elec_6.3x7.7
- JP1: moved to F.Cu
- R13: value 10k -> 1M
- moved TP1 50.2 mm to (147.7, 110.9), turned to 90 degrees
- moved C8 48.2 mm to (174.4, 80.9), turned to -90 degrees
- moved U4 47.9 mm to (176.6, 80.9), turned to 0 degrees
- moved TP2 46.7 mm to (151.2, 110.9), turned to 90 degrees
- moved D1 44.8 mm to (182.3, 85.5), turned to 0 degrees
- moved R4 44.1 mm to (182.3, 83.8)
- moved TP3 43.5 mm to (154.8, 110.9), turned to 90 degrees
- moved R5 41.5 mm to (181.3, 83.8), turned to -90 degrees
- moved TP4 40.7 mm to (158.3, 110.9), turned to 90 degrees
- moved C1 38.1 mm to (179.9, 84.7), turned to 90 degrees
- moved J1 37.5 mm to (178.5, 91.1), turned to 90 degrees
- moved U1 35.0 mm to (177.0, 84.5), turned to 0 degrees
- moved C2 31.9 mm to (174.2, 84.7), turned to 90 degrees
- moved JP1 26.5 mm to (108.0, 102.3), turned to 180 degrees
- moved U8 24.4 mm to (177.3, 120.9), turned to -90 degrees
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Connections:
- R8 pad 2: IMU_SDA -> IMU_SCL
- R9 pad 2: IMU_SCL -> IMU_SDA
- U2 pad 1: ESP_D+ -> USB_D+
- U2 pad 3: ESP_D- -> USB_D-
- U6 pad 16: unconnected-(U6-GPIO12/TOUCH12/ADC2_CH1/FSPICLK/FSPIIO6/SUBSPICLK-Pad16) -> IMU_SCL
- U6 pad 17: unconnected-(U6-GPIO13/TOUCH13/ADC2_CH2/FSPIQ/FSPIIO7/SUBSPIQ-Pad17) -> IMU_SDA
- U6 pad 27: unconnected-(U6-GPIO47/SPICLK_P/SUBSPICLK_P_DIFF-Pad27) -> A7670_PWR
- U6 pad 28: unconnected-(U6-SPIIO4/GPIO33/FSPIHD/SUBSPIHD-Pad28) -> A7670_STATUS
- U6 pad 29: unconnected-(U6-SPIIO5/GPIO34/FSPICS0/SUBSPICS0-Pad29) -> A7670_RST
- U6 pad 30: unconnected-(U6-GPIO48/SPICLK_N/SUBSPICLK_N_DIFF-Pad30) -> EN_MIC29302
- U6 pad 31: unconnected-(U6-SPIIO6/GPIO35/FSPID/SUBSPID-Pad31) -> GPS_RX
- U6 pad 32: unconnected-(U6-SPIIO7/GPIO36/FSPICLK/SUBSPICLK-Pad32) -> GPS_TX
- U6 pad 33: unconnected-(U6-SPIDQS/GPIO37/FSPIQ/SUBSPIQ-Pad33) -> GPS_FORCE_ON
- U6 pad 34: unconnected-(U6-GPIO38/FSPIWP/SUBSPIWP-Pad34) -> GPS_RST
- U6 pad 39: GPS_RX -> A7670_RX
- U6 pad 40: GPS_TX -> A7670_TX
Routing:
- net IMU_SCL: track 0.00 -> 92.5 mm, vias 0 -> 3
- net IMU_SDA: track 0.00 -> 91.5 mm, vias 0 -> 3
- net VBUS: track 0.00 -> 91.0 mm, vias 0 -> 6
- net EN_MIC29302: track 0.00 -> 73.6 mm, vias 0 -> 2
- net A7670_STATUS: track 0.00 -> 48.5 mm, vias 0 -> 2
- net A7670_PWR: track 0.00 -> 39.6 mm, vias 0 -> 2
- net VDD_BAT: track 53.8 -> 16.1 mm, vias 0 -> 26
- net GPS_FORCE_ON: track 0.00 -> 36.0 mm, vias 0 -> 2
- net A7670_TX: track 7.50 -> 43.1 mm
- net A7670_RX: track 0.00 -> 34.6 mm
- net USB_D+: track 3.40 -> 30.8 mm
- net GPS_RST: track 0.00 -> 27.0 mm, vias 0 -> 2
- net ESP_BOOT: track 0.00 -> 25.9 mm, vias 0 -> 2
- net A7670_BOOT: track 0.00 -> 25.9 mm
- net USB_D-: track 6.03 -> 30.0 mm
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- added copper zone on F.Cu, net +BATT
- added copper zone on In2.Cu, net +BATT
- added copper zone on B.Cu, net GND
- added copper zone on F.Cu, net IMU_VDD
- added copper zone on In2.Cu, net IMU_VDD
- added copper zone on F.Cu, net Net-(U3-SW)
- added copper zone on F.Cu, net VBUS
- added copper zone on F.Cu, net VDD_1V8
- added copper zone on In2.Cu, net VDD_1V8
- added copper zone on F.Cu, net VDD_BAT
- added copper zone on In2.Cu, net VDD_BAT
Other:
- outline, holes or cut-outs redrawn

Commit message: Update bwlc1a.kicad_pcb
Routing:
- net VDD_1V8: track 7.90 -> 13.9 mm
- net A7670_BOOT: track 25.9 -> 27.8 mm
- net IMU_VDD: track 23.7 -> 22.8 mm
- net A7670_UART_RX: track 8.28 -> 8.87 mm
Changed lines of the file:
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@@
   (via (at 178.8448 97.282) (size 0.4) (drill 0.3) (layers "F.Cu" "B.Cu") (free) (net 3))
   (via (at 175.247 86.815) (size 0.4) (drill 0.3) (layers "F.Cu" "B.Cu") (free) (net 3))
-  (segment (start 138.1836 91.4168) (end 140.766 91.4168) (width 0.4) (layer "F.Cu") (net 4))
-  (segment (start 140.766 91.4168) (end 140.9078 91.5586) (width 0.4) (layer "F.Cu") (net 4))
-  (segment (start 137.9762 92.0814) (end 137.9762 91.6242) (width 0.4) (layer "F.Cu") (net 4))
   (segment (start 113.4364 124.5388) (end 113.4364 123.1112) (width 0.4) (layer "F.Cu") (net 4))
   (segment (start 140.9078 93.113599) (end 140.9378 93.143599) (width 0.4) (layer "F.Cu") (net 4))
@@
   (segment (start 140.9078 92.0768) (end 140.9078 93.113599) (width 0.4) (layer "F.Cu") (net 4))
   (segment (start 119.788101 125.29205) (end 119.788101 124.7843) (width 0.3) (layer "F.Cu") (net 4))
+  (segment (start 140.9078 91.5586) (end 140.9078 92.0768) (width 0.4) (layer "F.Cu") (net 4))
   (segment (start 113.4364 124.5388) (end 112.2778 124.5388) (width 0.4) (layer "F.Cu") (net 4))
   (segment (start 132.0624 122.6278) (end 132.0924 122.6578) (width 0.4) (layer "F.Cu") (net 4))
@@
   (segment (start 122.0758 124.206) (end 122.2848 124.206) (width 0.6) (layer "F.Cu") (net 4))
   (segment (start 133.4164 122.9196) (end 133.4164 121.1026) (width 0.4) (layer "F.Cu") (net 4))
-  (segment (start 140.9078 91.5586) (end 140.9078 92.0768) (width 0.4) (layer "F.Cu") (net 4))
   (segment (start 131.0256 122.6278) (end 132.0624 122.6278) (width 0.4) (layer "F.Cu") (net 4))
   (segment (start 127.488 122.662999) (end 127.487999 122.663) (width 0.4) (layer "F.Cu") (net 4))
@@
   (segment (start 122.8756 126.3968) (end 122.8456 126.4268) (width 0.6) (layer "F.Cu") (net 4))
   (segment (start 127.487999 122.663) (end 127.9178 122.663) (width 0.4) (layer "F.Cu") (net 4))
-  (segment (start 137.9762 91.6242) (end 138.1836 91.4168) (width 0.4) (layer "F.Cu") (net 4))
   (segment (start 118.788101 126.6093) (end 118.788101 127.779299) (width 0.3) (layer "F.Cu") (net 4))
   (segment (start 132.0924 122.6578) (end 133.1546 122.6578) (width 0.4) (layer "F.Cu") (net 4))
@@
   (via (at 132.829 121.105) (size 0.4) (drill 0.3) (layers "F.Cu" "B.Cu") (free) (net 4))
   (via (at 122.0758 124.206) (size 0.4) (drill 0.3) (layers "F.Cu" "B.Cu") (net 4))
-  (via (at 137.9762 92.0814) (size 0.4) (drill 0.3) (layers "F.Cu" "B.Cu") (net 4))
+  (via (at 140.9078 91.5586) (size 0.4) (drill 0.3) (layers "F.Cu" "B.Cu") (net 4))
   (via (at 119.788101 125.29205) (size 0.4) (drill 0.3) (layers "F.Cu" "B.Cu") (net 4))
   (via (at 111.4078 123.952) (size 0.4) (drill 0.3) (layers "F.Cu" "B.Cu") (free) (net 4))
@@
   (via (at 127.9178 121.647) (size 0.4) (drill 0.3) (layers "F.Cu" "B.Cu") (net 4))
   (via (at 127.9178 122.663) (size 0.4) (drill 0.3) (layers "F.Cu" "B.Cu") (net 4))
+  (segment (start 140.9078 91.5586) (end 138.9588 91.5586) (width 0.4) (layer "In2.Cu") (net 4))
+  (segment (start 138.9588 91.5586) (end 138.4808 92.0366) (width 0.4) (layer "In2.Cu") (net 4))
   (segment (start 130.9728 123.7006) (end 131.0256 123.6478) (width 0.2) (layer "F.Cu") (net 5))
   (segment (start 132.0924 123.6178) (end 131.0556 123.6178) (width 0.2) (layer "F.Cu") (net 5))
@@
   (via (at 145.9608 102.309) (size 0.4) (drill 0.3) (layers "F.Cu" "B.Cu") (free) (net 17))
   (via (at 145.4782 102.7916) (size 0.4) (drill 0.3) (layers "F.Cu" "B.Cu") (free) (net 17))
+  (segment (start 138.7194 84.432) (end 138.6078 84.5436) (width 0.4) (layer "In2.Cu") (net 17))
+  (segment (start 138.6078 84.5436) (end 138.6078 86.9566) (width 0.4) (layer "In2.Cu") (net 17))
+  (segment (start 138.6078 86.9566) (end 138.6078 89.4966) (width 0.4) (layer "In2.Cu") (net 17))
+  (segment (start 139.56 84.432) (end 138.7194 84.432) (width 0.4) (layer "In2.Cu") (net 17))
   (segment (start 141.9498 94.0481) (end 142.3813 94.4796) (width 0.2) (layer "F.Cu") (net 18))
   (segment (start 141.9798 93.113599) (end 141.9498 93.143599) (width 0.2) (layer "F.Cu") (net 18))
@@
   (segment (start 150.6318 81.1228) (end 150.609 81.1) (width 0.34925) (layer "F.Cu") (net 27))
   (segment (start 151.623 81.1228) (end 150.6318 81.1228) (width 0.34925) (layer "F.Cu") (net 27))
-  (segment (start 138.7636 89.6176) (end 138.7636 80.6514) (width 0.2) (layer "F.Cu") (net 28))
-  (segment (start 142.1404 80.796446) (end 142.1404 81.1) (width 0.2) (layer "F.Cu") (net 28))
-  (segment (start 139.315 80.1) (end 141.443954 80.1) (width 0.2) (layer "F.Cu") (net 28))
-  (segment (start 139.297 90.151) (end 138.7636 89.6176) (width 0.2) (layer "F.Cu") (net 28))
-  (segment (start 143.9724 90.4322) (end 143.6912 90.151) (width 0.2) (layer "F.Cu") (net 28))
-  (segment (start 143.6912 90.151) (end 139.297 90.151) (width 0.2) (layer "F.Cu") (net 28))
+  (segment (start 138.303 80.1494) (end 138.4554 79.997) (width 0.2) (layer "F.Cu") (net 28))
   (segment (start 144.515 93.5218) (end 143.9724 92.9792) (width 0.2) (layer "F.Cu") (net 28))
+  (segment (start 138.303 90.0554) (end 138.303 80.1494) (width 0.2) (layer "F.Cu") (net 28))
+  (segment (start 142.0114 79.997) (end 142.1404 80.126) (width 0.2) (layer "F.Cu") (net 28))
+  (segment (start 143.7894 90.2586) (end 138.5062 90.2586) (width 0.2) (layer "F.Cu") (net 28))
+  (segment (start 144.715 93.5218) (end 144.515 93.5218) (width 0.2) (layer "F.Cu") (net 28))
+  (segment (start 142.1404 80.126) (end 142.1404 81.1) (width 0.2) (layer "F.Cu") (net 28))
+  (segment (start 143.9724 92.9792) (end 143.9724 90.4416) (width 0.2) (layer "F.Cu") (net 28))
+  (segment (start 138.5062 90.2586) (end 138.303 90.0554) (width 0.2) (layer "F.Cu") (net 28))
   (segment (start 142.961 81.9206) (end 142.1404 81.1) (width 0.2) (layer "F.Cu") (net 28))
-  (segment (start 141.443954 80.1) (end 142.1404 80.796446) (width 0.2) (layer "F.Cu") (net 28))
-  (segment (start 144.715 93.5218) (end 144.515 93.5218) (width 0.2) (layer "F.Cu") (net 28))
-  (segment (start 138.7636 80.6514) (end 139.315 80.1) (width 0.2) (layer "F.Cu") (net 28))
-  (segment (start 143.9724 92.9792) (end 143.9724 90.4322) (width 0.2) (layer "F.Cu") (net 28))
+  (segment (start 143.9724 90.4416) (end 143.7894 90.2586) (width 0.2) (layer "F.Cu") (net 28))
+  (segment (start 138.4554 79.997) (end 142.0114 79.997) (width 0.2) (layer "F.Cu") (net 28))
   (segment (start 142.961 84.432) (end 142.961 81.9206) (width 0.2) (layer "F.Cu") (net 28))
   (segment (start 145.42 119.4832) (end 145.42 121.124) (width 0.2) (layer "F.Cu") (net 29))
@@
   (segment (start 108.8471 95.842198) (end 107.8351 95.842198) (width 0.2) (layer "F.Cu") (net 42))
   (segment (start 107.8351 95.842198) (end 107.8351 94.8107) (width 0.2) (layer "F.Cu") (net 42))
-  (segment (start 143.0184 95.4296) (end 144.1106 96.5218) (width 0.2) (layer "F.Cu") (net 43))
-  (segment (start 144.1106 96.5218) (end 144.715 96.5218) (width 0.2) (layer "F.Cu") (net 43))
-  (segment (start 140.5063 95.4296) (end 143.0184 95.4296) (width 0.2) (layer "F.Cu") (net 43))
+  (segment (start 143.6518 95.4296) (end 143.8148 95.5926) (width 0.2) (layer "F.Cu") (net 43))
+  (segment (start 143.8148 96.3948) (end 143.9418 96.5218) (width 0.2) (layer "F.Cu") (net 43))
+  (segment (start 143.8148 95.5926) (end 143.8148 96.3948) (width 0.2) (layer "F.Cu") (net 43))
+  (segment (start 143.9418 96.5218) (end 144.715 96.5218) (width 0.2) (layer "F.Cu") (net 43))
+  (segment (start 140.5063 95.4296) (end 143.6518 95.4296) (width 0.2) (layer "F.Cu") (net 43))
   (segment (start 140.5041 98.107799) (end 143.608801 98.107799) (width 0.2) (layer "F.Cu") (net 44))
-  (segment (start 143.8018 100.5604) (end 143.8018 97.9148) (width 0.2) (layer "F.Cu") (net 44))
-  (segment (start 143.8018 97.9148) (end 144.1948 97.5218) (width 0.2) (layer "F.Cu") (net 44))
-  (segment (start 144.1948 97.5218) (end 144.715 97.5218) (width 0.2) (layer "F.Cu") (net 44))
+  (segment (start 143.8018 97.6618) (end 143.9418 97.5218) (width 0.2) (layer "F.Cu") (net 44))
+  (segment (start 143.7278 101.3946) (end 143.8018 101.3206) (width 0.2) (layer "F.Cu") (net 44))
+  (segment (start 143.8018 101.3206) (end 143.8018 97.9148) (width 0.2) (layer "F.Cu") (net 44))
+  (segment (start 143.8018 97.9148) (end 143.8018 97.6618) (width 0.2) (layer "F.Cu") (net 44))
   (segment (start 143.608801 98.107799) (end 143.8018 97.9148) (width 0.2) (layer "F.Cu") (net 44))
-  (segment (start 142.9676 101.3946) (end 143.8018 100.5604) (width 0.2) (layer "F.Cu") (net 44))
+  (segment (start 142.9676 101.3946) (end 143.7278 101.3946) (width 0.2) (layer "F.Cu") (net 44))
+  (segment (start 143.9418 97.5218) (end 144.715 97.5218) (width 0.2) (layer "F.Cu") (net 44))
   (segment (start 139.604001 99.057799) (end 142.3791 99.057799) (width 0.2) (layer "F.Cu") (net 45))
   (segment (start 117.0464 107.0104) (end 117.2942 106.7626) (width 0.2) (layer "F.Cu") (net 45))
@@
         (xy 146.926 109.167)
         (xy 137.274 109.167)
-        (xy 137.274 84.021)
-        (xy 146.926 84.021)
+        (xy 137.274 88.974)
+        (xy 146.926 88.974)
       )
     )
@@
         (xy 165.8178 79.8386)
         (xy 126.1938 79.8386)
-        (xy 126.1938 91.0146)
-        (xy 167.3418 91.0146)
+        (xy 126.1938 108.2866)
+        (xy 167.3418 108.2866)
         (xy 167.3418 115.9066)
       )

Commit message: PCB Layout update + Silkscreen
Parts:
- added G***: LOGO, Teapot:TeapotLogo, F.Cu at (133.5, 110.8)
- added G***: LOGO, Teapot:TeapotLogo, B.Cu at (140.1, 82.0)
- added J3: JTAG_10PIN, Connector:Tag-Connect_TC2050-IDC-NL_2x05_P1.27mm_Vertical, F.Cu at (116.6, 105.4)
- JP1: footprint Jumper:SolderJumper-2_P1.3mm_Open_RoundedPad1.0x1.5mm -> Button_Switch_SMD:SW_Push_1P1T_NO_CK_KMR2
- moved R11 7.03 mm to (109.4, 89.1), turned to 180 degrees
- moved R12 7.03 mm to (107.3, 89.1), turned to 180 degrees
- moved JP1 5.49 mm to (108.3, 96.9), turned to -90 degrees
- moved C17 5.13 mm to (107.3, 106.8), turned to 180 degrees
- moved R14 3.81 mm to (109.3, 106.8), turned to 180 degrees
- moved SW1 2.27 mm to (108.3, 103.5), turned to 90 degrees
- moved Q2 1.90 mm to (108.3, 91.5), turned to 180 degrees
Connections:
- R14 pad 1: +3V3 -> IMU_VDD
- U6 pad 25: unconnected-(U6-GPIO21-Pad25) -> MAX17048_INT
- U6 pad 6: unconnected-(U6-GPIO2/TOUCH2/ADC1_CH1-Pad6) -> IMU_INT
Routing:
- net MAX17048_INT: track 0.00 -> 75.2 mm, vias 0 -> 2
- net ESP_BOOT: track 25.9 -> 32.9 mm
- net JTAG_TDI: track 0.00 -> 5.86 mm
- net IMU_INT: track 0.00 -> 5.47 mm
- net JTAG_TDO: track 0.00 -> 5.46 mm
- net JTAG_TMS: track 0.00 -> 5.19 mm, vias 0 -> 2
- net GPS_RST: track 27.0 -> 32.2 mm
- net JTAG_TCK: track 0.00 -> 5.14 mm
- net ESP_EN: track 11.1 -> 15.3 mm
- net GND: track 56.6 -> 53.4 mm, vias 170 -> 246
- net Net-(Q2-C): track 6.30 -> 4.46 mm
- net IMU_VDD: track 22.8 -> 24.1 mm
- net Net-(U9-VBUS): track 7.73 -> 8.59 mm
- net A7670_RX: track 34.6 -> 33.9 mm, vias 0 -> 2
- net Net-(U9-USB_DP): track 7.23 -> 7.80 mm
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Other:
- board text added: "+"
- board text added: "3V3 POWER SUPPLY"
- board text added: "ANT"
- board text added: "B"
- board text added: "BATT"
- board text added: "BWLC1A"
- board text added: "CELL BOOT"
- board text added: "CELL USB TP"
- board text added: "D+"
- board text added: "D-"
- board text added: "DEBUG"
- board text added: "F"
- board text added: "GND"
- board text added: "GPS & CELL PWR SUPPLY"
- board text added: "IMU"
- board text added: "PWR SEL"
- board text added: "R"
- board text added: "Rev. 1"
- board text added: "Teapot Laboratories"
- board text added: "VBUS"
- board text added: "Vo=3.87V"
- board text added: "X X GND GND VDD -------------- RST TDI TDO TCK TMS"

Commit message: Update bwlc1a.kicad_pcb
Other:
- board text added: "CELL USB"
- board text added: "X X GND GND VDD - - - - - - - - - RST TDI TDO TCK TMS"
- board text removed: "CELL USB TP"
- board text removed: "X X GND GND VDD -------------- RST TDI TDO TCK TMS"
Changed lines of the file:
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@@
     (effects (font (size 1 1) (thickness 0.15)) (justify left))
   )
-  (gr_text "X  X  GND  GND  VDD \n--------------\nRST TDI TDO TCK TMS " (at 123.1138 107.1496) (layer "F.SilkS")
+  (gr_text "X  X  GND  GND  VDD \n- - - - - - - - -\nRST TDI TDO TCK TMS " (at 123.1138 107.1496) (layer "F.SilkS")
     (effects (font (size 0.6 0.6) (thickness 0.15)) (justify left bottom))
   )
@@
     (effects (font (size 0.8 0.8) (thickness 0.15)) (justify left))
   )
-  (gr_text "CELL\nUSB TP" (at 140.0048 110.8326) (layer "F.SilkS" knockout)
+  (gr_text "CELL\nUSB" (at 141.6558 110.8326) (layer "F.SilkS" knockout)
     (effects (font (size 0.8 0.8) (thickness 0.15)) (justify left))
   )
@@
   (via (at 180.5466 86.214) (size 0.4) (drill 0.3) (layers "F.Cu" "B.Cu") (net 1))
   (via (at 180.0894 86.214) (size 0.4) (drill 0.3) (layers "F.Cu" "B.Cu") (free) (net 1))
-  (segment (start 170.0818 91.0146) (end 173.1298 87.9666) (width 0.6) (layer "B.Cu") (net 1))
-  (segment (start 170.0818 106.2546) (end 170.0818 91.0146) (width 0.6) (layer "B.Cu") (net 1))
   (segment (start 179.175 86.214) (end 180.5466 86.214) (width 0.6) (layer "B.Cu") (net 1))
   (segment (start 144.786899 122.075701) (end 144.786899 116.6092) (width 0.6) (layer "B.Cu") (net 1))
-  (segment (start 167.2878 109.0486) (end 170.0818 106.2546) (width 0.6) (layer "B.Cu") (net 1))
+  (segment (start 170.0818 106.7271) (end 170.0818 91.0146) (width 0.6) (layer "B.Cu") (net 1))
+  (segment (start 177.4224 87.9666) (end 179.175 86.214) (width 0.6) (layer "B.Cu") (net 1))
+  (segment (start 144.786899 116.6092) (end 144.786899 111.737501) (width 0.6) (layer "B.Cu") (net 1))
+  (segment (start 170.0818 91.0146) (end 173.1298 87.9666) (width 0.6) (layer "B.Cu") (net 1))
+  (segment (start 167.7603 109.0486) (end 170.0818 106.7271) (width 0.6) (layer "B.Cu") (net 1))
+  (segment (start 173.1298 87.9666) (end 177.4224 87.9666) (width 0.6) (layer "B.Cu") (net 1))
+  (segment (start 147.4758 109.0486) (end 167.7603 109.0486) (width 0.6) (layer "B.Cu") (net 1))
   (segment (start 144.786899 111.737501) (end 147.4758 109.0486) (width 0.6) (layer "B.Cu") (net 1))
-  (segment (start 177.4224 87.9666) (end 179.175 86.214) (width 0.6) (layer "B.Cu") (net 1))
-  (segment (start 147.4758 109.0486) (end 167.2878 109.0486) (width 0.6) (layer "B.Cu") (net 1))
-  (segment (start 144.786899 116.6092) (end 144.786899 111.737501) (width 0.6) (layer "B.Cu") (net 1))
-  (segment (start 173.1298 87.9666) (end 177.4224 87.9666) (width 0.6) (layer "B.Cu") (net 1))
   (segment (start 144.5892 122.2734) (end 144.786899 122.075701) (width 0.6) (layer "B.Cu") (net 1))
   (segment (start 157.0808 83.5384) (end 157.7034 83.5384) (width 0.6) (layer "F.Cu") (net 2))
@@
   (segment (start 153.0822 109.0546) (end 154.115 108.0218) (width 0.2) (layer "F.Cu") (net 60))
   (segment (start 147.6686 110.8688) (end 147.6686 109.3918) (width 0.2) (layer "F.Cu") (net 60))
-  (segment (start 151.2186 109.9058) (end 151.5618 109.5626) (width 0.2) (layer "F.Cu") (net 61))
-  (segment (start 151.5618 109.5626) (end 155.6742 109.5626) (width 0.2) (layer "F.Cu") (net 61))
+  (segment (start 151.2186 109.7788) (end 151.4348 109.5626) (width 0.2) (layer "F.Cu") (net 61))
+  (segment (start 151.4348 109.5626) (end 155.6742 109.5626) (width 0.2) (layer "F.Cu") (net 61))
+  (segment (start 151.2186 110.8688) (end 151.2186 109.7788) (width 0.2) (layer "F.Cu") (net 61))
+  (segment (start 157.115 108.1218) (end 157.115 107.9218) (width 0.2) (layer "F.Cu") (net 61))
   (segment (start 155.6742 109.5626) (end 157.115 108.1218) (width 0.2) (layer "F.Cu") (net 61))
-  (segment (start 151.2186 110.8688) (end 151.2186 109.9058) (width 0.2) (layer "F.Cu") (net 61))
-  (segment (start 157.115 108.1218) (end 157.115 107.9218) (width 0.2) (layer "F.Cu") (net 61))
   (segment (start 155.82926 110.8688) (end 158.115 108.58306) (width 0.2) (layer "F.Cu") (net 62))
   (segment (start 154.7686 110.8688) (end 155.82926 110.8688) (width 0.2) (layer "F.Cu") (net 62))
