File: hardware/kicad/bwlc1a.kicad_pcb (KiCad board)
At the start: 4 copper layers, 80 x 50 mm, 106 parts, among them J1 JST-2PH, J2 USB_C_Receptacle_USB2.0, J3 JTAG_10PIN, J4 Nano SIM, J5 RSP-122811-02, Q1 DMG3415UQ-7, Q2 NPN, Q3 NPN, Q4 NPN, Q5 NPN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

Commit message: Update PCB
Parts:
- C15, C16: value 9p -> 12p
- C20: footprint Capacitor_SMD:CP_Elec_6.3x7.7 -> Capacitor_SMD:CP_Elec_6.3x5.4
- C31, C32: footprint Capacitor_SMD:C_0603_1608Metric -> Capacitor_SMD:C_0805_2012Metric
- C34: value 470p (N.C) -> 470p
- D3: value D_TVS -> ESDBW5V0A1
- F1: value 3A -> 2A; footprint Fuse:Fuse_1206_3216Metric -> Fuse:Fuse_1812_4532Metric
- Q1: footprint Keebio-Parts:SOT-23 -> Package_TO_SOT_SMD:SOT-23
- Q2, Q3, Q4, Q5, Q6: value NPN -> S8050
- R6: value 10K -> 10k
- Y1: footprint Crystal:Crystal_SMD_2012-2Pin_2.0x1.2mm -> Crystal:Crystal_SMD_3215-2Pin_3.2x1.5mm
- moved JP1 26.7 mm to (134.7, 92.2)
- moved SW1 26.7 mm to (134.7, 98.8)
- moved C17 26.4 mm to (133.4, 102.7), turned to -90 degrees
- moved R14 25.6 mm to (134.5, 102.7), turned to 90 degrees
- moved Q2 11.0 mm to (112.3, 81.2), turned to 90 degrees
- moved R11 10.3 mm to (114.6, 80.2), turned to -90 degrees
- moved R12 10.0 mm to (114.6, 82.3), turned to 90 degrees
- moved R13 6.19 mm to (115.6, 82.3)
- moved C14 2.47 mm to (132.9, 86.4), turned to 90 degrees
- moved C15 2.20 mm to (129.0, 119.7), turned to 90 degrees
- moved C16 2.12 mm to (129.0, 117.8), turned to 90 degrees
- moved C13 1.82 mm to (131.5, 87.0), turned to 90 degrees
- moved C28 1.18 mm to (159.4, 82.9)
- moved C30 1.18 mm to (161.2, 82.9)
- moved C27 1.18 mm to (158.4, 82.9)
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Routing:
- net ESP_EN: track 15.3 -> 37.5 mm
- net ESP_BOOT: track 32.9 -> 54.5 mm
- net Net-(Q2-C): track 4.46 -> 12.4 mm
- net GPS_RST: track 32.2 -> 39.7 mm
- net GND: track 53.4 -> 59.7 mm, vias 246 -> 250
- net VDD_BAT: track 16.1 -> 10.8 mm
- net GPS_FORCE_ON: track 36.0 -> 33.9 mm
- net Net-(Q2-B): track 2.75 -> 4.59 mm
- net Net-(J4-RST): track 11.7 -> 13.1 mm
- net IMU_SDA: track 91.8 -> 93.1 mm
- net Net-(J4-CLK): track 9.85 -> 10.9 mm
- net IMU_SCL: track 92.8 -> 93.8 mm
- net ESP_32K_N: track 3.54 -> 4.52 mm
- net ESP_32K_P: track 3.47 -> 4.43 mm
- net Net-(J4-I/O): track 20.9 -> 21.9 mm
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Other:
- board text added: "+ BATT -"
- board text removed: "+"
- board text removed: "BATT"
