File: hardware/kicad/bwlc1a.kicad_pcb (KiCad board)
At the start: 4 copper layers, 80 x 50 mm, 106 parts, among them J1 JST-2PH, J2 USB_C_Receptacle_USB2.0, J3 JTAG_10PIN, J4 Nano SIM, J5 RSP-122811-02, Q1 DMG3415UQ-7, Q2 S8050, Q3 S8050, Q4 S8050, Q5 S8050, Q6 S8050, SW1 EN_ESP, U1 MCP73831-2-OT, U2 USBLC6-2SC6, U3 TPS62290DRVR, U4 MAX17048G+, U5 LSM6DS3, U6 ESP32-S3-MINI-1, U7 L86-M33, U8 MIC29302WU, U9 A7670C_24x24mm, Y1 32.768 kHz

Commit message: Production file update
Parts:
- moved J1 1.29 mm to (177.2, 91.1)
- moved C9 0.11 mm to (119.2, 127.8)
Connections:
- J5 pad 3: (no net) -> GND
Routing:
- net IMU_VDD: track 21.4 -> 103.2 mm, vias 14 -> 11
- net +BATT: track 10.3 -> 64.7 mm
- net VDD_BAT: track 10.8 -> 51.6 mm
- net VDD_1V8: track 6.14 -> 28.3 mm, vias 10 -> 6
- net GND: track 52.3 -> 55.9 mm, vias 203 -> 320
- net ESP_BOOT: track 54.4 -> 53.1 mm
- net A7670_TX: track 39.8 -> 39.6 mm, vias 2 -> 3
- added copper zone on B.Cu, net +BATT
- added copper zone on In2.Cu, net GND
- added copper zone on B.Cu, net VDD_BAT
- removed copper zone on In2.Cu, net +BATT
- removed copper zone on In2.Cu, net IMU_VDD
- removed copper zone on In2.Cu, net VDD_1V8
- removed copper zone on In2.Cu, net VDD_BAT
Other:
- outline, holes or cut-outs redrawn

Commit message: Update bwlc1a.kicad_pcb
Routing:
- net GND: vias 320 -> 437

Commit message: Update PCB
Parts:
- J4: value Nano SIM -> SMN-304; footprint GCT_SIM8051-6-0-14-00-X-REVD:GCT_SIM8051-6-0-14-00-X-REVD -> SIM-SMD_SMN-304:SIM-SMD_SMN-304
- J5: value RSP-122811-02 -> BWIPX-1-001E
- JP2: footprint Jumper:SolderJumper-3_P1.3mm_Bridged2Bar12_RoundedPad1.0x1.5mm -> Jumper:SolderJumper-3_P1.3mm_Bridged12_RoundedPad1.0x1.5mm
- moved C25 16.2 mm to (166.4, 127.3), turned to 0 degrees
- moved U2 3.60 mm to (139.3, 115.4)
- moved D4 1.41 mm to (166.6, 112.5)
- moved R16 1.21 mm to (162.1, 111.8)
- moved R17 0.83 mm to (163.1, 111.8)
- moved G*** 0.79 mm to (133.2, 110.6)
- moved J4 0.30 mm to (159.4, 121.6), turned to 0 degrees
- moved R20 0.19 mm to (161.0, 111.8), turned to 90 degrees
Connections:
- D4 pad 1: Net-(J4-I/O) -> USIM_VDD
- D4 pad 3: Net-(J4-CLK) -> Net-(J4-RST)
- D4 pad 4: Net-(J4-RST) -> Net-(J4-CLK)
- D4 pad 5: USIM_VDD -> Net-(J4-I/O)
- J4 pad 1: USIM_VDD -> unconnected-(J4-Pad1)
- J4 pad 2: Net-(J4-RST) -> unconnected-(J4-Pad2)
- R16 pad 1: USIM_RST -> USIM_CLK
- R16 pad 2: Net-(J4-RST) -> Net-(J4-CLK)
- R17 pad 1: USIM_CLK -> USIM_RST
- R17 pad 2: Net-(J4-CLK) -> Net-(J4-RST)
- R20 pad 1: USIM_DATA -> Net-(J4-I/O)
- R20 pad 2: Net-(J4-I/O) -> USIM_DATA
Routing:
- net Net-(J4-CLK): track 7.85 -> 25.5 mm
- net USIM_VDD: track 13.8 -> 27.9 mm
- net Net-(J4-RST): track 11.2 -> 22.9 mm
- net Net-(J4-I/O): track 19.5 -> 12.6 mm, vias 0 -> 2
- net +BATT: track 64.7 -> 70.8 mm, vias 21 -> 8
- net VBUS: track 91.5 -> 95.5 mm
- net IMU_VDD: track 103.2 -> 106.1 mm, vias 11 -> 6
- net IMU_SCL: track 93.8 -> 92.9 mm
- net JTAG_TMS: track 5.12 -> 5.95 mm
- net ESP_BOOT: track 53.1 -> 53.8 mm
- net GND: track 55.9 -> 56.4 mm, vias 437 -> 429
- net VDD_BAT: track 51.6 -> 51.3 mm, vias 26 -> 12
- net VDD_1V8: vias 6 -> 2
- net A7670_TX: vias 3 -> 2

Commit message: update design
Parts:
- added TP5: BOOT, TestPoint:TestPoint_Pad_D1.0mm, F.Cu at (102.3, 93.8)
- added TP6: RESET, TestPoint:TestPoint_Pad_D1.0mm, F.Cu at (102.5, 99.2)
- added TP7: TXD, TestPoint:TestPoint_Pad_D1.0mm, F.Cu at (101.9, 105.1)
- added TP8: RXD, TestPoint:TestPoint_Pad_D1.0mm, F.Cu at (102.2, 111.3)
- JP2: footprint Jumper:SolderJumper-3_P1.3mm_Bridged12_RoundedPad1.0x1.5mm -> Jumper:SolderJumper-3_P1.3mm_Bridged2Bar12_RoundedPad1.0x1.5mm
- renumbered JP1 to SW2
Connections:
- U6 pad 39: A7670_RX -> Net-(U6-U0TXD/GPIO43/CLK_OUT1)
- U6 pad 40: A7670_TX -> Net-(U6-U0RXD/GPIO44/CLK_OUT2)
Routing:
- net +BATT: track 70.8 -> 74.1 mm, vias 8 -> 7
- net GND: track 56.4 -> 55.7 mm, vias 429 -> 385
Other:
- board text removed: "Vo=3.87V"

Commit message: Early PCB Layouting
Parts:
- removed D2: B5819W, Diode_SMD:D_SOD-123
- removed D3: ESDBW5V0A1, Capacitor_SMD:C_0402_1005Metric
- removed D6: PESD0402, Capacitor_SMD:C_0402_1005Metric
- removed G*** (x2): LOGO, Teapot:TeapotLogo
- removed JP2: EN_MIC29302, Jumper:SolderJumper-3_P1.3mm_Bridged2Bar12_RoundedPad1.0x1.5mm
- removed JP3: A7670_BOOT, Jumper:SolderJumper-2_P1.3mm_Open_RoundedPad1.0x1.5mm
- removed Q1: DMG3415UQ-7, Package_TO_SOT_SMD:SOT-23
- added C22: DNP, Capacitor_Tantalum_SMD:CP_EIA-3528-15_AVX-H, F.Cu at (137.3, 54.2)
- added C23: 10u, Capacitor_SMD:C_0603_1608Metric, F.Cu at (132.1, 51.9)
- added C24: 1u, Capacitor_SMD:C_0603_1608Metric, F.Cu at (182.1, 51.6)
- added C26: 10u, Capacitor_SMD:C_0603_1608Metric, F.Cu at (182.1, 54.1)
- added C39: 100n, Capacitor_SMD:C_0603_1608Metric, F.Cu at (150.5, 80.2)
- added C40: 100n, Capacitor_SMD:C_0603_1608Metric, F.Cu at (143.7, 81.8)
- added C41: 100n, Capacitor_SMD:C_0603_1608Metric, F.Cu at (143.7, 84.3)
- added C42: 10u, Capacitor_SMD:C_0603_1608Metric, F.Cu at (143.7, 86.8)
- added C43: 4u7, Capacitor_SMD:C_0603_1608Metric, F.Cu at (143.7, 89.3)
- added C44: 1u, Capacitor_SMD:C_0603_1608Metric, F.Cu at (174.2, 51.7)
- added C45: 10u, Capacitor_SMD:C_0603_1608Metric, F.Cu at (174.2, 54.2)
- added C47: 33p, Capacitor_SMD:C_0402_1005Metric, F.Cu at (190.0, 106.8)
- added C48: TBD, Capacitor_SMD:C_0402_1005Metric, F.Cu at (133.3, 70.9)
- added C49: TBD, Capacitor_SMD:C_0402_1005Metric, F.Cu at (133.3, 72.9)
- added C50: 47p, Capacitor_SMD:C_0402_1005Metric, F.Cu at (122.7, 121.5)
- added C51: 1.4p, Capacitor_SMD:C_0402_1005Metric, F.Cu at (122.7, 118.7)
- added C52: 1.2p, Capacitor_SMD:C_0402_1005Metric, F.Cu at (123.2, 117.2)
- added C53: 2p, Capacitor_SMD:C_0402_1005Metric, F.Cu at (123.2, 113.3)
- added D8: ESD5651N, Capacitor_SMD:C_0402_1005Metric, F.Cu at (147.1, 80.5)
- added E2: NN03-310, bwlc1a:NN03-310, F.Cu at (111.7, 109.8)
- added FB2: MMZ1608B601CTAH0, Inductor_SMD:L_0603_1608Metric, F.Cu at (160.9, 170.5)
- added FB3: 0.4p, Inductor_SMD:L_0402_1005Metric, F.Cu at (113.9, 121.5)
- added FB4: 11n, Inductor_SMD:L_0603_1608Metric, F.Cu at (115.2, 121.5)
- added FB5: 0, Inductor_SMD:L_0402_1005Metric, F.Cu at (113.9, 98.0)
- added FB6: 0, Inductor_SMD:L_0603_1608Metric, F.Cu at (115.2, 98.0)
- added J6: Qwiic, Connector_JST:JST_SH_SM04B-SRSS-TB_1x04-1MP_P1.00mm_Horizontal, F.Cu at (157.2, 138.2)
- added J7: BWIPX-1-001E, bwlc1a:BWIPX-1-001E, F.Cu at (159.9, 117.9)
- added JP1: SolderJumper_3_Bridged12, Jumper:SolderJumper-3_P1.3mm_Bridged2Bar12_RoundedPad1.0x1.5mm, F.Cu at (148.5, 77.5)
- added L2: 9.5n, Inductor_SMD:L_0402_1005Metric, F.Cu at (123.2, 79.9)
- added L3: 6.1n, Inductor_SMD:L_0402_1005Metric, F.Cu at (123.2, 120.1)
- added L4: 3n, Inductor_SMD:L_0402_1005Metric, F.Cu at (122.7, 115.8)
- added L5: 4.3n, Inductor_SMD:L_0402_1005Metric, F.Cu at (123.2, 114.3)
- added L6: 1.3n, Inductor_SMD:L_0402_1005Metric, F.Cu at (122.7, 111.9)
- added Q7: DMG1012UW, Package_TO_SOT_SMD:SOT-323_SC-70, F.Cu at (154.4, 55.3)
- added Q8: AO3407A, Package_TO_SOT_SMD:SOT-23, F.Cu at (144.3, 157.1)
- added R15: 10K, Resistor_SMD:R_0402_1005Metric, F.Cu at (207.4, 71.5)
- added R33: 10K, Resistor_SMD:R_0402_1005Metric, F.Cu at (207.4, 79.4)
- added R34: 0, Resistor_SMD:R_0402_1005Metric, F.Cu at (164.8, 119.2)
- added R35: 0, Resistor_SMD:R_0402_1005Metric, F.Cu at (135.7, 71.1)
- added R36: 0, Resistor_SMD:R_0402_1005Metric, F.Cu at (138.4, 71.0)
- added R37: 0, Resistor_SMD:R_0402_1005Metric, F.Cu at (138.4, 73.0)
- added R38: 0, Resistor_SMD:R_0402_1005Metric, F.Cu at (122.7, 81.3)
- added TP10: +LIPO, TestPoint:TestPoint_Pad_D1.0mm, F.Cu at (143.4, 160.9)
- added TP11: USB_BOOT, TestPoint:TestPoint_Pad_D1.0mm, F.Cu at (149.0, 127.6)
- added TP12: UART_LOG_TXD, TestPoint:TestPoint_Pad_D1.0mm, F.Cu at (172.3, 120.8)
- added TP9: VBUS_IN, TestPoint:TestPoint_Pad_D1.0mm, F.Cu at (168.8, 169.7)
- added U10: TPS7A0328DBVR, Package_TO_SOT_SMD:SOT-23-5, F.Cu at (186.6, 52.8)
- added U11: TXB0106PWR, bwlc1a:TSSOP-16_L5.0-W4.4-P0.65-LS6.4-BL, F.Cu at (151.3, 86.1)
- added U12: TPS7A0333DBVR, Package_TO_SOT_SMD:SOT-23-5, F.Cu at (170.1, 52.7)
- C1: value 10u -> 10n; footprint Capacitor_SMD:C_0603_1608Metric -> Capacitor_SMD:C_0402_1005Metric
- C10: value 100n -> 22u; footprint Capacitor_SMD:C_0402_1005Metric -> Capacitor_SMD:C_0603_1608Metric
- C11: value 22u -> 10u
- C12, C2, C6: value 10u -> 100n; footprint Capacitor_SMD:C_0603_1608Metric -> Capacitor_SMD:C_0402_1005Metric
- C13: value 100n -> 33p; footprint Capacitor_SMD:C_0402_1005Metric -> Capacitor_SMD:C_0603_1608Metric
- C14: value 10u -> 33p
- C15: value 12p -> 100n
- C17: value 100n -> 12p
- C18: value 100u -> 330uF; footprint Capacitor_SMD:CP_Elec_6.3x5.4 -> Capacitor_Tantalum_SMD:CP_EIA-3528-15_AVX-H_Pad1.50x2.35mm_HandSolder
- C19: value 1u -> 330uF; footprint Capacitor_SMD:C_0603_1608Metric -> Capacitor_Tantalum_SMD:CP_EIA-3528-15_AVX-H_Pad1.50x2.35mm_HandSolder
- C20: value 330u -> 10u; footprint Capacitor_SMD:CP_Elec_6.3x5.4 -> Capacitor_SMD:C_0603_1608Metric
- C21: value 100n -> 10u; footprint Capacitor_SMD:C_0805_2012Metric -> Capacitor_SMD:C_0603_1608Metric
- C3: value 22p -> 10u; footprint Capacitor_SMD:C_0402_1005Metric -> Capacitor_SMD:C_0603_1608Metric
- C7: value 100n -> 10u; footprint Capacitor_SMD:C_0402_1005Metric -> Capacitor_SMD:C_0603_1608Metric
- F1: value 2A -> 0.75A; footprint Fuse:Fuse_1812_4532Metric -> Fuse:Fuse_0805_2012Metric
- J1: value JST-2PH -> USB_C_Receptacle_USB2.0; footprint Teapot:JST_PH_S2B-PH-SM4-TB_1x02-1MP_P2.00mm_Horizontal -> Connector_USB:USB_C_Receptacle_HRO_TYPE-C-31-M-12
- J2: value USB_C_Receptacle_USB2.0 -> JST-2PH; footprint Connector_USB:USB_C_Receptacle_HRO_TYPE-C-31-M-12 -> Teapot:JST_PH_S2B-PH-SM4-TB_1x02-1MP_P2.00mm_Horizontal
- J5: footprint SAMTEC_RSP-122811-02:SAMTEC_RSP-122811-02 -> bwlc1a:BWIPX-1-001E
- L1: value 2.2u -> 10n; footprint Inductor_SMD:L_1008_2520Metric -> Inductor_SMD:L_0402_1005Metric
- Q2: value S8050 -> PMV32UP
- Q5, Q6: value S8050 -> PMBT3904
- R11, R8, R9: value 4.7k -> 10K
- R12: value 47k -> 1M; footprint Resistor_SMD:R_0402_1005Metric -> Resistor_SMD:R_0603_1608Metric
- R13: footprint Resistor_SMD:R_0402_1005Metric -> Resistor_SMD:R_0603_1608Metric
- R14: value 10k -> 4.7k
- R18: value 100k -> 4.7k
- R19: value 470 -> 5K1
- R21: value 47k -> 22
- R28: value 10k -> 0
- R3: value 453k -> 1k
- R5: value 1k -> 0
- R6: value 10k -> DNP; footprint Resistor_SMD:R_0402_1005Metric -> Resistor_SMD:R_0603_1608Metric
- R7: value 100k -> 10k
- SW1: value EN_ESP -> RESET
- TP1: value VBUS -> USB_DP; footprint TestPoint:TestPoint_Pad_D1.5mm -> TestPoint:TestPoint_Pad_D1.0mm
- TP2: value USB_DP -> USB_DM; footprint TestPoint:TestPoint_Pad_D1.5mm -> TestPoint:TestPoint_Pad_D1.0mm
- TP3: value USB_DM -> VBUS; footprint TestPoint:TestPoint_Pad_D1.5mm -> TestPoint:TestPoint_Pad_D1.0mm
- TP4: value GND -> UART_LOG_RXD; footprint TestPoint:TestPoint_Pad_D1.5mm -> TestPoint:TestPoint_Pad_D1.0mm
- TP5: value BOOT -> RESET
- TP6: value RESET -> BOOT
- U1: value MCP73831-2-OT -> USBLC6-2SC6; footprint Package_TO_SOT_SMD:SOT-23-5 -> Package_TO_SOT_SMD:SOT-23-6
- U2: value USBLC6-2SC6 -> MCP73831-2-OT; footprint Package_TO_SOT_SMD:SOT-23-6 -> Package_TO_SOT_SMD:SOT-23-5
- U3: value TPS62290DRVR -> RT9080-33GJ5; footprint TPS62290DRVR:SON65P200X200X80-7N -> Package_TO_SOT_SMD:SOT-23-5_HandSoldering
- U4: value MAX17048G+ -> LSM6DSOTR; footprint Package_DFN_QFN:DFN-8-1EP_2x2mm_P0.5mm_EP0.7x1.3mm -> Package_LGA:LGA-14_3x2.5mm_P0.5mm_LayoutBorder3x4y
- U5: value LSM6DS3 -> MAX17048G+; footprint Package_LGA:LGA-14_3x2.5mm_P0.5mm_LayoutBorder3x4y -> Package_DFN_QFN:DFN-8-1EP_2x2mm_P0.5mm_EP0.7x1.3mm
- U7: value L86-M33 -> L76L-M33; footprint Teapot:XCVR_L86-M33 -> bwlc1a:L76L-M33
- U8: value MIC29302WU -> TPS22917DBVR; footprint Package_TO_SOT_SMD:TO-263-5_TabPin3 -> Package_TO_SOT_SMD:SOT-23-6
- moved TP8 103.8 mm to (201.5, 81.2)
- moved TP7 103.3 mm to (201.5, 78.1)
- moved C7 99.1 mm to (205.0, 87.1), turned to 0 degrees
- moved R8 92.2 mm to (204.5, 73.5), turned to 0 degrees
- moved TP5 92.1 mm to (192.7, 76.5)
- moved C6 91.3 mm to (193.1, 83.4), turned to 0 degrees
- moved TP6 91.1 mm to (193.1, 90.1)
- moved R9 90.6 mm to (204.5, 75.5), turned to 0 degrees
- moved R11 90.0 mm to (204.5, 77.5), turned to 0 degrees
- moved Y1 85.7 mm to (205.5, 84.1), turned to 0 degrees
- moved J3 83.4 mm to (199.5, 95.6), turned to 0 degrees
- moved C2 82.7 mm to (168.7, 167.2), turned to 0 degrees
- moved C1 81.3 mm to (168.7, 165.2), turned to 0 degrees
- moved C15 80.3 mm to (201.6, 85.4), turned to 0 degrees
- moved U8 79.8 mm to (140.7, 50.0), turned to 0 degrees
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Connections:
- net A7670_BOOT renamed /Cellular/USB_BOOT
- net A7670_PWR renamed /Cellular/CELL_PWRKEY
- net A7670_RST renamed /Cellular/CELL_RESET
- net A7670_STATUS renamed /Cellular/CELL_STATUS
- net A7670_UART_RX renamed /Cellular/RXD
- net A7670_UART_TX renamed /Cellular/TXD
- net JTAG_TCK renamed /Main Controller/JTAG_TCK
- net JTAG_TDI renamed /Main Controller/JTAG_TDI
- net JTAG_TDO renamed /Main Controller/JTAG_TDO
- net JTAG_TMS renamed /Main Controller/JTAG_TMS
- net PWRKEY renamed /Cellular/PWRKEY
- net RESET renamed /Cellular/RESET
- net USIM_CLK renamed /Cellular/USIM_CLK
- net USIM_DATA renamed /Cellular/USIM_DATA
- net USIM_RST renamed /Cellular/USIM_RST
- net USIM_VDD renamed /Cellular/USIM_VDD
- C1 pad 1: VBUS -> Net-(C1-Pad1)
- C10 pad 1: IMU_VDD -> +3V3
- C11 pad 1: IMU_VDD -> +3V3
- C12 pad 1: IMU_VDD -> +BATT
- C13 pad 1: VDD_BAT -> /GNSS_3V3
- C14 pad 1: VDD_BAT -> Net-(JP1-C)
- C15 pad 1: ESP_32K_P -> +3V3
- C16 pad 1: GND -> Net-(C16-Pad1)
- C16 pad 2: ESP_32K_N -> GND
- C17 pad 1: ESP_EN -> GND
- C17 pad 2: GND -> Net-(U6-GPIO16/U0CTS/ADC2_CH5/XTAL_32K_N)
- C18 pad 1: Net-(JP2-A) -> /Cellular/CELL_BATT
- C19 pad 1: Net-(JP2-A) -> /Cellular/CELL_BATT
- C2 pad 1: +BATT -> Net-(C2-Pad1)
- C20 pad 1: VDD_BAT -> +3V3
- C21 pad 1: VDD_BAT -> +BATT
- C3 pad 1: IMU_VDD -> VBUS
- C3 pad 2: /TPS_FB -> GND
- C33 pad 1: VDD_1V8 -> /Cellular/VDD_1V8
- C34 pad 1: IMU_VDD -> +3V3
- C34 pad 2: A7670_TX -> /Cellular/CELL_TXD
- C35 pad 1: Net-(U9-RF_ANT) -> Net-(C35-Pad1)
- C37 pad 2: VDD_1V8 -> /Cellular/VDD_1V8
- C38 pad 1: VDD_1V8 -> /Cellular/VDD_1V8
- C4 pad 1: IMU_VDD -> +BATT
- C5 pad 1: TPS_VIN -> +BATT
- C6 pad 1: IMU_VDD -> /Main Controller/CHIP_EN
- C7 pad 1: IMU_VDD -> +3V3
- C8 pad 1: +BATT -> +3V3
- C9 pad 1: IMU_VDD -> +3V3
- D5 pad 2: VDD_BAT -> /Cellular/CELL_BATT
- F1 pad 1: +BATT -> Net-(C2-Pad1)
- F1 pad 2: Net-(JP2-A) -> VBUS
- FB1 pad 2: VDD_BAT -> /Cellular/CELL_BATT
- J3 pad 1: IMU_VDD -> +3V3
- J3 pad 10: ESP_EN -> /Main Controller/CHIP_EN
- J5 pad 1: Net-(D6-A2) -> Net-(J5-SIG)
- L1 pad 1: IMU_VDD -> Net-(L1-Pad1)
- L1 pad 2: Net-(U3-SW) -> Net-(E1-Pad4)
- Q2 pad 1: Net-(Q2-C) -> Net-(Q2-G)
- Q2 pad 2: Net-(Q2-B) -> +BATT
- Q2 pad 3: GND -> /GNSS_VBCKP
- Q3 pad 1: A7670_TX -> /Cellular/CELL_TXD
- Q4 pad 3: A7670_RX -> /Cellular/CELL_RXD
- R1 pad 1: Net-(J2-CC1) -> Net-(J1-CC1)
- R10 pad 2: Net-(U5-SDO/SA0) -> Net-(U4-SDO/SA0)
- R11 pad 1: GPS_RST -> GND
- R11 pad 2: Net-(Q2-B) -> /Main Controller/GNSS_EN
- R12 pad 1: Net-(Q2-B) -> +BATT
- R12 pad 2: GND -> Net-(Q2-G)
- R13 pad 1: GND -> /Main Controller/GNSS_VBCKP_EN
- R13 pad 2: GPS_FORCE_ON -> GND
- R14 pad 1: IMU_VDD -> +3V3
- R14 pad 2: ESP_EN -> /Main Controller/SCL
- R18 pad 1: VDD_BAT -> +3V3
- R18 pad 2: Net-(U8-ADJ) -> /Main Controller/SDA
- R19 pad 1: VDD_BAT -> /Main Controller/BOOT_MODE0
- R19 pad 2: GND -> +3V3
- R2 pad 1: Net-(J2-CC2) -> Net-(J1-CC2)
- R21 pad 1: Net-(U8-ADJ) -> Net-(U6-GPIO15/U0RTS/ADC2_CH4/XTAL_32K_P)
- R21 pad 2: GND -> Net-(C16-Pad1)
- R22 pad 2: VDD_1V8 -> /Cellular/VDD_1V8
- R23 pad 1: A7670_TX -> /Cellular/CELL_TXD
- R23 pad 2: IMU_VDD -> +3V3
- R24 pad 1: Net-(U9-RF_ANT) -> /Antenna/GNSS_ANT
- R24 pad 2: Net-(C36-Pad1) -> Net-(C48-Pad1)
- R25 pad 1: Net-(C36-Pad1) -> Net-(C35-Pad1)
- R25 pad 2: Net-(D6-A2) -> Net-(C36-Pad1)
- R26 pad 1: VDD_1V8 -> /Cellular/VDD_1V8
- R27 pad 1: VDD_1V8 -> /Cellular/VDD_1V8
- R28 pad 1: VDD_1V8 -> Net-(C36-Pad1)
- R3 pad 1: /TPS_FB -> Net-(U2-PROG)
- R3 pad 2: IMU_VDD -> GND
- R4 pad 1: Net-(U1-STAT) -> Net-(U2-STAT)
- R5 pad 1: Net-(U1-PROG) -> /Antenna/CELL_ANT
- R5 pad 2: GND -> Net-(C35-Pad1)
- R6 pad 1: GND -> Net-(U8-QOD)
- R6 pad 2: VBUS -> /Cellular/CELL_BATT
- R7 pad 1: GND -> +3V3
- R7 pad 2: /TPS_FB -> /Main Controller/CHIP_EN
- R8 pad 1: IMU_VDD -> GND
- R8 pad 2: IMU_SCL -> /GNSS/GNSS_FO
- R9 pad 1: IMU_VDD -> GND
- R9 pad 2: IMU_SDA -> /Main Controller/CELL_EN
- SW1 pad 2: ESP_EN -> /Main Controller/CHIP_EN
- SW2 pad 1: ESP_BOOT -> /Main Controller/BOOT_MODE0
- TP1 pad 1: Net-(U9-VBUS) -> /Cellular/USB_DP
- TP2 pad 1: Net-(U9-USB_DP) -> /Cellular/USB_DM
- TP3 pad 1: Net-(U9-USB_DM) -> /Cellular/VBUS
- TP4 pad 1: GND -> /Cellular/UART_LOG_RXD
- TP5 pad 1: ESP_BOOT -> /Main Controller/CHIP_EN
- TP6 pad 1: ESP_EN -> /Main Controller/BOOT_MODE0
- U1 pad 1: Net-(U1-STAT) -> /USB and Charger/D_IN+
- U1 pad 3: +BATT -> /USB and Charger/D_IN-
- U1 pad 4: VBUS -> /Main Controller/USB_D-
- U1 pad 5: Net-(U1-PROG) -> VBUS
- U2 pad 1: USB_D+ -> Net-(U2-STAT)
- U2 pad 3: USB_D- -> +BATT
- U2 pad 4: USB_D- -> VBUS
- U2 pad 5: VBUS -> Net-(U2-PROG)
- U3 pad 1: Net-(U3-SW) -> +BATT
- U3 pad 3: /TPS_FB -> +BATT
- U3 pad 4: TPS_VIN -> unconnected-(U3-NC/SNS-Pad4)
- U3 pad 5: TPS_VIN -> +3V3
- U4 pad 1: GND -> Net-(U4-SDO/SA0)
- U4 pad 2: +BATT -> GND
- U4 pad 3: +BATT -> GND
- U4 pad 4: GND -> /Main Controller/IMU_INT
- U4 pad 5: MAX17048_INT -> +3V3
- U4 pad 7: IMU_SCL -> GND
- U4 pad 8: IMU_SDA -> +3V3
- U4 pad 9: GND -> unconnected-(U4-INT2-Pad9)
- U5 pad 1: Net-(U5-SDO/SA0) -> GND
- U5 pad 2: GND -> +BATT
- U5 pad 3: GND -> +BATT
- U5 pad 4: IMU_INT -> GND
- U5 pad 5: IMU_VDD -> /Main Controller/FG_INT
- U5 pad 7: GND -> /Main Controller/SCL
- U5 pad 8: IMU_VDD -> /Main Controller/SDA
- U5 pad 9: unconnected-(U5-INT2-Pad9) -> GND
- U6 pad 16: IMU_SCL -> /Main Controller/SCL
- U6 pad 17: IMU_SDA -> /Main Controller/SDA
- U6 pad 19: ESP_32K_P -> Net-(U6-GPIO15/U0RTS/ADC2_CH4/XTAL_32K_P)
- U6 pad 20: ESP_32K_N -> Net-(U6-GPIO16/U0CTS/ADC2_CH5/XTAL_32K_N)
- U6 pad 21: unconnected-(U6-GPIO17/U1TXD/ADC2_CH6-Pad21) -> /Cellular/CELL_RXD
- U6 pad 22: unconnected-(U6-GPIO18/U1RXD/ADC2_CH7/CLK_OUT3-Pad22) -> /Cellular/CELL_TXD
- U6 pad 23: USB_D- -> /Main Controller/USB_D-
- U6 pad 24: USB_D+ -> /Main Controller/USB_D+
- U6 pad 25: MAX17048_INT -> /Main Controller/FG_INT
- U6 pad 26: unconnected-(U6-GPIO26-Pad26) -> /Main Controller/GNSS_VBCKP_EN
- U6 pad 3: IMU_VDD -> +3V3
- U6 pad 30: EN_MIC29302 -> /Main Controller/CELL_EN
- U6 pad 31: GPS_RX -> /GNSS/GNSS_RXD
- U6 pad 32: GPS_TX -> /GNSS/GNSS_TXD
- U6 pad 33: GPS_FORCE_ON -> /GNSS/GNSS_FO
- U6 pad 34: GPS_RST -> /GNSS/GNSS_RESET
- U6 pad 4: ESP_BOOT -> /Main Controller/BOOT_MODE0
- U6 pad 41: unconnected-(U6-GPIO45-Pad41) -> /GNSS/GNSS_SDBY
- U6 pad 44: unconnected-(U6-GPIO46-Pad44) -> /Main Controller/BOOT_MODE1
- U6 pad 45: ESP_EN -> /Main Controller/ESP_EN
- U6 pad 5: unconnected-(U6-GPIO1/TOUCH1/ADC1_CH0-Pad5) -> /Main Controller/GNSS_EN
- U6 pad 6: IMU_INT -> /Main Controller/IMU_INT
- U7 pad 1: GPS_RX -> GND
- U7 pad 10: Net-(Q2-C) -> GND
- U7 pad 11: unconnected-(U7-EX_ANT-Pad11) -> /Antenna/GNSS_ANT
- U7 pad 2: GPS_TX -> /GNSS/TXD
- U7 pad 3: GND -> /GNSS/RXD
- U7 pad 4: VDD_BAT -> unconnected-(U7-1PPS-Pad4)
- U7 pad 5: VDD_BAT -> /GNSS/STANDBY
- U7 pad 6: unconnected-(U7-1PPS-Pad6) -> Net-(JP1-C)
- U7 pad 7: GPS_FORCE_ON -> (no net)
- U7 pad 8: unconnected-(U7-AADET_N-Pad8) -> /GNSS_3V3
- U7 pad 9: (no net) -> /GNSS/RESET
- U8 pad 1: Net-(JP2-C) -> +BATT
- U8 pad 2: Net-(JP2-A) -> GND
- U8 pad 3: GND -> /Main Controller/CELL_EN
- U8 pad 4: VDD_BAT -> Net-(U8-CT)
- U8 pad 5: Net-(U8-ADJ) -> Net-(U8-QOD)
- U9 pad 15: VDD_1V8 -> /Cellular/VDD_1V8
- U9 pad 22: unconnected-(U9-UART_LOG_RX-Pad22) -> /Cellular/UART_LOG_RXD
- U9 pad 23: unconnected-(U9-UART_LOG_TX-Pad23) -> /Cellular/UART_LOG_TXD
- U9 pad 24: Net-(U9-VBUS) -> /Cellular/VBUS
- U9 pad 27: Net-(U9-USB_DP) -> /Cellular/USB_DP
- U9 pad 28: Net-(U9-USB_DM) -> /Cellular/USB_DM
- U9 pad 60: Net-(U9-RF_ANT) -> /Antenna/CELL_ANT
- Y1 pad 1: ESP_32K_N -> Net-(U6-GPIO16/U0CTS/ADC2_CH5/XTAL_32K_N)
- Y1 pad 2: ESP_32K_P -> Net-(C16-Pad1)
Routing:
- net IMU_VDD: track 106.1 -> 0.00 mm, vias 6 -> 0
- net VBUS: track 95.5 -> 0.00 mm, vias 6 -> 0
- net IMU_SDA: track 93.1 -> 0.00 mm, vias 3 -> 0
- net IMU_SCL: track 92.9 -> 0.00 mm, vias 3 -> 0
- net MAX17048_INT: track 75.0 -> 0.00 mm, vias 2 -> 0
- net EN_MIC29302: track 74.1 -> 0.00 mm, vias 2 -> 0
- net +BATT: track 74.1 -> 0.00 mm, vias 7 -> 0
- net GND: track 55.7 -> 0.00 mm, vias 385 -> 0
- net ESP_BOOT: track 53.8 -> 0.00 mm, vias 2 -> 0
- net VDD_BAT: track 51.3 -> 0.00 mm, vias 12 -> 0
- net /Cellular/CELL_STATUS: track 47.7 -> 0.00 mm, vias 2 -> 0
- net GPS_RST: track 39.6 -> 0.00 mm, vias 2 -> 0
- net A7670_TX: track 39.6 -> 0.00 mm, vias 2 -> 0
- net ESP_EN: track 37.5 -> 0.00 mm
- net /Cellular/CELL_PWRKEY: track 36.9 -> 0.00 mm, vias 2 -> 0
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- removed copper zone on B.Cu, net +BATT
- removed copper zone on F.Cu, net +BATT
- removed copper zone on B.Cu, net GND
- removed copper zone on F.Cu, net GND
- removed copper zone on In1.Cu, net GND
- removed copper zone on In2.Cu, net GND
- removed copper zone on F.Cu, net IMU_VDD
- removed copper zone on F.Cu, net Net-(C27-Pad1)
- removed copper zone on F.Cu, net Net-(JP2-A)
- removed copper zone on F.Cu, net Net-(U3-SW)
- removed copper zone on F.Cu, net VBUS
- removed copper zone on F.Cu, net VDD_1V8
- removed copper zone on B.Cu, net VDD_BAT
- removed copper zone on F.Cu, net VDD_BAT
Other:
- outline, holes or cut-outs redrawn
- board text removed: "+ BATT -"
- board text removed: "3V3 POWER SUPPLY"
- board text removed: "ANT"
- board text removed: "B"
- board text removed: "BWLC1A"
- board text removed: "CELL BOOT"
- board text removed: "CELL USB"
- board text removed: "DEBUG"
- board text removed: "F"
- board text removed: "GPS & CELL PWR SUPPLY"
- board text removed: "IMU"
- board text removed: "PWR SEL"
- board text removed: "R"
- board text removed: "Rev. 1"
- board text removed: "Teapot Laboratories"
- board text removed: "VBUS D+ D- GND"
- board text removed: "X X GND GND VDD - - - - - - - - - RST TDI TDO TCK TMS"

Commit message: PCB Layout Update
Parts:
- added D10: ESD5651N, Capacitor_SMD:C_0402_1005Metric, F.Cu at (183.5, 84.8)
- added D11: ESD5651N, Capacitor_SMD:C_0402_1005Metric, F.Cu at (183.5, 81.0)
- added D2: ESD5651N, Capacitor_SMD:C_0402_1005Metric, F.Cu at (144.0, 94.2)
- added D3: ESD5651N, Capacitor_SMD:C_0402_1005Metric, F.Cu at (141.5, 76.8)
- added D6: ESD5651N, Capacitor_SMD:C_0402_1005Metric, F.Cu at (178.7, 102.9)
- added D9: ESDA6V1W5, Package_TO_SOT_SMD:SOT-353_SC-70-5, F.Cu at (184.0, 88.5)
- added E1: NN03-320, bwlc1a:NN03-320, F.Cu at (110.2, 75.2)
- added G***: LOGO, Teapot:TeapotLogo, F.Cu at (184.1, 119.3)
- added R39: 0, Resistor_SMD:R_0402_1005Metric, F.Cu at (135.8, 92.6)
- added R40: 0, Resistor_SMD:R_0402_1005Metric, F.Cu at (133.3, 76.3)
- J2, J3, TP5, TP6, TP7, TP8: moved to B.Cu
- U3: footprint Package_TO_SOT_SMD:SOT-23-5_HandSoldering -> Package_TO_SOT_SMD:SOT-23-5
- moved TP9 67.3 mm to (180.7, 103.5), turned to -90 degrees
- moved R2 66.7 mm to (178.7, 104.0), turned to 180 degrees
- moved C21 64.6 mm to (159.2, 108.1)
- moved FB2 63.1 mm to (180.7, 110.6), turned to -90 degrees
- moved C33 61.4 mm to (126.5, 109.3), turned to 180 degrees
- moved J2 61.2 mm to (182.5, 119.9), turned to 90 degrees
- moved C34 60.5 mm to (128.7, 104.2)
- moved R23 59.9 mm to (126.5, 104.2)
- moved R1 59.8 mm to (178.7, 109.3), turned to 180 degrees
- moved C37 59.6 mm to (128.7, 110.6), turned to 180 degrees
- moved J1 58.6 mm to (187.2, 106.8), turned to 90 degrees
- moved U8 58.2 mm to (159.4, 105.1), turned to 90 degrees
- moved C22 58.1 mm to (163.1, 106.3), turned to 90 degrees
- moved R27 58.0 mm to (126.5, 110.6), turned to 180 degrees
- moved C23 57.0 mm to (159.2, 102.1)
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Connections:
- R28 pad 2: Net-(J7-SIG) -> Net-(R28-Pad2)
- R34 pad 1: Net-(J7-SIG) -> Net-(R28-Pad2)
- R36 pad 2: Net-(J5-SIG) -> Net-(R36-Pad2)
- R37 pad 1: Net-(J5-SIG) -> Net-(R36-Pad2)
- U1 pad 1: /USB and Charger/D_IN+ -> /USB and Charger/D_IN-
- U1 pad 3: /USB and Charger/D_IN- -> /USB and Charger/D_IN+
- U1 pad 4: /Main Controller/USB_D- -> /Main Controller/USB_D+
- U1 pad 6: /Main Controller/USB_D+ -> /Main Controller/USB_D-
- U6 pad 10: unconnected-(U6-GPIO6/TOUCH6/ADC1_CH5-Pad10) -> /GNSS/GNSS_RXD
- U6 pad 11: unconnected-(U6-GPIO7/TOUCH7/ADC1_CH6-Pad11) -> /GNSS/GNSS_TXD
- U6 pad 12: unconnected-(U6-GPIO8/TOUCH8/ADC1_CH7/SUBSPICS1-Pad12) -> /Main Controller/GNSS_VBCKP_EN
- U6 pad 13: unconnected-(U6-GPIO9/TOUCH9/ADC1_CH8/FSPIHD/SUBSPIHD-Pad13) -> /Cellular/CELL_PWRKEY
- U6 pad 14: unconnected-(U6-GPIO10/TOUCH10/ADC1_CH9/FSPICS0/FSPIIO4/SUBSPICS0-Pad14) -> /Cellular/CELL_TXD
- U6 pad 15: unconnected-(U6-GPIO11/TOUCH11/ADC2_CH0/FSPID/FSPIIO5/SUBSPID-Pad15) -> /Cellular/CELL_RXD
- U6 pad 16: /Main Controller/SCL -> /Cellular/CELL_RESET
- U6 pad 17: /Main Controller/SDA -> /Main Controller/IMU_INT
- U6 pad 18: unconnected-(U6-GPIO14/TOUCH14/ADC2_CH3/FSPIWP/FSPIDQS/SUBSPIWP-Pad18) -> /Main Controller/CELL_EN
- U6 pad 21: /Cellular/CELL_RXD -> /Cellular/CELL_STATUS
- U6 pad 22: /Cellular/CELL_TXD -> /Main Controller/FG_INT
- U6 pad 25: /Main Controller/FG_INT -> unconnected-(U6-GPIO21-Pad25)
- U6 pad 26: /Main Controller/GNSS_VBCKP_EN -> unconnected-(U6-GPIO26-Pad26)
- U6 pad 27: /Cellular/CELL_PWRKEY -> unconnected-(U6-GPIO47/SPICLK_P/SUBSPICLK_P_DIFF-Pad27)
- U6 pad 28: /Cellular/CELL_STATUS -> unconnected-(U6-SPIIO4/GPIO33/FSPIHD/SUBSPIHD-Pad28)
- U6 pad 29: /Cellular/CELL_RESET -> unconnected-(U6-SPIIO5/GPIO34/FSPICS0/SUBSPICS0-Pad29)
- U6 pad 30: /Main Controller/CELL_EN -> unconnected-(U6-GPIO48/SPICLK_N/SUBSPICLK_N_DIFF-Pad30)
- U6 pad 31: /GNSS/GNSS_RXD -> unconnected-(U6-SPIIO6/GPIO35/FSPID/SUBSPID-Pad31)
- U6 pad 32: /GNSS/GNSS_TXD -> /Main Controller/SCL
- U6 pad 33: /GNSS/GNSS_FO -> /Main Controller/SDA
- U6 pad 34: /GNSS/GNSS_RESET -> unconnected-(U6-GPIO38/FSPIWP/SUBSPIWP-Pad34)
- U6 pad 41: /GNSS/GNSS_SDBY -> unconnected-(U6-GPIO45-Pad41)
- U6 pad 45: /Main Controller/ESP_EN -> /Main Controller/CHIP_EN
- U6 pad 5: /Main Controller/GNSS_EN -> /GNSS/GNSS_RESET
- U6 pad 6: /Main Controller/IMU_INT -> /GNSS/GNSS_SDBY
- U6 pad 8: unconnected-(U6-GPIO4/TOUCH4/ADC1_CH3-Pad8) -> /GNSS/GNSS_FO
- U6 pad 9: unconnected-(U6-GPIO5/TOUCH5/ADC1_CH4-Pad9) -> /Main Controller/GNSS_EN
Routing:
- net +3V3: track 0.00 -> 124.1 mm, vias 0 -> 13
- net GND: track 0.00 -> 78.1 mm, vias 0 -> 477
- net +BATT: track 0.00 -> 69.8 mm, vias 0 -> 11
- net /Cellular/CELL_RESET: track 0.00 -> 64.8 mm, vias 0 -> 2
- net /Cellular/CELL_RXD: track 0.00 -> 55.8 mm, vias 0 -> 2
- net /Cellular/CELL_TXD: track 0.00 -> 55.3 mm, vias 0 -> 2
- net /Main Controller/GNSS_VBCKP_EN: track 0.00 -> 51.1 mm, vias 0 -> 2
- net /Main Controller/SCL: track 0.00 -> 50.8 mm, vias 0 -> 4
- net /Main Controller/SDA: track 0.00 -> 50.0 mm, vias 0 -> 4
- net /Cellular/CELL_PWRKEY: track 0.00 -> 47.7 mm, vias 0 -> 2
- net /Cellular/CELL_STATUS: track 0.00 -> 38.4 mm, vias 0 -> 2
- net /Main Controller/GNSS_EN: track 0.00 -> 33.4 mm, vias 0 -> 3
- net /GNSS/GNSS_TXD: track 0.00 -> 28.7 mm, vias 0 -> 2
- net /GNSS/GNSS_RESET: track 0.00 -> 28.1 mm, vias 0 -> 3
- net /GNSS/GNSS_SDBY: track 0.00 -> 27.0 mm, vias 0 -> 3
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- added copper zone on B.Cu, net +3V3
- added copper zone on F.Cu, net +3V3
- added copper zone on B.Cu, net +BATT
- added copper zone on F.Cu, net +BATT
- added copper zone on F.Cu, net /Cellular/CELL_BATT
- added copper zone on F.Cu, net /GNSS_3V3
- added copper zone on B.Cu, net GND
- added copper zone on F.Cu, net GND
- added copper zone on In1.Cu, net GND
- added copper zone on In2.Cu, net GND
- added copper zone on F.Cu, net Net-(C27-Pad1)
- added copper zone on B.Cu, net Net-(J2-Pin_1)
- added copper zone on F.Cu, net Net-(J2-Pin_1)
- added copper zone on F.Cu, net Net-(JP1-C)
Other:
- board size 80 x 50 mm -> 80.5 x 50 mm
- board text added: "+ BAT -"
- board text added: "B"
- board text added: "BATT&CHRG"
- board text added: "BOOT"
- board text added: "BWLC1A"
- board text added: "CELLULAR"
- board text added: "D+"
- board text added: "D-"
- board text added: "ESP32-S3"
- board text added: "GNSS"
- board text added: "IMU"
- board text added: "JTAG"
- board text added: "QWIIC"
- board text added: "R"
- board text added: "REV.B"
- board text added: "RST"
- board text added: "RX"
- board text added: "TX"
- board text added: "USB"
- board text added: "VBAT"
- board text added: "VBUS"

Commit message: PCB Layout Update
Parts:
- added D12: Yellow, LED_SMD:LED_0603_1608Metric, F.Cu at (180.9, 98.0)
- added D13: Green, LED_SMD:LED_0603_1608Metric, F.Cu at (178.8, 98.0)
- added R41: 1k, Resistor_SMD:R_0402_1005Metric, F.Cu at (180.9, 100.4)
- added R42: 1k, Resistor_SMD:R_0402_1005Metric, F.Cu at (178.8, 100.4)
- added TP13: GPIO35, TestPoint:TestPoint_Pad_D1.0mm, B.Cu at (179.1, 97.7)
- added TP14: GPIO34, TestPoint:TestPoint_Pad_D1.0mm, B.Cu at (176.7, 97.7)
- added TP15: GPIO33, TestPoint:TestPoint_Pad_D1.0mm, B.Cu at (174.4, 97.7)
- added TP16: GPIO21, TestPoint:TestPoint_Pad_D1.0mm, B.Cu at (172.0, 97.7)
- added TP17: GPIO38, TestPoint:TestPoint_Pad_D1.0mm, B.Cu at (181.6, 97.7)
- added TP18: GPIO45, TestPoint:TestPoint_Pad_D1.0mm, B.Cu at (185.9, 85.7)
- added TP19: GPIO46, TestPoint:TestPoint_Pad_D1.0mm, B.Cu at (185.9, 83.4)
- added TP20: GPIO03, TestPoint:TestPoint_Pad_D1.0mm, B.Cu at (168.9, 87.3)
- moved G*** 0.57 mm to (183.8, 119.8)
- moved TP5 0.20 mm to (183.5, 82.0)
- moved TP6 0.18 mm to (183.4, 84.4)
Connections:
- U6 pad 25: unconnected-(U6-GPIO21-Pad25) -> Net-(U6-GPIO21)
- U6 pad 27: unconnected-(U6-GPIO47/SPICLK_P/SUBSPICLK_P_DIFF-Pad27) -> Net-(D13-A)
- U6 pad 28: unconnected-(U6-SPIIO4/GPIO33/FSPIHD/SUBSPIHD-Pad28) -> Net-(U6-SPIIO4/GPIO33/FSPIHD/SUBSPIHD)
- U6 pad 29: unconnected-(U6-SPIIO5/GPIO34/FSPICS0/SUBSPICS0-Pad29) -> Net-(U6-SPIIO5/GPIO34/FSPICS0/SUBSPICS0)
- U6 pad 30: unconnected-(U6-GPIO48/SPICLK_N/SUBSPICLK_N_DIFF-Pad30) -> Net-(D12-A)
- U6 pad 31: unconnected-(U6-SPIIO6/GPIO35/FSPID/SUBSPID-Pad31) -> Net-(U6-SPIIO6/GPIO35/FSPID/SUBSPID)
- U6 pad 34: unconnected-(U6-GPIO38/FSPIWP/SUBSPIWP-Pad34) -> Net-(U6-GPIO38/FSPIWP/SUBSPIWP)
- U6 pad 41: unconnected-(U6-GPIO45-Pad41) -> Net-(U6-GPIO45)
- U6 pad 44: /Main Controller/BOOT_MODE1 -> Net-(U6-GPIO46)
- U6 pad 7: unconnected-(U6-GPIO3/TOUCH3/ADC1_CH2-Pad7) -> Net-(U6-GPIO3/TOUCH3/ADC1_CH2)
Routing:
- net Net-(U6-GPIO38/FSPIWP/SUBSPIWP): track 0.00 -> 7.82 mm, vias 0 -> 1
- net Net-(U6-GPIO21): track 0.00 -> 7.08 mm, vias 0 -> 1
- net Net-(U6-SPIIO4/GPIO33/FSPIHD/SUBSPIHD): track 0.00 -> 6.75 mm, vias 0 -> 1
- net Net-(U6-SPIIO5/GPIO34/FSPICS0/SUBSPICS0): track 0.00 -> 5.86 mm, vias 0 -> 1
- net Net-(U6-SPIIO6/GPIO35/FSPID/SUBSPID): track 0.00 -> 5.14 mm, vias 0 -> 1
- net Net-(U6-GPIO46): track 0.00 -> 4.80 mm, vias 0 -> 1
- net Net-(U6-GPIO45): track 0.00 -> 4.76 mm, vias 0 -> 1
- net GND: track 78.1 -> 81.7 mm, vias 477 -> 476
- net Net-(D13-A): track 0.00 -> 2.52 mm
- net Net-(D12-A): track 0.00 -> 2.36 mm
- net Net-(D13-K): track 0.00 -> 1.84 mm
- net Net-(D12-K): track 0.00 -> 1.84 mm
- net Net-(U6-GPIO3/TOUCH3/ADC1_CH2): track 0.00 -> 1.62 mm, vias 0 -> 1
- net +3V3: track 124.1 -> 123.4 mm
- net /Main Controller/CHIP_EN: track 16.5 -> 17.2 mm
Other:
- board text added: "03"
- board text added: "21"
- board text added: "33"
- board text added: "34"
- board text added: "35"
- board text added: "38"
- board text added: "45"
- board text added: "46"
- board text added: "A"
- board text added: "CHRG"
- board text removed: "BOOT"
- board text removed: "QWIIC"
- board text removed: "RST"
