File: hardware/kicad/bwlc1a.kicad_pcb (KiCad board)
At the start: 4 copper layers, 80.5 x 50 mm, 177 parts, among them J1 USB_C_Receptacle_USB2.0, J2 JST-2PH, J3 JTAG_10PIN, J4 SMN-304, J5 BWIPX-1-001E, J6 Qwiic, J7 BWIPX-1-001E, Q2 PMV32UP, Q3 S8050, Q4 S8050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

Commit message: change teapotlabs logo library
Parts:
- G***: footprint Teapot:TeapotLogo -> bwlc1a:TeapotLogo
Changed lines of the file:
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@@
 		)
 	)
-	(footprint "Teapot:TeapotLogo"
+	(footprint "bwlc1a:TeapotLogo"
 		(layer "F.Cu")
 		(at 183.837 119.126)

Commit message: update schematics bom
Parts:
- D1: value Orange -> E6C0603SEAC1UDA
- D6: footprint Capacitor_SMD:C_0402_1005Metric -> Diode_SMD:D_SOD-882
- F1: value 0.75A -> SMD0805P075TF
- J2: footprint Teapot:JST_PH_S2B-PH-SM4-TB_1x02-1MP_P2.00mm_Horizontal -> bwlc1a:JST_PH_S2B-PH-SM4-TB_1x02-1MP_P2.00mm_Horizontal
- R3: value 1k -> 2k

Commit message: update bill of materials
Parts:
- C26, C45: value 10u -> 1u
- C35, C36, C48, C49: value TBD -> DNP
- J2: value JST-2PH -> S2B-PH-SM4-TB(LF)(SN)
- L1, L2, L5: footprint Inductor_SMD:L_0402_1005Metric -> Inductor_SMD:L_0603_1608Metric
- R38: footprint Resistor_SMD:R_0402_1005Metric -> Resistor_SMD:R_0603_1608Metric
- moved R37 2.12 mm to (130.4, 75.7)
- moved R40 2.12 mm to (131.9, 76.2)
- moved R38 1.59 mm to (128.0, 75.7)
- moved L2 0.83 mm to (125.7, 76.5)
- moved L5 0.59 mm to (123.7, 114.1)
- moved L6 0.54 mm to (122.7, 111.5)
- moved C53 0.54 mm to (123.2, 112.9)
- moved J5 0.51 mm to (125.5, 80.5)
- moved Q7 0.20 mm to (125.3, 84.4)
Routing:
- net Net-(R36-Pad2): track 5.41 -> 1.89 mm
- net Net-(L1-Pad1): track 1.90 -> 0.00 mm
- net GND: track 74.4 -> 72.8 mm, vias 434 -> 435
- net Net-(R37-Pad2): track 0.89 -> 0.01 mm
- net Net-(L6-Pad1): track 17.9 -> 17.4 mm
- net Net-(C53-Pad2): track 2.87 -> 3.40 mm

Commit message: update bill of materials
Parts:
- C18, C19: footprint Capacitor_Tantalum_SMD:CP_EIA-3528-15_AVX-H_Pad1.50x2.35mm_HandSolder -> Capacitor_Tantalum_SMD:CP_EIA-3528-12_Kemet-T
- D12: value Yellow -> LTST-C191KGKT
- D13: value Green -> LTST-C191KRKT
- J3: value JTAG_10PIN -> Tag-Connect_TC2050-IDC-NL

Commit message: fix antenna impedance
Parts:
- C18, C19: value 330uF -> 330u; footprint Capacitor_Tantalum_SMD:CP_EIA-3528-12_Kemet-T -> Capacitor_Tantalum_SMD:CP_EIA-3528-21_Kemet-B
- C51: value 1.4p -> 1p4
- C52: value 1.2p -> 1p2
- D10, D11, D2, D3, D5, D7, D8: footprint Capacitor_SMD:C_0402_1005Metric -> Diode_SMD:D_SOD-882
- FB3: value 0.4p -> 0p4
- J6: value Qwiic -> SM04B-SRSS-TB(LF)(SN)
- L2: value 9.5n -> 9n5
- L3: value 6.1n -> 6n1
- L5: value 4.3n -> 4n3
- L6: value 1.3n -> 1n3
- R1, R2: value 5.1k -> 5k1
- R11, R15, R33, R8, R9: value 10K -> 10k
- R14, R18, R22, R23, R26, R27, R29, R31: value 4.7k -> 4k7
- R19: value 5K1 -> 5k1
- R43: value 120K -> 120k
- R44: value 20K -> 20k
- SW1: value RESET -> KMR233GLFG
- SW2: value BOOT -> KMR233GLFG
- U9: value A7670C_24x24mm -> A7670C
Routing:
- net Net-(L1-Pad1): track 0.00 -> 2.87 mm
- net Net-(J5-SIG): track 5.91 -> 7.68 mm
- net Net-(R36-Pad2): track 1.89 -> 3.29 mm
- net Net-(R37-Pad2): track 0.01 -> 1.11 mm
- net GND: vias 435 -> 430
