File: hardware/kicad/bwlc1a_A7670C.kicad_sch (KiCad schematic)
At the start: 54 parts, among them J3 Nano SIM, J5 RSP-122811-02, Q1 NPN, Q2 NPN, Q5 NPN, Q6 NPN, U2 A7670C_24x24mm, U5 MIC29302WU

Commit message: Update PCB
Parts:
- C16: Distributor (none) -> LCSC; Distributor Link (none) -> https://www.lcsc.com/product-detail/Multilayer-Ceramic-Capa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; Distributor Part Number (none) -> C106199; Id (none) -> 10; Manufacture (none) -> YAGEO; Manufacture Part Number (none) -> CC0402JRNPO9BN100; Type (none) -> SMD
- C17: Distributor (none) -> LCSC; Distributor Link (none) -> https://www.lcsc.com/product-detail/Multilayer-Ceramic-Capa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; Distributor Part Number (none) -> C1562; Id (none) -> 11; Manufacture (none) -> FH (Guangdong Fenghua Advanced Tech); Manufacture Part Number (none) -> 0402CG330J500NT; Type (none) -> SMD
- C18, C29, C36: Distributor (none) -> LCSC; Distributor Link (none) -> https://www.lcsc.com/product-detail/Multilayer-Ceramic-Capa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; Distributor Part Number (none) -> C1525; Id (none) -> 3; Manufacture (none) -> Samsung Electro-Mechanics; Manufacture Part Number (none) -> CL05B104KO5NNNC; Type (none) -> SMD
- C19: Distributor (none) -> LCSC; Distributor Link (none) -> https://www.lcsc.com/product-detail/Multilayer-Ceramic-Capa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; Distributor Part Number (none) -> C14445; Id (none) -> 12; Manufacture (none) -> Samsung Electro-Mechanics; Manufacture Part Number (none) -> CL05A105KP5NNNC; Type (none) -> SMD
- C20, C21: footprint Capacitor_SMD:C_0603_1608Metric -> Capacitor_SMD:C_0805_2012Metric; Distributor (none) -> LCSC; Distributor Link (none) -> https://www.lcsc.com/product-detail/Multilayer-Ceramic-Capa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; Distributor Part Number (none) -> C141660; Id (none) -> 13; Manufacture (none) -> Murata Electronics; Manufacture Part Number (none) -> GRM21BR60J107ME15L; Type (none) -> SMD
- C22: Distributor (none) -> LCSC; Distributor Link (none) -> https://www.lcsc.com/product-detail/Aluminum-Electrolytic-C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; Distributor Part Number (none) -> C90273; Id (none) -> 6; Manufacture (none) -> ROQANG; Manufacture Part Number (none) -> VT1C101M0605; Type (none) -> SMD
- C23: Distributor (none) -> LCSC; Distributor Link (none) -> https://www.lcsc.com/product-detail/Multilayer-Ceramic-Capa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; Distributor Part Number (none) -> C19702; Id (none) -> 7; Manufacture (none) -> Samsung Electro-Mechanics; Manufacture Part Number (none) -> CL10A106KP8NNNC; Type (none) -> SMD
- C24: footprint Capacitor_SMD:CP_Elec_6.3x7.7 -> Capacitor_SMD:CP_Elec_6.3x5.4; Distributor (none) -> LCSC; Distributor Link (none) -> https://www.lcsc.com/product-detail/Aluminum-Electrolytic-C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; Distributor Part Number (none) -> C2999060; Id (none) -> 8; Manufacture (none) -> ROQANG; Manufacture Part Number (none) -> RVT0J331M0605; Type (none) -> SMD
- C25: Distributor (none) -> LCSC; Distributor Link (none) -> https://www.lcsc.com/product-detail/Multilayer-Ceramic-Capa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; Distributor Part Number (none) -> C49678; Id (none) -> 9; Manufacture (none) -> YAGEO; Manufacture Part Number (none) -> CC0805KRX7R9BB104; Type (none) -> SMD
- C31, C32: Distributor (none) -> -; Distributor Link (none) -> -; Distributor Part Number (none) -> -; Id (none) -> 16; Manufacture (none) -> -; Manufacture Part Number (none) -> -; Type (none) -> SMD
- C35, C36: Distributor (none) -> LCSC; Distributor Link (none) -> https://www.lcsc.com/product-detail/Multilayer-Ceramic-Capa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; Distributor Part Number (none) -> C14442; Id (none) -> 14; Manufacture (none) -> Samsung Electro-Mechanics; Manufacture Part Number (none) -> CL05B102KB5NNNC; Type (none) -> SMD
- C37: value 470p (N.C) -> 470p; Distributor (none) -> LCSC; Distributor Link (none) -> https://www.lcsc.com/product-detail/Multilayer-Ceramic-Capa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; Distributor Part Number (none) -> C106207; Id (none) -> 15; Manufacture (none) -> YAGEO; Type (none) -> SMD
- D1, D4: Distributor (none) -> LCSC; Distributor Link (none) -> https://www.lcsc.com/product-detail/span-style-background-c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; Distributor Part Number (none) -> C5173252; Id (none) -> 19; Manufacture (none) -> Leiditech; Manufacture Part Number (none) -> ESDBW5V0A1; Type (none) -> SMD
- D5: Distributor (none) -> LCSC; Distributor Link (none) -> https://www.lcsc.com/product-detail/span-style-background-c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; Distributor Part Number (none) -> C970036; Id (none) -> 20; Manufacture (none) -> TECH PUBLIC; Manufacture Part Number (none) -> ESDA6V1W5-TP; Type (none) -> SMD
- D7: Distributor (none) -> LCSC; Distributor Link (none) -> https://www.lcsc.com/product-detail/span-style-background-c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; Distributor Part Number (none) -> C558621; Id (none) -> 21; Manufacture (none) -> TECH PUBLIC; Manufacture Part Number (none) -> TPESD0402G36V; Type (none) -> SMD
- F1: value 3A -> 2A; footprint Fuse:Fuse_1206_3216Metric -> Fuse:Fuse_1812_4532Metric; Distributor (none) -> LCSC; Distributor Link (none) -> https://www.lcsc.com/product-detail/span-style-background-c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; Distributor Part Number (none) -> C960026; Id (none) -> 22; Manufacture (none) -> BHFUSE; Manufacture Part Number (none) -> BSMD1812-200-30V; Type (none) -> SMD
- FB1: Distributor (none) -> LCSC; Distributor Link (none) -> https://www.lcsc.com/product-detail/Ferrite-Beads_Murata-El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; Distributor Part Number (none) -> C16903; Id (none) -> 23; Manufacture (none) -> Murata Electronics; Manufacture Part Number (none) -> BLM21PG300SN1D; Type (none) -> SMD
- J3: Distributor (none) -> LCSC; Distributor Link (none) -> https://www.lcsc.com/product-detail/span-style-background-c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; Distributor Part Number (none) -> C266889; Field4 C266889 -> (none); Id (none) -> 27; Manufacture (none) -> XUNPU; Manufacture Part Number (none) -> SMN-304; Type (none) -> SMD
- J5: Distributor (none) -> LCSC; Distributor Link (none) -> https://www.lcsc.com/product-detail/RF-Connectors-Coaxial-C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; Distributor Part Number (none) -> C88374; Id (none) -> 28; MANUFACTURER SAMTEC -> (none); Manufacture (none) -> HRS(Hirose); Manufacture Part Number (none) -> U.FL-R-SMT-1(80); STANDARD Manufacturer recommendations -> (none); Type (none) -> SMD
- JP1: Distributor (none) -> -; Distributor Link (none) -> -; Distributor Part Number (none) -> -; Id (none) -> 31; Manufacture (none) -> -; Manufacture Part Number (none) -> -; Type (none) -> SMD; now left out of the parts list
- JP2: Distributor (none) -> -; Distributor Link (none) -> -; Distributor Part Number (none) -> -; Id (none) -> 30; Manufacture (none) -> -; Manufacture Part Number (none) -> -; Type (none) -> SMD; now left out of the parts list
- Q1, Q2, Q5, Q6: value NPN -> S8050; Distributor (none) -> LCSC; Distributor Link (none) -> https://www.lcsc.com/product-detail/Bipolar-Transistors-BJT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; Distributor Part Number (none) -> C181158; Id (none) -> 34; Manufacture (none) -> Guangdong Hottech; Manufacture Part Number (none) -> S8050; Type (none) -> SMD
- R10, R12, R7: Distributor (none) -> LCSC; Distributor Link (none) -> https://www.lcsc.com/product-detail/Chip-Resistor-Surface-M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; Distributor Part Number (none) -> C25792; Id (none) -> 41; Manufacture (none) -> UNI-ROYAL(Uniroyal Elec); Manufacture Part Number (none) -> 0402WGF4702TCE; Type (none) -> SMD
- R11, R24, R25, R26, R27, R9: Distributor (none) -> LCSC; Distributor Link (none) -> https://www.lcsc.com/product-detail/Chip-Resistor-Surface-M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; Distributor Part Number (none) -> C25940; Id (none) -> 39; Manufacture (none) -> UNI-ROYAL(Uniroyal Elec); Manufacture Part Number (none) -> 0402WGJ0472TCE; Type (none) -> SMD
- R13: Distributor (none) -> LCSC; Distributor Link (none) -> https://www.lcsc.com/product-detail/Chip-Resistor-Surface-M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; Distributor Part Number (none) -> C25744; Id (none) -> 40; Manufacture (none) -> UNI-ROYAL(Uniroyal Elec); Manufacture Part Number (none) -> 0402WGF1002TCE; Type (none) -> SMD
- R14, R15, R16: Distributor (none) -> LCSC; Distributor Link (none) -> https://www.lcsc.com/product-detail/Chip-Resistor-Surface-M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; Distributor Part Number (none) -> C25092; Id (none) -> 43; Manufacture (none) -> UNI-ROYAL(Uniroyal Elec); Manufacture Part Number (none) -> 0402WGF220JTCE; Type (none) -> SMD
- R20, R21: Distributor (none) -> LCSC; Distributor Link (none) -> https://www.lcsc.com/product-detail/Chip-Resistor-Surface-M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; Distributor Part Number (none) -> C21376; Id (none) -> 45; Manufacture (none) -> UNI-ROYAL(Uniroyal Elec); Manufacture Part Number (none) -> 0402WGJ0000TCE; Type (none) -> SMD
- R6: Distributor (none) -> LCSC; Distributor Link (none) -> https://www.lcsc.com/product-detail/Chip-Resistor-Surface-M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; Distributor Part Number (none) -> C25741; Id (none) -> 38; Manufacture (none) -> UNI-ROYAL(Uniroyal Elec); Manufacture Part Number (none) -> 0402WGF1003TCE; Type (none) -> SMD
- R8: Distributor (none) -> LCSC; Distributor Link (none) -> https://www.lcsc.com/product-detail/Chip-Resistor-Surface-M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; Distributor Part Number (none) -> C25117; Id (none) -> 44; Manufacture (none) -> UNI-ROYAL(Uniroyal Elec); Manufacture Part Number (none) -> 0402WGF4700TCE; Type (none) -> SMD
- TP1: Distributor (none) -> -; Distributor Link (none) -> -; Distributor Part Number (none) -> -; Id (none) -> 47; Manufacture (none) -> -; Manufacture Part Number (none) -> -; Type (none) -> SMD; now left out of the parts list
- TP2: Distributor (none) -> -; Distributor Link (none) -> -; Distributor Part Number (none) -> -; Id (none) -> 48; Manufacture (none) -> -; Manufacture Part Number (none) -> -; Type (none) -> SMD; now left out of the parts list
- TP3: Distributor (none) -> -; Distributor Link (none) -> -; Distributor Part Number (none) -> -; Id (none) -> 49; Manufacture (none) -> -; Manufacture Part Number (none) -> -; Type (none) -> SMD; now left out of the parts list
- TP4: Distributor (none) -> -; Distributor Link (none) -> -; Distributor Part Number (none) -> -; Id (none) -> 50; Manufacture (none) -> -; Manufacture Part Number (none) -> -; Type (none) -> SMD; now left out of the parts list
- U2: Distributor (none) -> LCSC; Distributor Link (none) -> https://www.lcsc.com/product-detail/2G-3G-4G-5G-Modules_SIM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; Distributor Part Number (none) -> C2888406; Id (none) -> 59; Manufacture (none) -> SIMCom Wireless Solutions; Manufacture Part Number (none) -> A7670C-LASE; Type (none) -> SMD
- U5: Distributor (none) -> LCSC; Distributor Link (none) -> https://www.lcsc.com/product-detail/Linear-Voltage-Regulato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; Distributor Part Number (none) -> C11149; Id (none) -> 58; Manufacture (none) -> Microchip Tech; Manufacture Part Number (none) -> MIC29302WU-TR; Type (none) -> SMD

Commit message: Update A7670C footprint
Parts:
- U2: footprint Teapot:A7670C_24x24mm -> A7670C:LGA-124_L24.0-W24.0-P1.0-A7670C-LASS
Changed lines of the file:
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@@
       (effects (font (size 1.27 1.27)))
     )
-    (property "Footprint" "Teapot:A7670C_24x24mm" (at 62.865 95.885 0)
+    (property "Footprint" "A7670C:LGA-124_L24.0-W24.0-P1.0-A7670C-LASS" (at 62.865 95.885 0)
       (effects (font (size 1.27 1.27)) hide)
     )

Commit message: Production file update
Parts:
- J5: value RSP-122811-02 -> BWIPX-1-001E; Distributor Link https://www.lcsc.com/product-detail/RF-Connectors-Coaxial-Connectors_HRS-Hirose-U-FL-R-SMT-1-80_C88374.html -> https://www.lcsc.com/product-detail/RF-Connectors-Coaxial-Connectors_BAT-WIRELESS-BWIPX-1-001E_C496552.html; Distributor Part Number C88374 -> C496552; Manufacture HRS(Hirose) -> BAT WIRELESS; Manufacture Part Number U.FL-R-SMT-1(80) -> BWIPX-1-001E
Changed lines of the file:
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@@
       (effects (font (size 1.27 1.27)) (justify left))
     )
-    (property "Value" "RSP-122811-02" (at 171.45 110.617 0)
+    (property "Value" "BWIPX-1-001E" (at 171.45 110.617 0)
       (effects (font (size 1.27 1.27)) (justify left))
     )
@@
       (effects (font (size 1.27 1.27)) hide)
     )
-    (property "Description" "Brass 1 Inner needle IPEX Board Edge 1.25mm -40℃~+90℃ 6GHz 50Ω 2mm SMD RF Connectors / Coaxial Connectors ROHS" (at 160.782 107.442 0)
+    (property "Description" "1 Inner needle IPEX Board Edge 6GHz 50Ω SMD RF Connectors / Coaxial Connectors ROHS" (at 160.782 107.442 0)
       (effects (font (size 1.27 1.27)) hide)
     )
@@
       (effects (font (size 1.27 1.27)) hide)
     )
-    (property "Distributor Link" "https://www.lcsc.com/product-detail/RF-Connectors-Coaxial-Connectors_HRS-Hirose-U-FL-R-SMT-1-80_C88374.html" (at 160.782 107.442 0)
+    (property "Distributor Link" "https://www.lcsc.com/product-detail/RF-Connectors-Coaxial-Connectors_BAT-WIRELESS-BWIPX-1-001E_C496552.html" (at 160.782 107.442 0)
       (effects (font (size 1.27 1.27)) hide)
     )
-    (property "Distributor Part Number" "C88374" (at 160.782 107.442 0)
+    (property "Distributor Part Number" "C496552" (at 160.782 107.442 0)
       (effects (font (size 1.27 1.27)) hide)
     )
@@
       (effects (font (size 1.27 1.27)) hide)
     )
-    (property "Manufacture" "HRS(Hirose)" (at 160.782 107.442 0)
+    (property "Manufacture" "BAT WIRELESS" (at 160.782 107.442 0)
       (effects (font (size 1.27 1.27)) hide)
     )
-    (property "Manufacture Part Number" "U.FL-R-SMT-1(80)" (at 160.782 107.442 0)
+    (property "Manufacture Part Number" "BWIPX-1-001E" (at 160.782 107.442 0)
       (effects (font (size 1.27 1.27)) hide)
     )

Commit message: Update PCB
Parts:
- removed J3: Nano SIM, GCT_SIM8051-6-0-14-00-X-REVD:GCT_SIM8051-6-0-14-00-X-REVD, symbol Connector:SIM_Card
- added J4: SMN-304, SIM-SMD_SMN-304:SIM-SMD_SMN-304, symbol SIM-SMD_SMN-304:SMN-304
Connections:
- net GND: now also J4.C5 (GND)
- net USIM_CLK: now also R15.1; no longer R14.1
- net USIM_DATA: now also R16.2; no longer R16.1
- net USIM_RST: now also R14.1; no longer R15.1
- net USIM_VDD: now also D5.1 (K), J4.C1 (VCC); no longer D5.5 (K)
- net at D5.3 (K), R14.2: now also J4.C2 (RST)
- net at D5.4 (K), R15.2: now also J4.C3 (CLK)
- new net: D5.5 (K), J4.C7 (I/O), R16.1
- no-connect marks 36 -> 38
Other:
- moved on the sheet: C29, D5, R14, R15, R16
