File: hardware/kicad/bwlc1a_A7670C.kicad_sch (KiCad schematic)
At the start: 54 parts, among them J4 SMN-304, J5 BWIPX-1-001E, Q1 S8050, Q2 S8050, Q5 S8050, Q6 S8050, U2 A7670C_24x24mm, U5 MIC29302WU

Commit message: update design
Other:
- note added: "Power Off: 20uA LTE Sleep: 2.5mA LTE Idle: 25mA"
- note added: "TODO: Change to use 2x TPS27081A ( for Celullar and GPS ) Iq: 0.03 uA"
Changed lines of the file:
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@@
+    (effects (font (size 1.27 1.27)) (justify left bottom))
+  )
+  (text "Power Off: 20uA\nLTE Sleep: 2.5mA\nLTE Idle: 25mA" (at 14.605 73.66 0)
     (effects (font (size 1.27 1.27)) (justify left bottom))
   )
@@
     (effects (font (size 1.27 1.27)) (justify left bottom))
   )
+  (text "TODO: Change to use 2x TPS27081A ( for Celullar and GPS )\nIq: 0.03 uA"
+    (at 85.725 18.415 0)
+    (effects (font (size 1.27 1.27)) (justify left bottom))
+  )
