File: hardware/kicad/bwlc1a.kicad_sch (KiCad schematic)
At the start: 7 parts, among them U1 ESP32-C3, U2 W25Q32JVSS, Y1 40Mhz

Commit message: Push before change to ESP32 S3
Parts:
- removed U1: ESP32-C3, Package_DFN_QFN:QFN-32-1EP_5x5mm_P0.5mm_EP3.45x3.45mm, symbol Espressif:ESP32-C3
- removed U2: W25Q32JVSS, Package_SO:SOIC-8_5.23x5.23mm_P1.27mm, symbol Memory_Flash:W25Q32JVSS
- removed Y1: 40Mhz, symbol Device:Crystal_GND24
- added ANT1: ESP, symbol Connector_Generic:Conn_01x02
- added C10, C14, C3, C33, C39, C42, C47, C5, C6, C7: 100n, symbol Device:C_Small
- added C11: 22u, symbol Device:C_Small
- added C12, C13: 10p, symbol Device:C_Small
- added C15: 1u, symbol Device:C_Small
- added C34, C38, C4, C43, C44, C45, C46: 10u, symbol Device:C_Small
- added C40, C41: 9p, symbol Device:C_Small
- added C8, C9: TBD, symbol Device:C_Small
- added D6: B5819W, symbol Device:D_Schottky
- added D8: Orange, symbol Device:LED_Small
- added D9: D_TVS, symbol Device:D_TVS
- added J1: USB_C_Receptacle_USB2.0, symbol Connector:USB_C_Receptacle_USB2.0
- added J4: JST-2PH, symbol Connector_Generic:Conn_01x02
- added J6: Conn_ARM_JTAG_SWD_10, symbol Connector:Conn_ARM_JTAG_SWD_10
- added L2: TBD, symbol Device:L_Small
- added Q3: DMG3415UQ-7, symbol Simulation_SPICE:PMOS
- added Q4: NPN, symbol Simulation_SPICE:NPN
- added R17: 10K, symbol Device:R_Small
- added R2: 5.1k, symbol Device:R_Small
- added R20, R21: 1k, symbol Device:R_Small
- added R22: 4.7k, symbol Device:R_Small
- added R23: 47k, symbol Device:R_Small
- added R3, R4: 10k, symbol Device:R_Small
- added R5: 1M, symbol Device:R_Small
- added SW1: EN_ESP, symbol Switch:SW_Push
- added U1: USBLC6-2SC6, Package_TO_SOT_SMD:SOT-23-6, symbol Power_Protection:USBLC6-2SC6
- added U3: ESP32-C3FN4, Package_DFN_QFN:QFN-32-1EP_5x5mm_P0.5mm_EP3.45x3.45mm, symbol Espressif:ESP32-C3
- added U4: LSM6DS3, Package_LGA:LGA-14_3x2.5mm_P0.5mm_LayoutBorder3x4y, symbol Sensor_Motion:LSM6DS3
- added U6: L86-M33, XCVR_L86-M33, symbol L86-M33:L86-M33
- added U7: SPX3819M5-L-3-3, Package_TO_SOT_SMD:SOT-23-5, symbol Regulator_Linear:SPX3819M5-L-3-3
- added U8: MCP73831-2-OT, Package_TO_SOT_SMD:SOT-23-5, symbol Battery_Management:MCP73831-2-OT
- added U9: MAX17048G+, SON50P200X200X80-9N, symbol MAX17048G:MAX17048G+
- added Y1: 40Mhz, symbol Device:Crystal_GND24_Small
- added Y2: 32.768 kHz, symbol Device:Crystal_Small
- C1: value 10p -> 1u
- C2: value 10p -> 10n
- L1: value L_Small -> 2n
- R1: value R_Small -> 5.1k
Connections:
- net GND: now also R1.2, ANT1.2 (Pin_2), C10.2, C11.2, C12.2, C13.2, C14.2, C15.2, C3.2, C33.2, C34.2, C38.2, C39.2, C4.2, C40.2, C41.1, C42.2, C43.2, C44.2, C45.2, C46.2, C47.2, C5.2, C6.2, C7.2, C8.2, C9.2, D9.1 (A1), J1.A1 (GND), J1.A12 (GND), J1.B1 (GND), J1.B12 (GND), J4.2 (Pin_2), J6.3 (GND), J6.5 (GND), Q4.3 (E), R17.1, R2.2, R21.2, R23.2, R4.1, R5.1, SW1.1, U1.2 (GND), U3.33 (GND), U4.2 (SDX), U4.3 (SCX), U4.6 (GND), U4.7 (GND), U6.12 (GND), U6.3 (GND), U7.2 (GND), U8.2 (V_{SS}), U9.1 (CTG), U9.4 (GND), U9.6 (QSTRT), U9.9 (EP), Y1.2, Y1.4
- net +3.3V: now reaches L1.1
- net +3.3V: now also C1.1, C2.1, C10.1, C11.1, C3.1, C38.1, C39.1, C4.1, C43.1, C5.1, C7.1, D9.2 (A2), U3.11 (VDD3P3_RTC), U3.17 (VDD3P3_CPU), U3.31 (VDDA), U3.32 (VDDA), U4.12 (CS), U4.5 (VDDIO), U4.8 (VDD), U7.5 (OUT)
- net VDD3V3: now reaches L1.2
- net VDD3V3: now also C6.1, U3.2 (VDD3P3), U3.3 (VDD3P3)
- net at R1.1: now also J1.A5 (CC1)
- new net: Q4.1 (C), U6.10 (~{RESET})
- new net: Q4.2 (B), R22.2, R23.1
- new net: ANT1.1 (Pin_1), C8.1, L2.1
- new net: J1.B5 (CC2), R2.1
- new net: R20.1, U8.1 (STAT)
- new net: D8.1 (K), R20.2
- new net: R4.2, U4.1 (SDO/SA0)
- new net: R21.1, U8.5 (PROG)
- new net: C44.1, D6.1 (K), Q3.3 (S), U7.1 (IN), U7.3 (EN)
- new net: C42.1, U7.4 (BP)
- new net +3V3: J6.1 (VTref), R3.1
- new net +BATT: C46.1, C47.1, J4.1 (Pin_1), Q3.1 (D), U8.3 (V_{BAT}), U9.2 (CELL), U9.3 (VDD)
- new net A7670_RX: U3.28 (U0TXD/GPIO21)
- new net A7670_TX: U3.27 (U0RXD/GPIO20)
- new net EN_ESP: J6.10 (~{RESET})
- new net ESP_32K_N: C41.2, U3.5 (XTAL_32K_N/ADC1_CH1), Y2.1
- new net ESP_32K_P: C40.1, U3.4 (XTAL_32K_P/ADC1_CH0), Y2.2
- new net ESP_ANT: C9.1, L2.2, U3.1 (LNA_IN)
- new net ESP_D+: U1.1 (I/O1)
- new net ESP_D-: U1.3 (I/O2)
- new net ESP_EN: C14.1, R3.2, SW1.2, U3.7 (CHIP_EN)
- new net ESP_XTAL_N: C12.1, U3.29 (XTAL_N), Y1.3
- new net ESP_XTAL_P: C13.1, U3.30 (XTAL_P), Y1.1
- new net GPS_FORCE_ON: R5.2, U6.7 (FORCE_ON)
- new net GPS_RST: R22.1
- new net GPS_RX: U6.1 (RXD1)
- new net GPS_TX: U6.2 (TXD1)
- new net IMU_INT: U4.4 (INT1)
- new net IMU_SCL: U3.8 (GPIO3/ADC1_CH3), U4.13 (SCL), U9.7 (SCL)
- new net IMU_SDA: U3.6 (GPIO2/ADC1_CH2), U4.14 (SDA), U9.8 (SDA)
- new net JTAG_TCK: J6.4 (SWDCLK/TCK), U3.12 (MTCK/GPIO6)
- new net JTAG_TDI: J6.8 (NC/TDI), U3.10 (MTDI/GPIO5/ADC2_CH0)
- new net JTAG_TDO: J6.6 (SWO/TDO), U3.13 (MTDO/GPIO7)
- new net JTAG_TMS: J6.2 (SWDIO/TMS), U3.9 (MTMS/GPIO4/ADC1_CH4)
- new net MAX17048_INT: U9.5 (~{ALERT})
- new net USB_D+: J1.A6 (D+), J1.B6 (D+), U1.6 (I/O1), U3.26 (GPIO19/USB_D+)
- new net USB_D-: J1.A7 (D-), J1.B7 (D-), U1.4 (I/O2), U3.25 (GPIO18/USB_D-)
- new net VBUS: C45.1, D6.2 (A), D8.2 (A), J1.A4 (VBUS), J1.A9 (VBUS), J1.B4 (VBUS), J1.B9 (VBUS), Q3.2 (G), R17.2, U1.5 (VBUS), U8.4 (V_{DD})
- new net VDD_BAT: C33.1, C34.1, U6.4 (VCC), U6.5 (V_BCKP)
- new net VDD_SPI: C15.1, U3.18 (VDD_SPI/GPIO11)
- no-connect marks 0 -> 8
Other:
- added sheet bwlc1a_A7670C (bwlc1a_A7670C.kicad_sch)
- note added: "1-Cell LiPo Charger"
- note added: "32.768kHz Crystal"
- note added: "40MHz Crystal"
- note added: "5.5x8.5 cm"
- note added: "Antenna"
- note added: "DOES NOT REQUIRE FLASH MEMORY"
- note added: "Decoupling Capacitors"
- note added: "EN/Reset"
- note added: "ESD"
- note added: "ESP32 C3 Datasheet: https://www.espressif.com/sites/default/files/documentation/esp32-c3_datasheet_en.pdf"
- note added: "ESP32 C3 Design Guideline: https://www.espressif.com/sites/default/files/documentation/esp32-c3_hardware_design_guidelines_en.pdf"
- note added: "ESP32-C3FN4"
- note added: "Fuel Gauge"
- note added: "GPS"
- note added: "IMU Sensor"
- note added: "JTAG"
- note added: "LDO 3V3 500mA"
- note added: "Phil's C3 Board: https://www.youtube.com/watch?v=yxU_Kw2de08"
- note added: "Pull-up"
- note added: "USB C"

Commit message: Finish Sch, start Layouting
Parts:
- removed ANT1: ESP, symbol Connector_Generic:Conn_01x02
- removed C1: 1u, symbol Device:C_Small
- removed C12, C13: 10p, symbol Device:C_Small
- removed C2: 10n, symbol Device:C_Small
- removed C42, C5, C6: 100n, symbol Device:C_Small
- removed C43: 10u, symbol Device:C_Small
- removed C8, C9: TBD, symbol Device:C_Small
- removed L2: TBD, symbol Device:L_Small
- removed U3: ESP32-C3FN4, Package_DFN_QFN:QFN-32-1EP_5x5mm_P0.5mm_EP3.45x3.45mm, symbol Espressif:ESP32-C3
- removed U7: SPX3819M5-L-3-3, Package_TO_SOT_SMD:SOT-23-5, symbol Regulator_Linear:SPX3819M5-L-3-3
- removed Y1: 40Mhz, symbol Device:Crystal_GND24_Small
- added JP1: BOOT, Jumper:SolderJumper-2_P1.3mm_Open_RoundedPad1.0x1.5mm, symbol Jumper:SolderJumper_2_Open
- added R15: N.C, Resistor_SMD:R_0402_1005Metric, symbol Device:R_Small
- added R3: 453k, Resistor_SMD:R_0402_1005Metric, symbol Device:R_Small
- added R7: 100k, Resistor_SMD:R_0402_1005Metric, symbol Device:R_Small
- added R8, R9: 4.7k, Resistor_SMD:R_0402_1005Metric, symbol Device:R_Small
- added U3: TPS62290DRVR, TPS62290DRVR:SON65P200X200X80-7N, symbol TPS62290DRVR:TPS62290DRVR
- added U6: ESP32-S3-MINI-1, Espressif:ESP32-S3-MINI-1, symbol Espressif:ESP32-S3-MINI-1
- C1: renamed from C45; footprint (none) -> Capacitor_SMD:C_0603_1608Metric
- C10, C7: footprint (none) -> Capacitor_SMD:C_0402_1005Metric
- C11, C4: footprint (none) -> Capacitor_SMD:C_0603_1608Metric
- C12: renamed from C38; footprint (none) -> Capacitor_SMD:C_0603_1608Metric
- C13: renamed from C33; footprint (none) -> Capacitor_SMD:C_0402_1005Metric
- C14: renamed from C34; footprint (none) -> Capacitor_SMD:C_0603_1608Metric
- C15: renamed from C40; footprint (none) -> Capacitor_SMD:C_0402_1005Metric
- C16: renamed from C41; footprint (none) -> Capacitor_SMD:C_0402_1005Metric
- C17: renamed from C14; footprint (none) -> Capacitor_SMD:C_0402_1005Metric
- C2: renamed from C46; footprint (none) -> Capacitor_SMD:C_0603_1608Metric
- C3: value 100n -> 22p; footprint (none) -> Capacitor_SMD:C_0402_1005Metric
- C5: renamed from C44; footprint (none) -> Capacitor_SMD:C_0603_1608Metric
- C6: renamed from C15; value 1u -> 10u; footprint (none) -> Capacitor_SMD:C_0603_1608Metric
- C8: renamed from C47; footprint (none) -> Capacitor_SMD:C_0402_1005Metric
- C9: renamed from C39; footprint (none) -> Capacitor_SMD:C_0402_1005Metric
- D1: renamed from D8; footprint (none) -> LED_SMD:LED_0603_1608Metric
- D2: renamed from D6; footprint (none) -> Diode_SMD:D_SOD-123
- D3: renamed from D9; footprint (none) -> Capacitor_SMD:C_0402_1005Metric
- J1: renamed from J4; footprint (none) -> Teapot:JST_PH_S2B-PH-SM4-TB_1x02-1MP_P2.00mm_Horizontal
- J2: renamed from J1; footprint (none) -> Connector_USB:USB_C_Receptacle_HRO_TYPE-C-31-M-12
- J3: renamed from J6; value Conn_ARM_JTAG_SWD_10 -> JTAG_10PIN
- L1: value 2n -> 2.2u; footprint (none) -> Inductor_SMD:L_1008_2520Metric
- Q1: renamed from Q3; footprint (none) -> Keebio-Parts:SOT-23
- Q2: renamed from Q4; footprint (none) -> Package_TO_SOT_SMD:SOT-23
- R1, R2: footprint (none) -> Resistor_SMD:R_0402_1005Metric
- R10: renamed from R4; footprint (none) -> Resistor_SMD:R_0402_1005Metric
- R11: renamed from R22; footprint (none) -> Resistor_SMD:R_0402_1005Metric
- R12: renamed from R23; footprint (none) -> Resistor_SMD:R_0402_1005Metric
- R13: renamed from R5; value 1M -> 10k; footprint (none) -> Resistor_SMD:R_0402_1005Metric
- R14: renamed from R3; footprint (none) -> Resistor_SMD:R_0402_1005Metric
- R4: renamed from R20; footprint (none) -> Resistor_SMD:R_0402_1005Metric
- R5: renamed from R21; footprint (none) -> Resistor_SMD:R_0402_1005Metric
- R6: renamed from R17; footprint (none) -> Resistor_SMD:R_0402_1005Metric
- SW1: footprint (none) -> Button_Switch_SMD:SW_Push_1P1T_NO_CK_KMR2
- U4: renamed from U9; footprint SON50P200X200X80-9N -> Package_DFN_QFN:DFN-8-1EP_2x2mm_P0.5mm_EP0.7x1.3mm
- U7: renamed from U6; footprint XCVR_L86-M33 -> Teapot:XCVR_L86-M33
- Y1: renamed from Y2; footprint (none) -> Crystal:Crystal_SMD_2012-2Pin_2.0x1.2mm
- renumbered U8 to U1, U1 to U2, U4 to U5
Connections:
- net VDD_SPI is gone; now on net +3.3V: C6.1
- net +3.3V: now also R3.2, R8.1, R9.1, U6.3 (3V3)
- net ESP_32K_N: now also R15.2, U6.20 (GPIO16/U0CTS/ADC2_CH5/XTAL_32K_N)
- net ESP_32K_P: now also R15.1, U6.19 (GPIO15/U0RTS/ADC2_CH4/XTAL_32K_P)
- net ESP_EN: now also U6.45 (EN)
- net GND: now also JP1.2 (B), R7.1, U3.2 (MODE), U3.6 (GND), U3.7 (THERMALPAD), U6.1 (GND), U6.2 (GND), U6.42 (GND), U6.43 (GND), U6.46 (GND), U6.47 (GND), U6.48 (GND), U6.49 (GND), U6.50 (GND), U6.51 (GND), U6.52 (GND), U6.53 (GND), U6.54 (GND), U6.55 (GND), U6.56 (GND), U6.57 (GND), U6.58 (GND), U6.59 (GND), U6.60 (GND), U6.61 (GND), U6.62 (GND), U6.63 (GND), U6.64 (GND), U6.65 (GND); no longer C3.2
- net GPS_RX: now also U6.39 (U0TXD/GPIO43/CLK_OUT1)
- net GPS_TX: now also U6.40 (U0RXD/GPIO44/CLK_OUT2)
- net IMU_SCL: now also R9.2
- net IMU_SDA: now also R8.2
- net JTAG_TCK: now also U6.35 (MTCK/GPIO39/CLK_OUT3/SUBSPICS1)
- net JTAG_TDI: now also U6.37 (MTDI/GPIO41/CLK_OUT1)
- net JTAG_TDO: now also U6.36 (MTDO/GPIO40/CLK_OUT2)
- net JTAG_TMS: now also U6.38 (MTMS/GPIO42)
- net USB_D+: now also U6.24 (GPIO20/U1CTS/ADC2_CH9/CLK_OUT1/USB_D+)
- net USB_D-: now also U6.23 (GPIO19/U1RTS/ADC2_CH8/CLK_OUT2/USB_D-)
- net TPS_VIN: now reaches C5.1, D2.1 (K), Q1.3 (S)
- net TPS_VIN: now also U3.4 (EN), U3.5 (VIN)
- net VDD3V3: no longer names the net of L1.2
- net VDD3V3: now also U3.1 (SW)
- new net ESP_BOOT: JP1.1 (A), U6.4 (GPIO0/BOOT)
- new net TPS_FB: C3.2, R3.1, R7.2, U3.3 (FB)
- no-connect marks 8 -> 12
Other:
- note added: "Cellular Module"
- note added: "Datasheet: https://datasheet.lcsc.com/lcsc/1810291810_Texas-Instruments-TPS62290DRVR_C129315.pdf"
- note added: "ESP32-MINI"
- note added: "R1"
- note added: "R2"
- note added: "Step Down/LDO 3V3"
- note added: "USB C + ESD"
- note added: "Vout = 3.318V"
- note added: "Vout = Vref*(1+(R1/R2)) Vref = 0.6V (Typical)"
- note removed: "40MHz Crystal"
- note removed: "Antenna"
- note removed: "DOES NOT REQUIRE FLASH MEMORY"
- note removed: "Decoupling Capacitors"
- note removed: "ESD"
- note removed: "ESP32 C3 Datasheet: https://www.espressif.com/sites/default/files/documentation/esp32-c3_datasheet_en.pdf"
- note removed: "ESP32 C3 Design Guideline: https://www.espressif.com/sites/default/files/documentation/esp32-c3_hardware_design_guidelines_en.pdf"
- note removed: "ESP32-C3FN4"
- note removed: "LDO 3V3 500mA"
- note removed: "Phil's C3 Board: https://www.youtube.com/watch?v=yxU_Kw2de08"
- note removed: "Pull-up"
- note removed: "USB C"
- moved on the sheet: C1, C10, C11, C12, C13, C14, C15, C16, C17, C2, C5, C6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

Commit message: Update on routing
Parts:
- removed R15: N.C, Resistor_SMD:R_0402_1005Metric, symbol Device:R_Small
- R13: value 10k -> 1M
Connections:
- net ESP_D+ is gone; now on net USB_D+: U2.1 (I/O1)
- net ESP_D- is gone; now on net USB_D-: U2.3 (I/O2)
- net A7670_PWR: now also U6.27 (GPIO47/SPICLK_P/SUBSPICLK_P_DIFF)
- net A7670_RST: now also U6.29 (SPIIO5/GPIO34/FSPICS0/SUBSPICS0)
- net A7670_RX: now also U6.39 (U0TXD/GPIO43/CLK_OUT1)
- net A7670_STATUS: now also U6.28 (SPIIO4/GPIO33/FSPIHD/SUBSPIHD)
- net A7670_TX: now also U6.40 (U0RXD/GPIO44/CLK_OUT2)
- net EN_MIC29302: now also U6.30 (GPIO48/SPICLK_N/SUBSPICLK_N_DIFF)
- net GPS_FORCE_ON: now also U6.33 (SPIDQS/GPIO37/FSPIQ/SUBSPIQ)
- net GPS_RST: now also U6.34 (GPIO38/FSPIWP/SUBSPIWP)
- net GPS_RX: now also U6.31 (SPIIO6/GPIO35/FSPID/SUBSPID); no longer U6.39 (U0TXD/GPIO43/CLK_OUT1)
- net GPS_TX: now also U6.32 (SPIIO7/GPIO36/FSPICLK/SUBSPICLK); no longer U6.40 (U0RXD/GPIO44/CLK_OUT2)
- net IMU_SCL: now also R8.2, U6.16 (GPIO12/TOUCH12/ADC2_CH1/FSPICLK/FSPIIO6/SUBSPICLK); no longer R9.2
- net IMU_SDA: now also R9.2, U6.17 (GPIO13/TOUCH13/ADC2_CH2/FSPIQ/FSPIIO7/SUBSPIQ); no longer R8.2
Other:
- moved on the sheet: R8, R9

Commit message: PCB Layout update + Silkscreen
Parts:
- J3: footprint (none) -> Connector:Tag-Connect_TC2050-IDC-NL_2x05_P1.27mm_Vertical
- JP1: footprint Jumper:SolderJumper-2_P1.3mm_Open_RoundedPad1.0x1.5mm -> Button_Switch_SMD:SW_Push_1P1T_NO_CK_KMR2
Connections:
- net +3V3 is gone; now on net +3.3V: J3.1 (VTref), R14.1
- net EN_ESP is gone; now on net ESP_EN: J3.10 (~{RESET})
- net IMU_INT: now also U6.6 (GPIO2/TOUCH2/ADC1_CH1)
- net MAX17048_INT: now also U6.25 (GPIO21)

Commit message: Update PCB
Parts:
- C1, C12, C14, C2, C4, C5, C6: Distributor (none) -> LCSC; Distributor Link (none) -> https://www.lcsc.com/product-detail/Multilayer-Ceramic-Capa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; Distributor Part Number (none) -> C19702; Id (none) -> 1; Manufacture (none) -> Samsung Electro-Mechanics; Manufacture Part Number (none) -> CL10A106KP8NNNC; Type (none) -> SMD
- C10, C13, C17, C7, C8, C9: Distributor (none) -> LCSC; Distributor Link (none) -> https://www.lcsc.com/product-detail/Multilayer-Ceramic-Capa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; Distributor Part Number (none) -> C1525; Id (none) -> 3; Manufacture (none) -> Samsung Electro-Mechanics; Manufacture Part Number (none) -> CL05B104KO5NNNC; Type (none) -> SMD
- C11: Distributor (none) -> LCSC; Distributor Link (none) -> https://www.lcsc.com/product-detail/Multilayer-Ceramic-Capa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; Distributor Part Number (none) -> C86295; Id (none) -> 4; Manufacture (none) -> Samsung Electro-Mechanics; Manufacture Part Number (none) -> CL10A226MP8NUNE; Type (none) -> SMD
- C15, C16: value 9p -> 12p; Distributor (none) -> LCSC; Distributor Link (none) -> https://www.lcsc.com/product-detail/Multilayer-Ceramic-Capa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; Distributor Part Number (none) -> C1547; Id (none) -> 5; Manufacture (none) -> FH (Guangdong Fenghua Advanced Tech); Manufacture Part Number (none) -> 0402CG120J500NT; Type (none) -> SMD
- C3: Distributor (none) -> LCSC; Distributor Link (none) -> https://www.lcsc.com/product-detail/Multilayer-Ceramic-Capa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; Distributor Part Number (none) -> C70464; Id (none) -> 2; Manufacture (none) -> Samsung Electro-Mechanics; Manufacture Part Number (none) -> CL05C220JB5NNNC; Type (none) -> SMD
- D1: Distributor (none) -> LCSC; Distributor Link (none) -> https://www.lcsc.com/product-detail/Light-Emitting-Diodes-L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; Distributor Part Number (none) -> C375450; Id (none) -> 17; Manufacture (none) -> EKINGLUX; Manufacture Part Number (none) -> E6C0603SEAC1UDA; Type (none) -> SMD
- D2: Distributor (none) -> LCSC; Distributor Link (none) -> https://www.lcsc.com/product-detail/Schottky-Barrier-Diodes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; Distributor Part Number (none) -> C8598; Id (none) -> 18; Manufacture (none) -> Jiangsu Changjing Electronics Technology Co., Ltd; Manufacture Part Number (none) -> B5819W SL; Type (none) -> SMD
- D3: value D_TVS -> ESDBW5V0A1; Distributor (none) -> LCSC; Distributor Link (none) -> https://www.lcsc.com/product-detail/span-style-background-c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; Distributor Part Number (none) -> C5173252; Id (none) -> 19; Manufacture (none) -> Leiditech; Manufacture Part Number (none) -> ESDBW5V0A1; Type (none) -> SMD
- J1: Distributor (none) -> LCSC; Distributor Link (none) -> https://www.lcsc.com/product-detail/Wire-To-Board-Wire-To-W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; Distributor Part Number (none) -> C295747; Id (none) -> 24; Manufacture (none) -> JST Sales America Inc.; Manufacture Part Number (none) -> S2B-PH-SM4-TB(LF)(SN); Type (none) -> SMD
- J2: Distributor (none) -> LCSC; Distributor Link (none) -> https://www.lcsc.com/product-detail/span-style-background-c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; Distributor Part Number (none) -> C165948; Id (none) -> 25; Manufacture (none) -> Korean Hroparts Elec; Manufacture Part Number (none) -> TYPE-C-31-M-12; Type (none) -> SMD
- J3: Distributor (none) -> -; Distributor Link (none) -> -; Distributor Part Number (none) -> -; Id (none) -> 26; Manufacture (none) -> -; Manufacture Part Number (none) -> -; Type (none) -> SMD; now left out of the parts list
- JP1: Distributor (none) -> LCSC; Distributor Link (none) -> https://www.lcsc.com/product-detail/Tactile-Switches_C-K-KM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; Distributor Part Number (none) -> C2689601; Id (none) -> 29; Manufacture (none) -> C&K; Manufacture Part Number (none) -> KMR233GLFG; Type (none) -> SMD
- L1: Distributor (none) -> LCSC; Distributor Link (none) -> https://www.lcsc.com/product-detail/Inductors-SMD_Murata-El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; Distributor Part Number (none) -> C86092; Id (none) -> 32; Manufacture (none) -> Murata Electronics; Manufacture Part Number (none) -> LQM2HPN2R2MG0L; Type (none) -> SMD
- Q1: footprint Keebio-Parts:SOT-23 -> Package_TO_SOT_SMD:SOT-23; Distributor (none) -> LCSC; Distributor Link (none) -> https://www.lcsc.com/product-detail/MOSFETs_Diodes-Incorpor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; Distributor Part Number (none) -> C459537; Id (none) -> 33; Manufacture (none) -> Diodes Incorporated; Manufacture Part Number (none) -> DMG3415UQ-7; Type (none) -> SMD
- Q2: value NPN -> S8050; Distributor (none) -> LCSC; Distributor Link (none) -> https://www.lcsc.com/product-detail/Bipolar-Transistors-BJT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; Distributor Part Number (none) -> C181158; Id (none) -> 34; Manufacture (none) -> Guangdong Hottech; Manufacture Part Number (none) -> S8050; Type (none) -> SMD
- R1, R2: Distributor (none) -> LCSC; Distributor Link (none) -> https://www.lcsc.com/product-detail/Chip-Resistor-Surface-M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; Distributor Part Number (none) -> C25905; Id (none) -> 35; Manufacture (none) -> UNI-ROYAL(Uniroyal Elec); Manufacture Part Number (none) -> 0402WGF5101TCE; Type (none) -> SMD
- R10, R14: Distributor (none) -> LCSC; Distributor Link (none) -> https://www.lcsc.com/product-detail/Chip-Resistor-Surface-M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; Distributor Part Number (none) -> C25744; Id (none) -> 40; Manufacture (none) -> UNI-ROYAL(Uniroyal Elec); Manufacture Part Number (none) -> 0402WGF1002TCE; Type (none) -> SMD
- R11, R8, R9: Distributor (none) -> LCSC; Distributor Link (none) -> https://www.lcsc.com/product-detail/Chip-Resistor-Surface-M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; Distributor Part Number (none) -> C25940; Id (none) -> 39; Manufacture (none) -> UNI-ROYAL(Uniroyal Elec); Manufacture Part Number (none) -> 0402WGJ0472TCE; Type (none) -> SMD
- R12: Distributor (none) -> LCSC; Distributor Link (none) -> https://www.lcsc.com/product-detail/Chip-Resistor-Surface-M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; Distributor Part Number (none) -> C25792; Id (none) -> 41; Manufacture (none) -> UNI-ROYAL(Uniroyal Elec); Manufacture Part Number (none) -> 0402WGF4702TCE; Type (none) -> SMD
- R13: Distributor (none) -> LCSC; Distributor Link (none) -> https://www.lcsc.com/product-detail/Chip-Resistor-Surface-M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; Distributor Part Number (none) -> C26083; Id (none) -> 42; Manufacture (none) -> UNI-ROYAL(Uniroyal Elec); Manufacture Part Number (none) -> 0402WGF1004TCE; Type (none) -> SMD
- R3: Distributor (none) -> LCSC; Distributor Link (none) -> https://www.lcsc.com/product-detail/Chip-Resistor-Surface-M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; Distributor Part Number (none) -> C27009; Id (none) -> 36; Manufacture (none) -> UNI-ROYAL(Uniroyal Elec); Manufacture Part Number (none) -> 0402WGF4533TCE; Type (none) -> SMD
- R4, R5: Distributor (none) -> LCSC; Distributor Link (none) -> https://www.lcsc.com/product-detail/Chip-Resistor-Surface-M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; Distributor Part Number (none) -> C25543; Id (none) -> 37; Manufacture (none) -> UNI-ROYAL(Uniroyal Elec); Manufacture Part Number (none) -> 0402WGJ0102TCE; Type (none) -> SMD
- R6: value 10K -> 10k; Distributor (none) -> LCSC; Distributor Link (none) -> https://www.lcsc.com/product-detail/Chip-Resistor-Surface-M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; Distributor Part Number (none) -> C25744; Id (none) -> 40; Manufacture (none) -> UNI-ROYAL(Uniroyal Elec); Manufacture Part Number (none) -> 0402WGF1002TCE; Type (none) -> SMD
- R7: Distributor (none) -> LCSC; Distributor Link (none) -> https://www.lcsc.com/product-detail/Chip-Resistor-Surface-M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; Distributor Part Number (none) -> C25741; Id (none) -> 38; Manufacture (none) -> UNI-ROYAL(Uniroyal Elec); Manufacture Part Number (none) -> 0402WGF1003TCE; Type (none) -> SMD
- SW1: Distributor (none) -> LCSC; Distributor Link (none) -> https://www.lcsc.com/product-detail/Tactile-Switches_C-K-KM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; Distributor Part Number (none) -> C2689601; Id (none) -> 46; Manufacture (none) -> C&K; Manufacture Part Number (none) -> KMR233GLFG; Type (none) -> SMD
- U1: Distributor (none) -> LCSC; Distributor Link (none) -> https://www.lcsc.com/product-detail/Battery-Management-ICs_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; Distributor Part Number (none) -> C14879; Id (none) -> 51; Manufacture (none) -> Microchip Tech; Manufacture Part Number (none) -> MCP73831T-2ATI/OT; Type (none) -> SMD
- U2: Distributor (none) -> LCSC; Distributor Link (none) -> https://www.lcsc.com/product-detail/ESD-Protection-Devices_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; Distributor Part Number (none) -> C2827654; Id (none) -> 52; Manufacture (none) -> TECH PUBLIC; Manufacture Part Number (none) -> USBLC6-2SC6; Type (none) -> SMD
- U3: Distributor (none) -> LCSC; Distributor Link (none) -> https://www.lcsc.com/product-detail/DC-DC-Converters_Texas-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; Distributor Part Number (none) -> C129315; Id (none) -> 53; Manufacture (none) -> Texas Instruments; Manufacture Part Number (none) -> TPS62290DRVR; Type (none) -> SMD
- U4: Distributor (none) -> LCSC; Distributor Link (none) -> https://www.lcsc.com/product-detail/Battery-Management-ICs_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; Distributor Part Number (none) -> C2682616; Id (none) -> 54; MANUFACTURER Maxim Semiconductor -> (none); Manufacture (none) -> Analog Devices Inc./Maxim Integrated; Manufacture Part Number (none) -> MAX17048G+T10; Type (none) -> SMD
- U5: Distributor (none) -> LCSC; Distributor Link (none) -> https://www.lcsc.com/product-detail/Attitude-Sensor-Gyrosco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; Distributor Part Number (none) -> C95230; Id (none) -> 55; Manufacture (none) -> STMicroelectronics; Manufacture Part Number (none) -> LSM6DS3TR; Type (none) -> SMD
- U6: Distributor (none) -> LCSC; Distributor Link (none) -> https://www.lcsc.com/product-detail/WiFi-Modules_Espressif-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; Distributor Part Number (none) -> C3013941; Id (none) -> 56; Manufacture (none) -> Espressif Systems; Manufacture Part Number (none) -> ESP32-S3-MINI-1-N4R2; Type (none) -> SMD
- U7: AVAILABILITY Unavailable -> (none); DESCRIPTION L86 is an ultra-compact GNSS POT _Patch on Top_ module with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 -> (none); Distributor (none) -> Mouser; Distributor Link (none) -> https://www.mouser.co.id/ProductDetail/Quectel/L86-M33?qs=G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; Distributor Part Number (none) -> 277-L86-M33; Id (none) -> 57; MF Quectel -> (none); MP L86 -> (none); Manufacture (none) -> Quectel; Manufacture Part Number (none) -> L86-M33; PACKAGE None -> (none); PRICE None -> (none); Type (none) -> SMD
- Y1: footprint Crystal:Crystal_SMD_2012-2Pin_2.0x1.2mm -> Crystal:Crystal_SMD_3215-2Pin_3.2x1.5mm; Distributor (none) -> LCSC; Distributor Link (none) -> https://www.lcsc.com/product-detail/Crystals_Seiko-Epson-Q1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; Distributor Part Number (none) -> C32346; Id (none) -> 60; Manufacture (none) -> Seiko Epson; Manufacture Part Number (none) -> Q13FC1350000400; Type (none) -> SMD

Commit message: update design
Parts:
- added TP5: BOOT, TestPoint:TestPoint_Pad_D1.0mm, symbol Connector:TestPoint
- added TP6: RESET, TestPoint:TestPoint_Pad_D1.0mm, symbol Connector:TestPoint
- added TP7: TXD, TestPoint:TestPoint_Pad_D1.0mm, symbol Connector:TestPoint
- added TP8: RXD, TestPoint:TestPoint_Pad_D1.0mm, symbol Connector:TestPoint
- SW2: renamed from JP1; symbol Jumper:SolderJumper_2_Open -> Switch:SW_Push
Connections:
- net A7670_RX: now also U6.21 (GPIO17/U1TXD/ADC2_CH6); no longer U6.39 (U0TXD/GPIO43/CLK_OUT1)
- net A7670_TX: now also U6.22 (GPIO18/U1RXD/ADC2_CH7/CLK_OUT3); no longer U6.40 (U0RXD/GPIO44/CLK_OUT2)
- net ESP_BOOT: now also TP5.1
- net ESP_EN: now also TP6.1
- new net: TP7.1, U6.39 (U0TXD/GPIO43/CLK_OUT1)
- new net: TP8.1, U6.40 (U0RXD/GPIO44/CLK_OUT2)
- no-connect marks 12 -> 22
Other:
- note added: "- Acquisition: 30mA @VCC=V_BCKP=3.3V (GPS+GLONASS) - Tracking : 26mA @VCC=V_BCKP=3.3V (GPS+GLONASS) - Standby : 1mA @VCC=V_BCKP=3.3V - Backup : 7uA @V_BCKP=3.3V"
- note added: "- Sleep mode: 0.5µA - Hibernate mode: 4uA - Active mode: 23uA ( automatically switches to hibernate when low current )"
- note added: "LSM6DSOXTR Power Profile - ULP: @1.6Hz 4.4uA - OFF: 3uA"
- note added: "Light-sleep: 240uA Deep-sleep: 8uA"
- note added: "TODO: Change to LSM6DSOXTR"
- note added: "TODO: Change to XC6220 ( or something lower ) - PS Mode: 8uA"
- note added: "Vout = Vref*(1+(R1/R2)) Vref = 0.6V (Typical) Iq = 15uA"
- note removed: "5.5x8.5 cm"
- note removed: "Datasheet: https://datasheet.lcsc.com/lcsc/1810291810_Texas-Instruments-TPS62290DRVR_C129315.pdf"
- note removed: "Vout = Vref*(1+(R1/R2)) Vref = 0.6V (Typical)"
- moved on the sheet: Q2, R11, R12
