File: hardware/kicad/bwlc1a.kicad_sch (KiCad schematic)
At the start: 54 parts, among them J1 JST-2PH, J2 USB_C_Receptacle_USB2.0, J3 JTAG_10PIN, Q1 DMG3415UQ-7, Q2 S8050, SW1 EN_ESP, SW2 BOOT, U1 MCP73831-2-OT, U2 USBLC6-2SC6, U3 TPS62290DRVR, U4 MAX17048G+, U5 LSM6DS3, U6 ESP32-S3-MINI-1, U7 L86-M33, Y1 32.768 kHz

Commit message: wip
Parts:
- removed L1: 2.2u, Inductor_SMD:L_1008_2520Metric, symbol Device:L_Small
- removed U3: TPS62290DRVR, TPS62290DRVR:SON65P200X200X80-7N, symbol TPS62290DRVR:TPS62290DRVR
- added C22: 100n, Capacitor_SMD:C_0402_1005Metric, symbol Device:C_Small
- added C23, C26, C39, C41: 10u, Capacitor_SMD:C_0603_1608Metric, symbol Device:C_Small
- added C24, C40: DNP, Capacitor_Tantalum_SMD:CP_EIA-3528-15_AVX-H, symbol Device:C_Polarized_Small
- added F2: 0.75A, Fuse:Fuse_0805_2012Metric, symbol Device:Polyfuse_Small
- added FB2: MMZ1608B601CTAH0, Inductor_SMD:L_0603_1608Metric, symbol Device:FerriteBead_Small
- added R15, R18: 1M, Resistor_SMD:R_0402_1005Metric, symbol Device:R_Small
- added U10: RT9080-33GJ5, Package_TO_SOT_SMD:SOT-23-5_HandSoldering, symbol bwcl1a:RT9080
- added U11, U3: TPS22917DBVR, Package_TO_SOT_SMD:SOT-23-6, symbol bwcl1a:TPS22917DBVR
- C3: value 22p -> 10n; Distributor LCSC -> (none); Distributor Link https://www.lcsc.com/product-detail/Multilayer-Ceramic-Capa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 -> (none); Distributor Part Number C70464 -> (none); Id 2 -> (none); Manufacture Samsung Electro-Mechanics -> (none); Manufacture Part Number CL05C220JB5NNNC -> (none); Manufacturer (none) -> YAGEO; Part Description (none) -> Ceramic Capacitor 10nF 10% 50V X7R; Part Number (none) -> CC0402KRX7R9BB103; Type SMD -> (none)
- R3: value 453k -> DNP; footprint Resistor_SMD:R_0402_1005Metric -> Resistor_SMD:R_0603_1608Metric; Distributor LCSC -> (none); Distributor Link https://www.lcsc.com/product-detail/Chip-Resistor-Surface-M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 -> (none); Distributor Part Number C27009 -> (none); Id 36 -> (none); Manufacture UNI-ROYAL(Uniroyal Elec) -> (none); Manufacture Part Number 0402WGF4533TCE -> (none); Type SMD -> (none)
- R7: value 100k -> DNP; footprint Resistor_SMD:R_0402_1005Metric -> Resistor_SMD:R_0603_1608Metric; Distributor LCSC -> (none); Distributor Link https://www.lcsc.com/product-detail/Chip-Resistor-Surface-M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 -> (none); Distributor Part Number C25741 -> (none); Id 38 -> (none); Manufacture UNI-ROYAL(Uniroyal Elec) -> (none); Manufacture Part Number 0402WGF1003TCE -> (none); Type SMD -> (none)
Connections:
- net +3.3V: now also U10.5 (VOUT); no longer C3.1, R3.2
- net +BATT: now also C23.1, C24.1, C39.1, C40.1, U11.1 (VIN), U3.1 (VIN)
- net GND: now also C3.2, C22.2, C23.2, C26.2, C39.2, C41.2, R15.1, R18.1, U10.2 (VSS), U11.2 (GND), U3.2 (GND); no longer R7.1
- net USB_D+: no longer J2.A6 (D+), J2.B6 (D+), U2.1 (I/O1)
- net USB_D-: no longer J2.A7 (D-), J2.B7 (D-), U2.3 (I/O2)
- net VBUS: now also F2.2; no longer J2.A4 (VBUS), J2.A9 (VBUS), J2.B4 (VBUS), J2.B9 (VBUS)
- net EN_VBAT_GPS: now reaches U6.5 (GPIO1/TOUCH1/ADC1_CH0)
- net EN_VBAT_GPS: now also R18.2, U11.3 (ON)
- net EN_MIC29302 renamed EN_VBAT_CELL
- net EN_VBAT_CELL: now also R15.2, U3.3 (ON)
- removed net TPS_FB: C3.2, R3.1, R7.2
- net TPS_VIN: no longer names the net of C5.1, D2.1 (K), Q1.3 (S)
- net TPS_VIN: now also U10.1 (VIN), U10.3 (CE)
- net VDD_BAT renamed VBAT_GPS
- net VBAT_GPS: now also R7.2, C41.1, U11.6 (VOUT)
- new net: C24.2, U3.4 (CT)
- new net: R3.1, U3.5 (QOD)
- new net: C22.1, F2.1, FB2.2
- new net: C3.1, FB2.1, J2.A4 (VBUS), J2.A9 (VBUS), J2.B4 (VBUS), J2.B9 (VBUS)
- new net: C40.2, U11.4 (CT)
- new net: R7.1, U11.5 (QOD)
- new net USB_D_IN+: J2.A6 (D+), J2.B6 (D+), U2.1 (I/O1)
- new net USB_D_IN-: J2.A7 (D-), J2.B7 (D-), U2.3 (I/O2)
- new net VBAT_CELL: C26.1, R3.2, U3.6 (VOUT)
Other:
- sheet bwlc1a_A7670C renamed a7670
- sheet a7670: file bwlc1a_A7670C.kicad_sch -> a7670.kicad_sch
- note added: "3V3 Volatege Regulator (LDO)"
- note added: "Battery Fuel Gauge"
- note added: "Charge Rate: 1A"
- note added: "Iq: 2uA"
- note added: "Load Switch for Cell & GPS"
- note removed: "Fuel Gauge"
- note removed: "R1"
- note removed: "R2"
- note removed: "Step Down/LDO 3V3"
- note removed: "TODO: Change to XC6220 ( or something lower ) - PS Mode: 8uA"
- note removed: "Vout = 3.318V"
- note removed: "Vout = Vref*(1+(R1/R2)) Vref = 0.6V (Typical) Iq = 15uA"
- moved on the sheet: C1, C2, C4, C5, D1, D2, D3, J1, J2, Q1, R1, R2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

Commit message: wip: revision 2
Parts:
- added TP9: VBUS_IN, TestPoint:TestPoint_Pad_D1.0mm, symbol Connector:TestPoint
- U5: value LSM6DS3 -> LSM6DSOTR; Distributor Link https://www.lcsc.com/product-detail/Attitude-Sensor-Gyrosco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 -> https://datasheet.lcsc.com/lcsc/2108070730_STMicroelectroni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; Distributor Part Number C95230 -> C2655100; Id 55 -> (none); Manufacture STMicroelectronics -> (none); Manufacture Part Number LSM6DS3TR -> (none); Manufacturer (none) -> STMicroelectronics; Manufacturer Part Number (none) -> LSM6DSOTR; Part Description (none) -> LGA-14 Attitude Sensor/Gyroscope ROHS; Type SMD -> (none)
Connections:
- net at C3.1, FB2.1, J2.A4 (VBUS)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: now also TP9.1
Other:
- note removed: "TODO: Change to LSM6DSOXTR"
Changed lines of the file:
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@@
   (junction (at 331.47 43.18) (diameter 0) (color 0 0 0 0)
   )
+  (junction (at 53.34 34.29) (diameter 0) (color 0 0 0 0)
+  )
   (junction (at 132.715 193.675) (diameter 0) (color 0 0 0 0)
   )
@@
     (stroke (width 0) (type default))
   )
-  (wire (pts (xy 45.72 34.29) (xy 64.77 34.29))
+  (wire (pts (xy 45.72 34.29) (xy 53.34 34.29))
     (stroke (width 0) (type default))
   )
@@
     (stroke (width 0) (type default))
   )
+  (wire (pts (xy 53.34 28.575) (xy 53.34 34.29))
+    (stroke (width 0) (type default))
+  )
   (wire (pts (xy 291.465 58.42) (xy 291.465 61.595))
     (stroke (width 0) (type default))
@@
     (stroke (width 0) (type default))
   )
+  (wire (pts (xy 53.34 34.29) (xy 64.77 34.29))
+    (stroke (width 0) (type default))
+  )
   (wire (pts (xy 28.575 247.65) (xy 28.575 249.555))
     (stroke (width 0) (type default))
@@
     (effects (font (size 2.5 2.5) (thickness 0.254) bold) (justify left bottom))
   )
-  (text "TODO: Change to LSM6DSOXTR" (at 245.11 190.5 0)
-    (effects (font (size 1.27 1.27)) (justify left bottom))
-  )
   (text "Battery Fuel Gauge" (at 280.67 89.535 0)
     (effects (font (size 2.5 2.5) (thickness 0.254) bold) (justify left bottom))
@@
       (effects (font (size 1.27 1.27)) hide)
     )
+    (property "Part Description" "" (at 209.55 47.625 0)
+      (effects (font (size 1.27 1.27)) hide)
+    )
+    (property "Manufacturer" "" (at 209.55 47.625 0)
+      (effects (font (size 1.27 1.27)) hide)
+    )
+    (property "Manufacturer Part Number" "" (at 209.55 47.625 0)
+      (effects (font (size 1.27 1.27)) hide)
+    )
     (pin "1")
     (pin "2")
@@
       (effects (font (size 1.27 1.27)) (justify left))
     )
-    (property "Value" "LSM6DS3" (at 236.2709 171.45 0)
+    (property "Value" "LSM6DSOTR" (at 236.2709 171.45 0)
       (effects (font (size 1.27 1.27)) (justify left))
     )
@@
       (effects (font (size 1.27 1.27)) (justify left) hide)
     )
-    (property "Datasheet" "https://www.st.com/resource/en/datasheet/lsm6ds3tr-c.pdf" (at 236.855 170.18 0)
-      (effects (font (size 1.27 1.27)) hide)
-    )
-    (property "Description" "LGA-14 Attitude Sensor/Gyroscope ROHS" (at 234.315 153.67 0)
-      (effects (font (size 1.27 1.27)) hide)
-    )
-    (property "Distributor" "LCSC" (at 234.315 153.67 0)
+    (property "Datasheet" "https://datasheet.lcsc.com/lcsc/2108070730_STMicroelectronics-LSM6DSOTR_C2655100.pdf" (at 236.855 170.18 0)
       (effects (font (size 1.27 1.27)) hide)
     )
-    (property "Distributor Link" "https://www.lcsc.com/product-detail/Attitude-Sensor-Gyroscope_STMicroelectronics-LSM6DS3TR_C95230.html" (at 234.315 153.67 0)
+    (property "Part Description" "LGA-14 Attitude Sensor/Gyroscope ROHS" (at 234.315 153.67 0)
       (effects (font (size 1.27 1.27)) hide)
     )
-    (property "Distributor Part Number" "C95230" (at 234.315 153.67 0)
+    (property "Manufacturer" "STMicroelectronics" (at 234.315 153.67 0)
       (effects (font (size 1.27 1.27)) hide)
     )
-    (property "Id" "55" (at 234.315 153.67 0)
+    (property "Manufacturer Part Number" "LSM6DSOTR" (at 234.315 153.67 0)
       (effects (font (size 1.27 1.27)) hide)
     )
-    (property "Manufacture" "STMicroelectronics" (at 234.315 153.67 0)
+    (property "Distributor" "LCSC" (at 234.315 153.67 0)
       (effects (font (size 1.27 1.27)) hide)
     )
-    (property "Manufacture Part Number" "LSM6DS3TR" (at 234.315 153.67 0)
+    (property "Distributor Part Number" "C2655100" (at 234.315 153.67 0)
       (effects (font (size 1.27 1.27)) hide)
     )
-    (property "Type" "SMD" (at 234.315 153.67 0)
+    (property "Distributor Link" "https://datasheet.lcsc.com/lcsc/2108070730_STMicroelectronics-LSM6DSOTR_C2655100.pdf" (at 234.315 153.67 0)
       (effects (font (size 1.27 1.27)) hide)
     )
@@
         )
       )
+    )
+  )
+  (symbol (lib_id "Connector:TestPoint") (at 53.34 28.575 0) (unit 1)
+    (in_bom yes) (on_board yes) (dnp no)
+    (property "Reference" "TP9" (at 48.895 22.86 0)
+      (effects (font (size 1.27 1.27)) (justify left))
+    )
+    (property "Value" "VBUS_IN" (at 53.975 22.86 0)
+      (effects (font (size 1.27 1.27)) (justify left))
+    )
+    (property "Footprint" "TestPoint:TestPoint_Pad_D1.0mm" (at 58.42 28.575 0)
+      (effects (font (size 1.27 1.27)) hide)
+    )
+    (property "Datasheet" "~" (at 58.42 28.575 0)
+      (effects (font (size 1.27 1.27)) hide)
+    )
+    (property "Part Description" "" (at 53.34 28.575 0)
+      (effects (font (size 1.27 1.27)) hide)
+    )
+    (property "Manufacturer" "" (at 53.34 28.575 0)
+      (effects (font (size 1.27 1.27)) hide)
+    )
+    (property "Manufacturer Part Number" "" (at 53.34 28.575 0)
+      (effects (font (size 1.27 1.27)) hide)
+    )
+    (property "Distributor" "" (at 53.34 28.575 0)
+      (effects (font (size 1.27 1.27)) hide)
+    )
+    (property "Distributor Part Number" "" (at 53.34 28.575 0)
+      (effects (font (size 1.27 1.27)) hide)
+    )
+    (property "Distributor Link" "" (at 53.34 28.575 0)
+      (effects (font (size 1.27 1.27)) hide)
+    )
+    (pin "1")
+    (instances
+      (project "bwlc1a"
+        (path "/388039b1-99cc-430f-bd4a-010573fde798"
+          (reference "TP9") (unit 1)
+        )
+      )
