File: hardware/kicad/bwlc1a.kicad_sch (KiCad schematic)
At the start: 0 parts

Commit message: wip: revision 2
Other:
- sheet Battery ports: added +BATT; removed none
- sheet Power ports: added +3V3, +BATT, +BATT_CELL, 2V8_GNSS, 3V3_GNSS, EN_CELL, EN_GNSS, VBUS; removed none
- sheet USB and Charger ports: added +BATT, USB_D+, USB_D-, VBUS; removed none
Changed lines of the file:
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@@
     )
   )
-  (sheet (at 36.83 34.925) (size 76.2 33.02) (fields_autoplaced)
+  (sheet (at 45.085 104.775) (size 31.75 16.51) (fields_autoplaced)
     (stroke (width 0.1524) (type solid))
     (fill (color 0 0 0 0.0000))
-    (property "Sheetname" "USB and Charger" (at 36.83 34.2134 0)
+    (property "Sheetname" "USB and Charger" (at 45.085 104.0634 0)
       (effects (font (size 1.27 1.27)) (justify left bottom))
     )
-    (property "Sheetfile" "usb_and_charger.kicad_sch" (at 36.83 68.5296 0)
+    (property "Sheetfile" "usb_and_charger.kicad_sch" (at 45.085 121.8696 0)
       (effects (font (size 1.27 1.27)) (justify left top))
+    )
+    (pin "USB_D+" output (at 76.835 117.475 0)
+      (effects (font (size 1.27 1.27)) (justify right))
+    )
+    (pin "USB_D-" output (at 76.835 114.935 0)
+      (effects (font (size 1.27 1.27)) (justify right))
+    )
+    (pin "VBUS" output (at 76.835 110.49 0)
+      (effects (font (size 1.27 1.27)) (justify right))
+    )
+    (pin "+BATT" bidirectional (at 76.835 107.95 0)
+      (effects (font (size 1.27 1.27)) (justify right))
     )
     (instances
@@
     )
   )
-  (sheet (at 38.1 129.54) (size 69.85 30.48) (fields_autoplaced)
+  (sheet (at 46.99 130.175) (size 29.845 30.48) (fields_autoplaced)
     (stroke (width 0.1524) (type solid))
     (fill (color 0 0 0 0.0000))
-    (property "Sheetname" "Power" (at 38.1 128.8284 0)
+    (property "Sheetname" "Power" (at 46.99 129.4634 0)
       (effects (font (size 1.27 1.27)) (justify left bottom))
     )
-    (property "Sheetfile" "power.kicad_sch" (at 38.1 160.6046 0)
+    (property "Sheetfile" "power.kicad_sch" (at 46.99 161.2396 0)
       (effects (font (size 1.27 1.27)) (justify left top))
+    )
+    (pin "3V3_GNSS" output (at 76.835 154.305 0)
+      (effects (font (size 1.27 1.27)) (justify right))
+    )
+    (pin "2V8_GNSS" output (at 76.835 156.845 0)
+      (effects (font (size 1.27 1.27)) (justify right))
+    )
+    (pin "EN_GNSS" input (at 76.835 151.765 0)
+      (effects (font (size 1.27 1.27)) (justify right))
+    )
+    (pin "VBUS" input (at 76.835 138.43 0)
+      (effects (font (size 1.27 1.27)) (justify right))
+    )
+    (pin "+3V3" output (at 76.835 133.35 0)
+      (effects (font (size 1.27 1.27)) (justify right))
+    )
+    (pin "+BATT" input (at 76.835 135.89 0)
+      (effects (font (size 1.27 1.27)) (justify right))
+    )
+    (pin "+BATT_CELL" output (at 76.835 146.05 0)
+      (effects (font (size 1.27 1.27)) (justify right))
+    )
+    (pin "EN_CELL" input (at 76.835 143.51 0)
+      (effects (font (size 1.27 1.27)) (justify right))
     )
     (instances
@@
     )
   )
-  (sheet (at 36.195 76.2) (size 68.58 45.72) (fields_autoplaced)
+  (sheet (at 52.705 76.2) (size 23.495 17.78) (fields_autoplaced)
     (stroke (width 0.1524) (type solid))
     (fill (color 0 0 0 0.0000))
-    (property "Sheetname" "Battery" (at 36.195 75.4884 0)
+    (property "Sheetname" "Battery" (at 52.705 75.4884 0)
       (effects (font (size 1.27 1.27)) (justify left bottom))
     )
-    (property "Sheetfile" "battery.kicad_sch" (at 36.195 122.5046 0)
+    (property "Sheetfile" "battery.kicad_sch" (at 52.705 94.5646 0)
       (effects (font (size 1.27 1.27)) (justify left top))
     )
+    (pin "+BATT" bidirectional (at 76.2 85.09 0)
+      (effects (font (size 1.27 1.27)) (justify right))
+    )
     (instances

Commit message: wip: revision 2
Other:
- sheet Main Controller ports: added +3V3, CELL_EN, CELL_PWRKEY, CELL_RESET, CELL_RXD, CELL_STATUS, CELL_TXD, FG_INT, FG_SCL, FG_SDA, GNSS_EN, GNSS_FO, GNSS_RESET, GNSS_RXD, GNSS_TXD, GNSS_VBCKP_EN, IMU_INT, IMU_SCL, IMU_SDA, USB_D+, USB_D-; removed none
- sheet Power ports: added CELL_BATT, CELL_EN, GNSS_2V8, GNSS_3V3, GNSS_EN, GNSS_VBCKP, GNSS_VBCKP_EN; removed +BATT_CELL, 2V8_GNSS, 3V3_GNSS, EN_CELL, EN_GNSS
- sheet Sensors ports: added +3V3, +BATT, FG_INT, FG_SCL, FG_SDA, IMU_INT, IMU_SCL, IMU_SDA; removed none

Commit message: wip: revision 2
Other:
- sheet GNSS ports: added +BATT, GNSS_2V8, GNSS_3V3, GNSS_ANT, GNSS_FO, GNSS_RESET, GNSS_RXD, GNSS_SDBY, GNSS_TXD, GNSS_VBCKP; removed none
- sheet Main Controller ports: added GNSS_SDBY, SCL, SDA; removed FG_SCL, FG_SDA, IMU_SCL, IMU_SDA
- sheet Sensors ports: added SCL, SDA; removed FG_SCL, FG_SDA, IMU_SCL, IMU_SDA

Commit message: wip: revision 2
Other:
- added sheet Antenna (antenna.kicad_sch)
- sheet Cellular ports: added CELL_ANT, CELL_BATT, CELL_PWRKEY, CELL_RESET, CELL_RXD, CELL_STATUS, CELL_TXD; removed none

Commit message: add page info
Other:
- company: (none) -> Teapot Laboratories
- title: (none) -> Teapotlabs BWLC1A
Changed lines of the file:
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@@
 	(generator_version "8.0")
 	(paper "A4")
+	(title_block
+		(title "Teapotlabs BWLC1A")
+		(date "2024-05-17")
+		(rev "1")
+		(company "Teapot Laboratories")
+	)
 	(junction
 		(at 75.565 58.42)
