File: hardware/kicad/usb_and_charger.kicad_sch (KiCad schematic)
At the start: 15 parts, among them J2 USB_C_Receptacle_USB2.0, U1 MCP73831-2-OT, U2 USBLC6-2SC6

Commit message: wip: revision 2
Connections:
- net USB_D_IN+ renamed D_IN+
- net USB_D_IN- renamed D_IN-
Other:
- note added: "Battery Charger"
- note added: "Charge LED"
- note added: "Sheets Connection"
- note added: "USB trace is less than Critical Length (2.4 inch) for USB2.0 Full-speed specification. No need for impedance control."
- note added: "USB-C and ESD Protection"
- note removed: "1-Cell LiPo Charger"
- note removed: "USB C + ESD"
- moved on the sheet: C1, C2, C22, C3, D1, F2, FB2, J2, R1, R2, R4, R5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

Commit message: wip: revision 2
Changed lines of the file:
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@@
     (effects (font (size 1.27 1.27)) (justify left))
   )
-  (hierarchical_label "USB_D-" (shape output) (at 131.445 101.6 0) (fields_autoplaced)
+  (hierarchical_label "USB_D-" (shape bidirectional) (at 131.445 101.6 0) (fields_autoplaced)
     (effects (font (size 1.27 1.27)) (justify left))
   )
-  (hierarchical_label "USB_D+" (shape output) (at 111.125 101.6 180) (fields_autoplaced)
+  (hierarchical_label "USB_D+" (shape bidirectional) (at 111.125 101.6 180) (fields_autoplaced)
     (effects (font (size 1.27 1.27)) (justify right))
   )

Commit message: PCB Layout Update
Parts:
- added D9: ESD5651N, Capacitor_SMD:C_0402_1005Metric, symbol Device:D_TVS
Connections:
- net D_IN+: now also U2.3 (I/O2); no longer U2.1 (I/O1)
- net D_IN-: now also U2.1 (I/O1); no longer U2.3 (I/O2)
- net GND: now also D9.1 (A1)
- net USB_D+: now also U2.4 (I/O2); no longer U2.6 (I/O1)
- net USB_D-: now also U2.6 (I/O1); no longer U2.4 (I/O2)
- net at C3.1, FB2.1, J2.A4 (VBUS)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: now also D9.2 (A2)
Other:
- moved on the sheet: C22, C3, F2, FB2

Commit message: update to KiCAD 8 and add cell power regulator
Parts:
- renumbered C3 to C1, C22 to C2, C1 to C3, C2 to C4, D9 to D6, F2 to F1, J2 to J1, R5 to R3, U2 to U1, U1 to U2

Commit message: finalizing usb and charger bom
Parts:
- C1: Distributor (none) -> LCSC; Distributor Link (none) -> https://www.lcsc.com/product-detail/Multilayer-Ceramic-Capa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; Distributor Part Number (none) -> C60133; Manufacturer Part Number (none) -> CC0402KRX7R9BB103; Part Description Ceramic Capacitor 10nF 10% 50V X7R -> (none); Part Number CC0402KRX7R9BB103 -> (none)
- C2: Distributor (none) -> LCSC; Distributor Link (none) -> https://www.lcsc.com/product-detail/Multilayer-Ceramic-Capa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; Distributor Part Number (none) -> C129131; Manufacturer Part Number (none) -> CC0402KRX5R6BB104; Part Description Ceramic Capacitor 100nF 10% 10V X5R -> (none); Part Number CC0402KRX5R6BB104 -> (none)
- C3, C4: Id 1 -> (none); Manufacture Samsung Electro-Mechanics -> (none); Manufacture Part Number CL10A106KP8NNNC -> (none); Manufacturer (none) -> Samsung Electro-Mechanics; Manufacturer Part Number (none) -> CL10A106KP8NNNC; Type SMD -> (none)
- D1: value Orange -> E6C0603SEAC1UDA; Id 17 -> (none); Manufacture EKINGLUX -> (none); Manufacture Part Number E6C0603SEAC1UDA -> (none); Manufacturer (none) -> EKINGLUX; Manufacturer Part Number (none) -> E6C0603SEAC1UDA; Type SMD -> (none)
- D6: footprint Capacitor_SMD:C_0402_1005Metric -> Diode_SMD:D_SOD-882; Distributor (none) -> LCSC; Distributor Part Number (none) -> C5173251; Manufacturer (none) -> Leiditech; Manufacturer Part Number (none) -> ESD5651N
- F1: value 0.75A -> SMD0805P075TF; Distributor (none) -> LCSC; Distributor Link (none) -> https://www.lcsc.com/product-detail/Resettable-Fuses_RUILON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; Distributor Part Number (none) -> C20979; Manufacturer RUILON -> RUILON(Shenzhen Ruilongyuan Elec); Manufacturer Part Number (none) -> SMD0805P075TF; Part Description Resettable Fuses 6V 750mA 40A 1.5A -> (none); Part Number SMD0805P075TF -> (none)
- FB2: Distributor (none) -> LCSC; Distributor Link (none) -> https://www.lcsc.com/product-detail/Ferrite-Beads_TDK-MMZ16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; Distributor Part Number (none) -> C97120; Manufacturer Part Number (none) -> MMZ1608B601CTAH0; Part Number MMZ1608B601CTAH0 -> (none)
- J1: Id 25 -> (none); Manufacture Korean Hroparts Elec -> (none); Manufacture Part Number TYPE-C-31-M-12 -> (none); Manufacturer (none) -> Korean Hroparts Elec; Manufacturer Part Number (none) -> TYPE-C-31-M-12; Type SMD -> (none)
- R1, R2: Id 35 -> (none); Manufacture UNI-ROYAL(Uniroyal Elec) -> (none); Manufacture Part Number 0402WGF5101TCE -> (none); Manufacturer (none) -> UNI-ROYAL(Uniroyal Elec); Manufacturer Part Number (none) -> 0402WGF5101TCE; Type SMD -> (none)
- R3: value 1k -> 2k; Distributor Link https://www.lcsc.com/product-detail/Chip-Resistor-Surface-Mount_UNI-ROYAL-Uniroyal-Elec-0402WGJ0102TCE_C25543.html -> https://www.lcsc.com/product-detail/Chip-Resistor-Surface-Mount_YAGEO-RC0402FR-072KL_C60488.html; Distributor Part Number C25543 -> C60488; Id 37 -> (none); Manufacture UNI-ROYAL(Uniroyal Elec) -> (none); Manufacture Part Number 0402WGJ0102TCE -> (none); Manufacturer (none) -> YAGEO; Manufacturer Part Number (none) -> RC0402FR-072KL; Type SMD -> (none)
- R4: Id 37 -> (none); Manufacture UNI-ROYAL(Uniroyal Elec) -> (none); Manufacture Part Number 0402WGJ0102TCE -> (none); Manufacturer (none) -> UNI-ROYAL(Uniroyal Elec); Manufacturer Part Number (none) -> 0402WGJ0102TCE; Type SMD -> (none)
- U1: Id 52 -> (none); Manufacture TECH PUBLIC -> (none); Manufacture Part Number USBLC6-2SC6 -> (none); Manufacturer (none) -> TECH PUBLIC; Manufacturer Part Number (none) -> USBLC6-2SC6; Type SMD -> (none)
- U2: Id 51 -> (none); Manufacture Microchip Tech -> (none); Manufacture Part Number MCP73831T-2ATI/OT -> (none); Manufacturer (none) -> Microchip Tech; Manufacturer Part Number (none) -> MCP73831T-2ATI/OT; Type SMD -> (none)
Other:
- note added: "750mA"
- note added: "Orange Charge LED"
- note added: "USB trace is less than Critical Length (2.4 inch) for USB2.0 Full-speed specification. Impedance control is not critical"
- note removed: "Charge LED"
- note removed: "USB trace is less than Critical Length (2.4 inch) for USB2.0 Full-speed specification. No need for impedance control."
