File: hardware/kicad/usb_and_charger.kicad_sch (KiCad schematic)
At the start: 16 parts, among them J1 USB_C_Receptacle_USB2.0, U1 USBLC6-2SC6, U2 MCP73831-2-OT

Commit message: update bill of materials
Parts:
- C2: Distributor Link https://www.lcsc.com/product-detail/Multilayer-Ceramic-Capacitors-MLCC-SMD-SMT_YAGEO-CC0402KRX5R6BB104_C129131.html -> https://www.lcsc.com/product-detail/Multilayer-Ceramic-Capacitors-MLCC-SMD-SMT_Samsung-Electro-Mechanics-CL05B104KO5NNNC_C1525.html; Distributor Part Number C129131 -> C1525; Manufacturer YAGEO -> Samsung Electro-Mechanics; Manufacturer Part Number CC0402KRX5R6BB104 -> CL05B104KO5NNNC
- R1, R2: value 5.1k -> 5k1
Other:
- note added: "Charge Rate: 500mA"
- note removed: "Charge Rate: 1A"
Changed lines of the file:
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@@
 		)
 	)
-	(text "Charge Rate: 1A"
+	(text "Charge Rate: 500mA"
 		(exclude_from_sim no)
 		(at 170.815 98.425 0)
@@
 			)
 		)
-		(property "Description" " 62.5mW Thick Film Resistors 50V ±100ppm/℃ ±1% 2kΩ 0402 Chip Resistor - Surface Mount ROHS"
+		(property "Description" "62.5mW Thick Film Resistors 50V ±100ppm/℃ ±1% 2kΩ 0402 Chip Resistor - Surface Mount ROHS"
 			(at 177.8 86.36 0)
 			(effects
@@
 			)
 		)
-		(property "Value" "5.1k"
+		(property "Value" "5k1"
 			(at 100.965 78.105 90)
 			(effects
@@
 			)
 		)
-		(property "Datasheet" "https://www.lcsc.com/datasheet/lcsc_datasheet_1912111437_YAGEO-CC0402KRX5R6BB104_C129131.pdf"
+		(property "Datasheet" "https://www.lcsc.com/datasheet/lcsc_datasheet_2304140030_Samsung-Electro-Mechanics-CL05B104KO5NNNC_C1525.pdf"
 			(at 132.715 73.025 0)
 			(effects
@@
 			)
 		)
-		(property "Description" "10V 100nF X5R ±10% 0402 Multilayer Ceramic Capacitors MLCC - SMD/SMT ROHS"
+		(property "Description" "16V 100nF X7R ±10% 0402 Multilayer Ceramic Capacitors MLCC - SMD/SMT ROHS"
 			(at 132.715 73.025 0)
 			(effects
@@
 			)
 		)
-		(property "Manufacturer" "YAGEO"
+		(property "Manufacturer" "Samsung Electro-Mechanics"
 			(at 132.715 73.025 0)
 			(effects
@@
 			)
 		)
-		(property "Manufacturer Part Number" "CC0402KRX5R6BB104"
+		(property "Manufacturer Part Number" "CL05B104KO5NNNC"
 			(at 132.715 73.025 0)
 			(effects
@@
 			)
 		)
-		(property "Distributor Part Number" "C129131"
+		(property "Distributor Part Number" "C1525"
 			(at 132.715 73.025 0)
 			(effects
@@
 			)
 		)
-		(property "Distributor Link" "https://www.lcsc.com/product-detail/Multilayer-Ceramic-Capacitors-MLCC-SMD-SMT_YAGEO-CC0402KRX5R6BB104_C129131.html"
+		(property "Distributor Link" "https://www.lcsc.com/product-detail/Multilayer-Ceramic-Capacitors-MLCC-SMD-SMT_Samsung-Electro-Mechanics-CL05B104KO5NNNC_C1525.html"
 			(at 132.715 73.025 0)
 			(effects
@@
 			)
 		)
-		(property "Description" " 6V 750mA 40A 1.5A 0805 Resettable Fuses ROHS"
+		(property "Description" "6V 750mA 40A 1.5A 0805 Resettable Fuses ROHS"
 			(at 138.43 68.58 0)
 			(effects
@@
 			)
 		)
-		(property "Value" "5.1k"
+		(property "Value" "5k1"
 			(at 100.965 71.755 90)
 			(effects

Commit message: add page info
Other:
- company: (none) -> Teapot Laboratories
- title: (none) -> USB and Charger
Changed lines of the file:
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@@
 	(generator_version "8.0")
 	(paper "A4")
+	(title_block
+		(title "USB and Charger")
+		(date "2024-05-17")
+		(rev "1")
+		(company "Teapot Laboratories")
+	)
 	(junction
 		(at 120.015 68.58)

Commit message: Update for PCB Layout
Parts:
- renumbered C1 to C30, C2 to C31, C3 to C32, C4 to C33, D6 to D10, D1 to D11, J1 to J3, R1 to R28, R2 to R29, R4 to R30, R3 to R31, TP9 to TP19, U2 to U7, U1 to U8

Commit message: Update Production File
Parts:
- D10: Distributor Link https://www.lcsc.com/product-detail/span-style-background-color-ff0-ESD-span-Protection-Devices_Leiditech-ESD5651N_C5173251.html -> https://www.lcsc.com/product-detail/span-style-background-color-ff0-ESD-span-and-Surge-Protection-TVS-span-style-background-color-ff0-ESD-span_TECH-PUBLIC-ESD5651N_C5342369.html; Distributor Part Number C5173251 -> C5342369; Manufacturer Leiditech -> TECH PUBLIC
- renumbered C30 to C32, C31 to C33, C32 to C34, C33 to C35, R28 to R20, R29 to R21, R30 to R22, R31 to R23, TP19 to TP32, U7 to U8, U8 to U9
