File: hardware/kicad/gnss.kicad_sch (KiCad schematic)
At the start: 14 parts, among them Q2 PMV32UP, Q7 DMG1012UW, U11 L76L-M33, U13 TXB0106PWR

Commit message: wip: revision 2
Parts:
- added JP1: SolderJumper_3_Bridged12, symbol Jumper:SolderJumper_3_Bridged12
Connections:
- net +BATT: now also JP1.3 (B)
- net GNSS_VBCKP: now also JP1.1 (A); no longer C42.1, C43.1, C44.1, U11.6 (V_BCKP)
- new net: C42.1, C43.1, C44.1, JP1.2 (C), U11.6 (V_BCKP)
Changed lines of the file:
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@@
+    (stroke (width 0) (type default))
+  )
+  (wire (pts (xy 163.83 82.55) (xy 163.83 84.455))
+    (stroke (width 0) (type default))
+  )
+  (wire (pts (xy 163.83 84.455) (xy 164.465 84.455))
     (stroke (width 0) (type default))
   )
@@
     )
   )
-  (global_label "GNSS_VBCKP" (shape input) (at 160.02 77.47 0) (fields_autoplaced)
-    (effects (font (size 1.27 1.27)) (justify left))
-    (property "Intersheetrefs" "${INTERSHEET_REFS}" (at 175.0815 77.47 0)
+  (global_label "GNSS_VBCKP" (shape input) (at 164.465 84.455 0) (fields_autoplaced)
+    (effects (font (size 1.27 1.27)) (justify left))
+    (property "Intersheetrefs" "${INTERSHEET_REFS}" (at 179.5265 84.455 0)
       (effects (font (size 1.27 1.27)) (justify left) hide)
     )
@@
     )
   )
+  (symbol (lib_id "Jumper:SolderJumper_3_Bridged12") (at 163.83 77.47 270) (mirror x) (unit 1)
+    (in_bom yes) (on_board yes) (dnp no)
+    (property "Reference" "JP1" (at 166.37 78.74 90)
+      (effects (font (size 1.27 1.27)) (justify left))
+    )
+    (property "Value" "SolderJumper_3_Bridged12" (at 166.37 76.2 90)
+      (effects (font (size 1.27 1.27)) (justify left))
+    )
+    (property "Footprint" "" (at 163.83 77.47 0)
+      (effects (font (size 1.27 1.27)) hide)
+    )
+    (property "Datasheet" "~" (at 163.83 77.47 0)
+      (effects (font (size 1.27 1.27)) hide)
+    )
+    (pin "1")
+    (pin "2")
+    (pin "3")
+    (instances
+      (project "bwlc1a"
+        (path "/388039b1-99cc-430f-bd4a-010573fde798/6908783c-0fa0-46ec-befb-a4abfbcaa74b"
+          (reference "JP1") (unit 1)
+        )
+      )
+    )
+  )
   (symbol (lib_id "power:GND") (at 250.19 111.125 0) (mirror y) (unit 1)
     (in_bom yes) (on_board yes) (dnp no)
@@
         )
       )
+    )
+  )
+  (symbol (lib_id "power:+BATT") (at 163.83 72.39 0) (unit 1)
+    (in_bom yes) (on_board yes) (dnp no) (fields_autoplaced)
+    (property "Reference" "#PWR0104" (at 163.83 76.2 0)
+      (effects (font (size 1.27 1.27)) hide)
+    )
+    (property "Value" "+BATT" (at 163.83 68.58 0)
+      (effects (font (size 1.27 1.27)))
+    )
+    (property "Footprint" "" (at 163.83 72.39 0)
+      (effects (font (size 1.27 1.27)) hide)
+    )
+    (property "Datasheet" "" (at 163.83 72.39 0)
+      (effects (font (size 1.27 1.27)) hide)
+    )
+    (pin "1")
+    (instances
+      (project "bwlc1a"
+        (path "/388039b1-99cc-430f-bd4a-010573fde798"
+          (reference "#PWR0104") (unit 1)
+        )
+        (path "/388039b1-99cc-430f-bd4a-010573fde798/6908783c-0fa0-46ec-befb-a4abfbcaa74b"
+          (reference "#PWR0103") (unit 1)
+        )
+      )

Commit message: wip: revision 2
Parts:
- removed Q2: PMV32UP, Package_TO_SOT_SMD:SOT-23, symbol Device:Q_PMOS_GSD
- removed Q7: DMG1012UW, Package_TO_SOT_SMD:SOT-323_SC-70, symbol Device:Q_NMOS_GSD
- removed R21, R33: 1M, Resistor_SMD:R_0603_1608Metric, symbol Device:R_Small

Commit message: wip: revision 2
Connections:
- net 2V8_GPS renamed GNSS_2V8
- net 3V3_GPS renamed GNSS_3V3
- net GPS_ANT renamed GNSS_ANT
- net GPS_HV_FO renamed GNSS_FO
- net GPS_HV_RST renamed GNSS_RESET
- net GPS_HV_RXD renamed GNSS_RXD
- net GPS_HV_SDBY renamed GNSS_SDBY
- net GPS_HV_TXD renamed GNSS_TXD
- net GPS_LV_FO renamed FORCE_ON
- net GPS_LV_RST renamed RESET
- net GPS_LV_RXD renamed RXD
- net GPS_LV_SDBY renamed STANDBY
- net GPS_LV_TXD renamed TXD
Other:
- note added: "Sheets Connection"

Commit message: wip: revision 2
Other:
- note added: "3V3-to-2V8 Level Shifter"
- note added: "GNSS Module"
- note removed: "GNSS"
- moved on the sheet: C48, U13

Commit message: wip: revision 2
Changed lines of the file:
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@@
     (stroke (width 0) (type default))
-  )
-  (polyline (pts (xy 54.61 52.07) (xy 194.31 52.07))
-    (stroke (width 0.5) (type default))
   )
   (wire (pts (xy 262.89 113.03) (xy 262.89 116.84))
@@
     (stroke (width 0) (type default))
   )
-  (polyline (pts (xy 194.31 120.015) (xy 54.61 120.015))
-    (stroke (width 0.5) (type default))
-  )
-  (polyline (pts (xy 269.24 52.07) (xy 269.24 103.505))
-    (stroke (width 0.5) (type default))
-  )
   (polyline (pts (xy 269.24 105.41) (xy 248.285 105.41))
     (stroke (width 0) (type dash))
@@
     (stroke (width 0) (type default))
   )
-  (polyline (pts (xy 194.31 52.07) (xy 194.31 120.015))
-    (stroke (width 0.5) (type default))
-  )
   (wire (pts (xy 218.44 69.85) (xy 222.885 69.85))
     (stroke (width 0) (type default))
@@
   (wire (pts (xy 116.205 64.77) (xy 116.205 77.47))
     (stroke (width 0) (type default))
-  )
-  (polyline (pts (xy 196.215 52.07) (xy 269.24 52.07))
-    (stroke (width 0.5) (type default))
-  )
-  (polyline (pts (xy 54.61 52.07) (xy 54.61 120.015))
-    (stroke (width 0.5) (type default))
   )
   (wire (pts (xy 210.82 82.55) (xy 220.345 82.55))
@@
     (stroke (width 0) (type default))
   )
-  (polyline (pts (xy 269.24 103.505) (xy 196.215 103.505))
-    (stroke (width 0.5) (type default))
-  )
   (wire (pts (xy 141.605 62.23) (xy 151.765 62.23))
     (stroke (width 0) (type default))
@@
     (stroke (width 0) (type default))
   )
-  (polyline (pts (xy 196.215 52.07) (xy 196.215 103.505))
-    (stroke (width 0.5) (type default))
-  )
   (wire (pts (xy 222.25 67.31) (xy 222.25 66.675))
     (stroke (width 0) (type default))
@@
     (stroke (width 0) (type default))
   )
+  (rectangle (start 196.215 52.07) (end 269.24 103.505)
+    (stroke (width 0.5) (type default))
+    (fill (type none))
+  )
+  (rectangle (start 54.61 52.07) (end 194.31 120.015)
+    (stroke (width 0.5) (type default))
+    (fill (type none))
+  )
   (text "GNSS Module" (at 161.925 117.475 0)

Commit message: Added Ignion Antenna
Parts:
- JP1: footprint (none) -> Jumper:SolderJumper-3_P1.3mm_Bridged2Bar12_RoundedPad1.0x1.5mm
Changed lines of the file:
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@@
       (effects (font (size 1.27 1.27)) (justify left))
     )
-    (property "Footprint" "" (at 163.83 77.47 0)
+    (property "Footprint" "Jumper:SolderJumper-3_P1.3mm_Bridged2Bar12_RoundedPad1.0x1.5mm" (at 163.83 77.47 0)
       (effects (font (size 1.27 1.27)) hide)
     )

Commit message: update to KiCAD 8 and add cell power regulator
Parts:
- renumbered C41 to C13, C42 to C14, C48 to C39, C43 to C41, C39 to C42, C44 to C43, D9 to D8, U13 to U11, U11 to U7
