File: hardware/kicad/gnss.kicad_sch (KiCad schematic)
At the start: 10 parts, among them U2 L96-M33

Commit message: update
Connections:
- net GNSS_GEOFENCE: no longer names the net of TP22.1, U2.24 (GEO_FENCE)
- net GNSS_JAMDET: no longer names the net of TP21.1, U2.20 (JAM_DET)
Other:
- moved on the sheet: TP21, TP22
Changed lines of the file:
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@@
-	)
-	(junction
-		(at 147.32 96.52)
-		(diameter 0)
-		(color 0 0 0 0)
 	)
 	(junction
@@
 	)
 	(junction
-		(at 147.32 99.06)
-		(diameter 0)
-		(color 0 0 0 0)
-	)
-	(junction
 		(at 177.8 55.88)
 		(diameter 0)
@@
 	(wire
 		(pts
-			(xy 156.21 101.6) (xy 147.32 101.6)
+			(xy 146.05 99.06) (xy 156.21 99.06)
 		)
 		(stroke
@@
 		)
 	)
-	(wire
-		(pts
-			(xy 147.32 96.52) (xy 146.05 96.52)
-		)
-		(stroke
-			(width 0)
-			(type default)
-		)
-	)
 	(polyline
 		(pts
@@
 	(wire
 		(pts
-			(xy 148.59 96.52) (xy 147.32 96.52)
-		)
-		(stroke
-			(width 0)
-			(type default)
-		)
-	)
-	(wire
-		(pts
-			(xy 147.32 99.06) (xy 148.59 99.06)
+			(xy 146.05 96.52) (xy 156.21 96.52)
 		)
 		(stroke
@@
 		)
 	)
-	(wire
-		(pts
-			(xy 147.32 93.98) (xy 147.32 96.52)
-		)
-		(stroke
-			(width 0)
-			(type default)
-		)
-	)
 	(polyline
 		(pts
@@
 	(wire
 		(pts
-			(xy 156.21 93.98) (xy 147.32 93.98)
-		)
-		(stroke
-			(width 0)
-			(type default)
-		)
-	)
-	(wire
-		(pts
 			(xy 146.05 74.93) (xy 148.59 74.93)
 		)
@@
 	(wire
 		(pts
-			(xy 147.32 101.6) (xy 147.32 99.06)
-		)
-		(stroke
-			(width 0)
-			(type default)
-		)
-	)
-	(wire
-		(pts
 			(xy 177.8 55.88) (xy 182.88 55.88)
-		)
-		(stroke
-			(width 0)
-			(type default)
-		)
-	)
-	(wire
-		(pts
-			(xy 146.05 99.06) (xy 147.32 99.06)
 		)
 		(stroke
@@
 			)
 			(justify right)
-		)
-	)
-	(hierarchical_label "GNSS_JAMDET"
-		(shape output)
-		(at 148.59 96.52 0)
-		(fields_autoplaced yes)
-		(effects
-			(font
-				(size 1.27 1.27)
-			)
-			(justify left)
-		)
-	)
-	(hierarchical_label "GNSS_GEOFENCE"
-		(shape output)
-		(at 148.59 99.06 0)
-		(fields_autoplaced yes)
-		(effects
-			(font
-				(size 1.27 1.27)
-			)
-			(justify left)
 		)
 	)
@@
 	(symbol
 		(lib_id "Connector:TestPoint")
-		(at 156.21 93.98 270)
+		(at 156.21 96.52 270)
 		(unit 1)
 		(exclude_from_sim no)
@@
 		(dnp no)
 		(property "Reference" "TP21"
-			(at 160.655 93.98 90)
+			(at 160.655 96.52 90)
 			(effects
 				(font
@@
 		)
 		(property "Value" "GPIO46"
-			(at 149.225 92.71 90)
+			(at 149.225 95.25 90)
 			(effects
 				(font
@@
 		)
 		(property "Footprint" "TestPoint:TestPoint_Pad_D1.0mm"
-			(at 156.21 99.06 0)
+			(at 156.21 101.6 0)
 			(effects
 				(font
@@
 		)
 		(property "Datasheet" "~"
-			(at 156.21 99.06 0)
+			(at 156.21 101.6 0)
 			(effects
 				(font
@@
 		)
 		(property "Description" ""
-			(at 156.21 93.98 0)
+			(at 156.21 96.52 0)
 			(effects
 				(font
@@
 		)
 		(property "Part Description" ""
-			(at 156.21 93.98 0)
+			(at 156.21 96.52 0)
 			(effects
 				(font
@@
 		)
 		(property "Manufacturer" ""
-			(at 156.21 93.98 0)
+			(at 156.21 96.52 0)
 			(effects
 				(font
@@
 		)
 		(property "Manufacturer Part Number" ""
-			(at 156.21 93.98 0)
+			(at 156.21 96.52 0)
 			(effects
 				(font
@@
 		)
 		(property "Distributor" ""
-			(at 156.21 93.98 0)
+			(at 156.21 96.52 0)
 			(effects
 				(font
@@
 		)
 		(property "Distributor Part Number" ""
-			(at 156.21 93.98 0)
+			(at 156.21 96.52 0)
 			(effects
 				(font
@@
 		)
 		(property "Distributor Link" ""
-			(at 156.21 93.98 0)
+			(at 156.21 96.52 0)
 			(effects
 				(font
@@
 		)
 		(property "Id" ""
-			(at 156.21 93.98 0)
+			(at 156.21 96.52 0)
 			(effects
 				(font
@@
 		)
 		(property "Manufacture" ""
-			(at 156.21 93.98 0)
+			(at 156.21 96.52 0)
 			(effects
 				(font
@@
 		)
 		(property "Manufacture Part Number" ""
-			(at 156.21 93.98 0)
+			(at 156.21 96.52 0)
 			(effects
 				(font
@@
 		)
 		(property "Type" ""
-			(at 156.21 93.98 0)
+			(at 156.21 96.52 0)
 			(effects
 				(font
@@
 	(symbol
 		(lib_id "Connector:TestPoint")
-		(at 156.21 101.6 270)
+		(at 156.21 99.06 270)
 		(unit 1)
 		(exclude_from_sim no)
@@
 		(dnp no)
 		(property "Reference" "TP22"
-			(at 160.655 101.6 90)
+			(at 160.655 99.06 90)
 			(effects
 				(font
@@
 		)
 		(property "Value" "GPIO46"
-			(at 149.225 100.33 90)
+			(at 149.225 97.79 90)
 			(effects
 				(font
@@
 		)
 		(property "Footprint" "TestPoint:TestPoint_Pad_D1.0mm"
-			(at 156.21 106.68 0)
+			(at 156.21 104.14 0)
 			(effects
 				(font
@@
 		)
 		(property "Datasheet" "~"
-			(at 156.21 106.68 0)
+			(at 156.21 104.14 0)
 			(effects
 				(font
@@
 		)
 		(property "Description" ""
-			(at 156.21 101.6 0)
+			(at 156.21 99.06 0)
 			(effects
 				(font
@@
 		)
 		(property "Part Description" ""
-			(at 156.21 101.6 0)
+			(at 156.21 99.06 0)
 			(effects
 				(font
@@
 		)
 		(property "Manufacturer" ""
-			(at 156.21 101.6 0)
+			(at 156.21 99.06 0)
 			(effects
 				(font
@@
 		)
 		(property "Manufacturer Part Number" ""
-			(at 156.21 101.6 0)
+			(at 156.21 99.06 0)
 			(effects
 				(font
@@
 		)
 		(property "Distributor" ""
-			(at 156.21 101.6 0)
+			(at 156.21 99.06 0)
 			(effects
 				(font
@@
 		)
 		(property "Distributor Part Number" ""
-			(at 156.21 101.6 0)
+			(at 156.21 99.06 0)
 			(effects
 				(font
@@
 		)
 		(property "Distributor Link" ""
-			(at 156.21 101.6 0)
+			(at 156.21 99.06 0)
 			(effects
 				(font
@@
 		)
 		(property "Id" ""
-			(at 156.21 101.6 0)
+			(at 156.21 99.06 0)
 			(effects
 				(font
@@
 		)
 		(property "Manufacture" ""
-			(at 156.21 101.6 0)
+			(at 156.21 99.06 0)
 			(effects
 				(font
@@
 		)
 		(property "Manufacture Part Number" ""
-			(at 156.21 101.6 0)
+			(at 156.21 99.06 0)
 			(effects
 				(font
@@
 		)
 		(property "Type" ""
-			(at 156.21 101.6 0)
-			(effects
-				(font
+			(at 156.21 99.06 0)
+			(effects
+				(font

Commit message: Update Production File
Parts:
- D4: Distributor Link https://www.lcsc.com/product-detail/span-style-background-color-ff0-ESD-span-Protection-Devices_Leiditech-ESD5651N_C5173251.html -> https://www.lcsc.com/product-detail/span-style-background-color-ff0-ESD-span-and-Surge-Protection-TVS-span-style-background-color-ff0-ESD-span_TECH-PUBLIC-ESD5651N_C5342369.html; Distributor Part Number C5173251 -> C5342369; Manufacturer Leiditech -> TECH PUBLIC
- renumbered C12 to C14, C13 to C15, C14 to C16, C15 to C17, R12 to R4, TP21 to TP7, TP22 to TP8, U2 to U3
Changed lines of the file:
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@@
 		(on_board yes)
 		(dnp no)
-		(property "Reference" "C14"
+		(property "Reference" "C16"
 			(at 160.02 73.66 0)
 			(effects
@@
 			(project "bwlc1a"
 				(path "/388039b1-99cc-430f-bd4a-010573fde798/6908783c-0fa0-46ec-befb-a4abfbcaa74b"
-					(reference "C14")
+					(reference "C16")
 					(unit 1)
 				)
@@
 		(on_board yes)
 		(dnp no)
-		(property "Reference" "#PWR024"
+		(property "Reference" "#PWR025"
 			(at 167.64 67.31 0)
 			(effects
@@
 			(project "bwlc1a"
 				(path "/388039b1-99cc-430f-bd4a-010573fde798/6908783c-0fa0-46ec-befb-a4abfbcaa74b"
-					(reference "#PWR024")
+					(reference "#PWR025")
 					(unit 1)
 				)
@@
 		(on_board yes)
 		(dnp no)
-		(property "Reference" "R12"
+		(property "Reference" "R4"
 			(at 151.13 76.2 0)
 			(effects
@@
 			(project "bwlc1a"
 				(path "/388039b1-99cc-430f-bd4a-010573fde798/6908783c-0fa0-46ec-befb-a4abfbcaa74b"
-					(reference "R12")
+					(reference "R4")
 					(unit 1)
 				)
@@
 		(on_board yes)
 		(dnp no)
-		(property "Reference" "TP21"
+		(property "Reference" "TP7"
 			(at 160.655 96.52 90)
 			(effects
@@
 			(project "bwlc1a"
 				(path "/388039b1-99cc-430f-bd4a-010573fde798/6908783c-0fa0-46ec-befb-a4abfbcaa74b"
-					(reference "TP21")
+					(reference "TP7")
 					(unit 1)
 				)
@@
 		(on_board yes)
 		(dnp no)
-		(property "Reference" "#PWR029"
+		(property "Reference" "#PWR030"
 			(at 237.49 132.08 0)
 			(effects
@@
 			(project "bwlc1a"
 				(path "/388039b1-99cc-430f-bd4a-010573fde798/6908783c-0fa0-46ec-befb-a4abfbcaa74b"
-					(reference "#PWR029")
+					(reference "#PWR030")
 					(unit 1)
 				)
@@
 		(on_board yes)
 		(dnp no)
-		(property "Reference" "#PWR026"
+		(property "Reference" "#PWR027"
 			(at 157.48 82.55 0)
 			(effects
@@
 			(project "bwlc1a"
 				(path "/388039b1-99cc-430f-bd4a-010573fde798/6908783c-0fa0-46ec-befb-a4abfbcaa74b"
-					(reference "#PWR026")
+					(reference "#PWR027")
 					(unit 1)
 				)
@@
 		(on_board yes)
 		(dnp no)
-		(property "Reference" "#PWR027"
+		(property "Reference" "#PWR028"
 			(at 167.64 82.55 0)
 			(effects
@@
 			(project "bwlc1a"
 				(path "/388039b1-99cc-430f-bd4a-010573fde798/6908783c-0fa0-46ec-befb-a4abfbcaa74b"
-					(reference "#PWR027")
+					(reference "#PWR028")
 					(unit 1)
 				)
@@
 			)
 		)
-		(property "Datasheet" "https://www.lcsc.com/datasheet/lcsc_datasheet_2209151800_Leiditech-ESD5651N_C5173251.pdf"
+		(property "Datasheet" "https://www.lcsc.com/datasheet/lcsc_datasheet_2301051530_TECH-PUBLIC-ESD5651N_C5342369.pdf"
 			(at 177.8 59.69 0)
 			(effects
@@
 			)
 		)
-		(property "Description" "DFN1006 Electrostatic and Surge Protection (TVS/ESD) ROHS"
+		(property "Description" "DFN1006-2L ESD and Surge Protection (TVS/ESD) ROHS "
 			(at 177.8 59.69 0)
 			(effects
@@
 			)
 		)
-		(property "Manufacturer" "Leiditech"
+		(property "Manufacturer" "TECH PUBLIC"
 			(at 177.8 59.69 0)
 			(effects
@@
 			)
 		)
-		(property "Distributor Part Number" "C5173251"
+		(property "Distributor Part Number" "C5342369"
 			(at 177.8 59.69 0)
 			(effects
@@
 			)
 		)
-		(property "Distributor Link" "https://www.lcsc.com/product-detail/span-style-background-color-ff0-ESD-span-Protection-Devices_Leiditech-ESD5651N_C5173251.html"
+		(property "Distributor Link" "https://www.lcsc.com/product-detail/span-style-background-color-ff0-ESD-span-and-Surge-Protection-TVS-span-style-background-color-ff0-ESD-span_TECH-PUBLIC-ESD5651N_C5342369.html"
 			(at 177.8 59.69 0)
 			(effects
@@
 		(on_board yes)
 		(dnp no)
-		(property "Reference" "#PWR025"
+		(property "Reference" "#PWR026"
 			(at 177.8 69.85 0)
 			(effects
@@
 			(project "bwlc1a"
 				(path "/388039b1-99cc-430f-bd4a-010573fde798/6908783c-0fa0-46ec-befb-a4abfbcaa74b"
-					(reference "#PWR025")
+					(reference "#PWR026")
 					(unit 1)
 				)
@@
 		(on_board yes)
 		(dnp no)
-		(property "Reference" "#PWR028"
+		(property "Reference" "#PWR029"
 			(at 146.05 113.03 0)
 			(effects
@@
 			(project "bwlc1a"
 				(path "/388039b1-99cc-430f-bd4a-010573fde798/6908783c-0fa0-46ec-befb-a4abfbcaa74b"
-					(reference "#PWR028")
+					(reference "#PWR029")
 					(unit 1)
 				)
@@
 		(on_board yes)
 		(dnp no)
-		(property "Reference" "C13"
+		(property "Reference" "C15"
 			(at 173.99 58.42 0)
 			(effects
@@
 			(project "bwlc1a"
 				(path "/388039b1-99cc-430f-bd4a-010573fde798/6908783c-0fa0-46ec-befb-a4abfbcaa74b"
-					(reference "C13")
+					(reference "C15")
 					(unit 1)
 				)
@@
 		(on_board yes)
 		(dnp no)
-		(property "Reference" "C12"
+		(property "Reference" "C14"
 			(at 160.02 58.42 0)
 			(effects
@@
 			(project "bwlc1a"
 				(path "/388039b1-99cc-430f-bd4a-010573fde798/6908783c-0fa0-46ec-befb-a4abfbcaa74b"
-					(reference "C12")
+					(reference "C14")
 					(unit 1)
 				)
@@
 		(dnp no)
 		(fields_autoplaced yes)
-		(property "Reference" "U2"
+		(property "Reference" "U3"
 			(at 123.19 60.96 0)
 			(effects
@@
 			(project ""
 				(path "/388039b1-99cc-430f-bd4a-010573fde798/6908783c-0fa0-46ec-befb-a4abfbcaa74b"
-					(reference "U2")
+					(reference "U3")
 					(unit 1)
 				)
@@
 		(on_board yes)
 		(dnp no)
-		(property "Reference" "#PWR023"
+		(property "Reference" "#PWR024"
 			(at 157.48 67.31 0)
 			(effects
@@
 			(project "bwlc1a"
 				(path "/388039b1-99cc-430f-bd4a-010573fde798/6908783c-0fa0-46ec-befb-a4abfbcaa74b"
-					(reference "#PWR023")
+					(reference "#PWR024")
 					(unit 1)
 				)
@@
 		(on_board yes)
 		(dnp no)
-		(property "Reference" "TP22"
+		(property "Reference" "TP8"
 			(at 160.655 99.06 90)
 			(effects
@@
 			(project "bwlc1a"
 				(path "/388039b1-99cc-430f-bd4a-010573fde798/6908783c-0fa0-46ec-befb-a4abfbcaa74b"
-					(reference "TP22")
+					(reference "TP8")
 					(unit 1)
 				)
@@
 		(on_board yes)
 		(dnp no)
-		(property "Reference" "C15"
+		(property "Reference" "C17"
 			(at 170.18 73.66 0)
 			(effects
@@
 			(project ""
 				(path "/388039b1-99cc-430f-bd4a-010573fde798/6908783c-0fa0-46ec-befb-a4abfbcaa74b"
-					(reference "C15")
-					(unit 1)
-				)
+					(reference "C17")
+					(unit 1)
+				)

Commit message: minor aesthetic changes
Parts:
- C17: value 4.7u -> 4u7
Changed lines of the file:
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@@
 			)
 		)
-		(property "Value" "4.7u"
+		(property "Value" "4u7"
 			(at 170.18 76.2 0)
 			(effects
