File: hardware/kicad/battery.kicad_sch (KiCad schematic)
At the start: 1 part, among them J1 JST-2PH

Commit message: wip: revision 2
Parts:
- added Q8: AO3407A, Package_TO_SOT_SMD:SOT-23, symbol Device:Q_PMOS_GSD
- added TP10: +LIPO, TestPoint:TestPoint_Pad_D1.0mm, symbol Connector:TestPoint
Connections:
- net +BATT: now also Q8.2 (S); no longer J1.1 (Pin_1)
- net GND: now also Q8.1 (G)
- new net: J1.1 (Pin_1), Q8.3 (D), TP10.1
Other:
- note added: "Battery Polar Protection"
- note added: "Sheets Connection"
- moved on the sheet: J1

Commit message: wip: revision 2
Other:
- moved on the sheet: J1, Q8, TP10

Commit message: update to KiCAD 8 and add cell power regulator
Parts:
- renumbered J1 to J2

Commit message: update schematics bom
Parts:
- J2: footprint Teapot:JST_PH_S2B-PH-SM4-TB_1x02-1MP_P2.00mm_Horizontal -> bwlc1a:JST_PH_S2B-PH-SM4-TB_1x02-1MP_P2.00mm_Horizontal
Changed lines of the file:
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@@
 			)
 		)
-		(property "Footprint" "Teapot:JST_PH_S2B-PH-SM4-TB_1x02-1MP_P2.00mm_Horizontal"
+		(property "Footprint" "bwlc1a:JST_PH_S2B-PH-SM4-TB_1x02-1MP_P2.00mm_Horizontal"
 			(at 93.345 55.88 0)
 			(effects

Commit message: uppdate bill of materials
Parts:
- J2: value JST-2PH -> S2B-PH-SM4-TB(LF)(SN); Id 24 -> (none); Manufacture JST Sales America Inc. -> (none); Manufacture Part Number S2B-PH-SM4-TB(LF)(SN) -> (none); Manufacturer (none) -> JST; Manufacturer Part Number (none) -> S2B-PH-SM4-TB(LF)(SN); Type SMD -> (none)
Changed lines of the file:
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@@
 			)
 		)
-		(property "Value" "JST-2PH"
+		(property "Value" "S2B-PH-SM4-TB(LF)(SN)"
 			(at 86.995 58.42 0)
 			(effects
@@
 			)
 		)
-		(property "Datasheet" "~"
+		(property "Datasheet" "https://datasheet.lcsc.com/lcsc/2102031704_JST-S2B-PH-SM4-TB-LF-SN_C295747.pdf?_gl=1*1e18khi*_ga*MTY2MjYzODk0OS4xNjk1MzQ0NTg0*_ga_98M84MKSZH*MTcxNDM2Mzg4Ni43NS4xLjE3MTQzNjM5NTAuNjAuMC4w"
 			(at 93.345 55.88 0)
 			(effects
@@
 			)
 		)
-		(property "Id" "24"
-			(at 93.345 55.88 0)
-			(effects
-				(font
-					(size 1.27 1.27)
-				)
-				(hide yes)
-			)
-		)
-		(property "Manufacture" "JST Sales America Inc."
-			(at 93.345 55.88 0)
-			(effects
-				(font
-					(size 1.27 1.27)
-				)
-				(hide yes)
-			)
-		)
-		(property "Manufacture Part Number" "S2B-PH-SM4-TB(LF)(SN)"
-			(at 93.345 55.88 0)
-			(effects
-				(font
-					(size 1.27 1.27)
-				)
-				(hide yes)
-			)
-		)
-		(property "Type" "SMD"
-			(at 93.345 55.88 0)
-			(effects
-				(font
-					(size 1.27 1.27)
-				)
-				(hide yes)
-			)
-		)
-		(property "Part Description" ""
-			(at 93.345 55.88 0)
-			(effects
-				(font
-					(size 1.27 1.27)
-				)
-				(hide yes)
-			)
-		)
-		(property "Manufacturer" ""
-			(at 93.345 55.88 0)
-			(effects
-				(font
-					(size 1.27 1.27)
-				)
-				(hide yes)
-			)
-		)
-		(property "Manufacturer Part Number" ""
+		(property "Manufacturer" "JST"
+			(at 93.345 55.88 0)
+			(effects
+				(font
+					(size 1.27 1.27)
+				)
+				(hide yes)
+			)
+		)
+		(property "Manufacturer Part Number" "S2B-PH-SM4-TB(LF)(SN)"
 			(at 93.345 55.88 0)
 			(effects
@@
 			)
 		)
-		(property "Description" ""
+		(property "Description" "30V 4.3A 48mΩ@10V,4.3A 1.4W 3V@250uA"
 			(at 127 49.53 0)
 			(effects
