File: hardware/kicad/battery.kicad_sch (KiCad schematic)
At the start: 3 parts, among them J2 S2B-PH-SM4-TB(LF)(SN), Q8 AO3407A

Commit message: add page info
Other:
- company: (none) -> Teapot Laboratories
- title: (none) -> Battery
Changed lines of the file:
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@@
 	(paper "A5")
 	(title_block
-		(date "2023-10-29")
-		(rev "2")
+		(title "Battery")
+		(date "2024-05-17")
+		(rev "1")
+		(company "Teapot Laboratories")
 	)
 	(junction

Commit message: Update for PCB Layout
Parts:
- renumbered J2 to J4, Q8 to Q7, TP10 to TP20
Changed lines of the file:
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@@
 		(on_board yes)
 		(dnp no)
-		(property "Reference" "#PWR0105"
+		(property "Reference" "#PWR093"
 			(at 98.425 72.39 0)
 			(effects
@@
 			(project "bwlc1a"
 				(path "/388039b1-99cc-430f-bd4a-010573fde798/fc98a97f-c593-44d5-bbd7-e4921ada3217"
-					(reference "#PWR0105")
+					(reference "#PWR093")
 					(unit 1)
 				)
@@
 		(on_board yes)
 		(dnp no)
-		(property "Reference" "#PWR0104"
+		(property "Reference" "#PWR091"
 			(at 63.5 43.18 0)
 			(effects
@@
 			(project "bwlc1a"
 				(path "/388039b1-99cc-430f-bd4a-010573fde798/fc98a97f-c593-44d5-bbd7-e4921ada3217"
-					(reference "#PWR0104")
+					(reference "#PWR091")
 					(unit 1)
 				)
@@
 		(on_board yes)
 		(dnp no)
-		(property "Reference" "J2"
+		(property "Reference" "J4"
 			(at 90.17 55.88 0)
 			(effects
@@
 			(project "bwlc1a"
 				(path "/388039b1-99cc-430f-bd4a-010573fde798/fc98a97f-c593-44d5-bbd7-e4921ada3217"
-					(reference "J2")
+					(reference "J4")
 					(unit 1)
 				)
@@
 		(on_board yes)
 		(dnp no)
-		(property "Reference" "#PWR0106"
+		(property "Reference" "#PWR092"
 			(at 141.605 46.99 0)
 			(effects
@@
 			(project "bwlc1a"
 				(path "/388039b1-99cc-430f-bd4a-010573fde798/fc98a97f-c593-44d5-bbd7-e4921ada3217"
-					(reference "#PWR0106")
+					(reference "#PWR092")
 					(unit 1)
 				)
@@
 		(on_board yes)
 		(dnp no)
-		(property "Reference" "TP10"
+		(property "Reference" "TP20"
 			(at 100.965 40.64 0)
 			(effects
@@
 			(project "bwlc1a"
 				(path "/388039b1-99cc-430f-bd4a-010573fde798/fc98a97f-c593-44d5-bbd7-e4921ada3217"
-					(reference "TP10")
+					(reference "TP20")
 					(unit 1)
 				)
@@
 		(dnp no)
 		(fields_autoplaced yes)
-		(property "Reference" "Q8"
+		(property "Reference" "Q7"
 			(at 127 39.37 90)
 			(effects
@@
 			(project "bwlc1a"
 				(path "/388039b1-99cc-430f-bd4a-010573fde798/fc98a97f-c593-44d5-bbd7-e4921ada3217"
-					(reference "Q8")
-					(unit 1)
-				)
+					(reference "Q7")
+					(unit 1)
+				)

Commit message: Update Production File
Parts:
- renumbered Q7 to Q3, TP20 to TP33
Changed lines of the file:
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@@
 		(on_board yes)
 		(dnp no)
-		(property "Reference" "#PWR093"
+		(property "Reference" "#PWR095"
 			(at 98.425 72.39 0)
 			(effects
@@
 			(project "bwlc1a"
 				(path "/388039b1-99cc-430f-bd4a-010573fde798/fc98a97f-c593-44d5-bbd7-e4921ada3217"
-					(reference "#PWR093")
+					(reference "#PWR095")
 					(unit 1)
 				)
@@
 		(on_board yes)
 		(dnp no)
-		(property "Reference" "#PWR091"
+		(property "Reference" "#PWR093"
 			(at 63.5 43.18 0)
 			(effects
@@
 			(project "bwlc1a"
 				(path "/388039b1-99cc-430f-bd4a-010573fde798/fc98a97f-c593-44d5-bbd7-e4921ada3217"
-					(reference "#PWR091")
+					(reference "#PWR093")
 					(unit 1)
 				)
@@
 		(on_board yes)
 		(dnp no)
-		(property "Reference" "#PWR092"
+		(property "Reference" "#PWR094"
 			(at 141.605 46.99 0)
 			(effects
@@
 			(project "bwlc1a"
 				(path "/388039b1-99cc-430f-bd4a-010573fde798/fc98a97f-c593-44d5-bbd7-e4921ada3217"
-					(reference "#PWR092")
+					(reference "#PWR094")
 					(unit 1)
 				)
@@
 		(on_board yes)
 		(dnp no)
-		(property "Reference" "TP20"
+		(property "Reference" "TP33"
 			(at 100.965 40.64 0)
 			(effects
@@
 			(project "bwlc1a"
 				(path "/388039b1-99cc-430f-bd4a-010573fde798/fc98a97f-c593-44d5-bbd7-e4921ada3217"
-					(reference "TP20")
+					(reference "TP33")
 					(unit 1)
 				)
@@
 		(dnp no)
 		(fields_autoplaced yes)
-		(property "Reference" "Q7"
+		(property "Reference" "Q3"
 			(at 127 39.37 90)
 			(effects
@@
 			(project "bwlc1a"
 				(path "/388039b1-99cc-430f-bd4a-010573fde798/fc98a97f-c593-44d5-bbd7-e4921ada3217"
-					(reference "Q7")
-					(unit 1)
-				)
+					(reference "Q3")
+					(unit 1)
+				)
