File: hardware/kicad/sensors.kicad_sch (KiCad schematic)
At the start: 9 parts, among them J6 Qwiic, U4 LSM6DSOTR, U5 MAX17048G+

Commit message: move components to use bwlc1a library
Parts:
- J6: footprint Connector_JST:JST_SH_SM04B-SRSS-TB_1x04-1MP_P1.00mm_Horizontal -> bwlc1a:JST_SH_SM04B-SRSS-TB_1x04-1MP_P1.00mm_Horizontal
Changed lines of the file:
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@@
 			)
 		)
-		(property "Footprint" "Connector_JST:JST_SH_SM04B-SRSS-TB_1x04-1MP_P1.00mm_Horizontal"
+		(property "Footprint" "bwlc1a:JST_SH_SM04B-SRSS-TB_1x04-1MP_P1.00mm_Horizontal"
 			(at 179.07 122.555 0)
 			(effects

Commit message: update bill of materials
Parts:
- C10: Id 4 -> (none); Manufacture Samsung Electro-Mechanics -> (none); Manufacture Part Number CL10A226MP8NUNE -> (none); Manufacturer (none) -> Samsung Electro-Mechanics; Manufacturer Part Number (none) -> CL10A226MP8NUNE; Type SMD -> (none)
- C11: Id 1 -> (none); Manufacture Samsung Electro-Mechanics -> (none); Manufacture Part Number CL10A106KP8NNNC -> (none); Manufacturer (none) -> Samsung Electro-Mechanics; Manufacturer Part Number (none) -> CL10A106KP8NNNC; Type SMD -> (none)
- C12, C8, C9: Id 3 -> (none); Manufacture Samsung Electro-Mechanics -> (none); Manufacture Part Number CL05B104KO5NNNC -> (none); Manufacturer (none) -> Samsung Electro-Mechanics; Manufacturer Part Number (none) -> CL05B104KO5NNNC; Type SMD -> (none)
- J6: Distributor (none) -> LCSC; Distributor Link (none) -> https://www.lcsc.com/product-detail/Wire-To-Board-Wire-To-W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; Distributor Part Number (none) -> C160404; Manufacturer JST Sales America -> JST; Manufacturer Part Number (none) -> SM04B-SRSS-TB(LF)(SN); Part Number SM04B-SRSS-TB -> (none)
- R10: Id 40 -> (none); Manufacture UNI-ROYAL(Uniroyal Elec) -> (none); Manufacture Part Number 0402WGF1002TCE -> (none); Manufacturer (none) -> UNI-ROYAL(Uniroyal Elec); Manufacturer Part Number (none) -> 0402WGF1002TCE; Type SMD -> (none)
- U4: Distributor Link https://datasheet.lcsc.com/lcsc/2108070730_STMicroelectroni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 -> https://www.lcsc.com/product-detail/Attitude-Sensor-Gyrosco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; Part Description LGA-14 Attitude Sensor/Gyroscope ROHS -> (none)
- U5: Id 54 -> (none); Manufacture Analog Devices Inc./Maxim Integrated -> (none); Manufacture Part Number MAX17048G+T10 -> (none); Manufacturer (none) -> Analog Devices Inc./Maxim Integrated; Manufacturer Part Number (none) -> MAX17048G+T10; Type SMD -> (none)
Other:
- moved on the sheet: C10, C11, C8, U5

Commit message: update bill of materials
Parts:
- J6: value Qwiic -> SM04B-SRSS-TB(LF)(SN)
Changed lines of the file:
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@@
 			)
 		)
-		(property "Datasheet" "https://datasheet.lcsc.com/lcsc/2206010100_UNI-ROYAL-Uniroyal-Elec-0402WGF1002TCE_C25744.pdf?_gl=1*15oda6t*_ga*MTY2MjYzODk0OS4xNjk1MzQ0NTg0*_ga_98M84MKSZH*MTcxNDQxNTczMy43Ny4xLjE3MTQ0MTY0MTMuMTEuMC4w"
+		(property "Datasheet" "https://www.lcsc.com/datasheet/lcsc_datasheet_2206010100_UNI-ROYAL-Uniroyal-Elec-0402WGF1002TCE_C25744.pdf"
 			(at 86.995 97.79 0)
 			(effects
@@
 			)
 		)
-		(property "Description" "62.5mW Thick Film Resistors ±100ppm/℃ ±1% 10kΩ 0402 Chip Resistor - Surface Mount ROHS"
+		(property "Description" "62.5mW Thick Film Resistors 50V ±100ppm/℃ ±1% 10kΩ 0402 Chip Resistor - Surface Mount ROHS"
 			(at 86.995 97.79 0)
 			(effects
@@
 			)
 		)
-		(property "Value" "Qwiic"
+		(property "Value" "SM04B-SRSS-TB(LF)(SN)"
 			(at 182.245 120.015 0)
 			(effects
@@
 			)
 		)
-		(property "Description" " 1x4P 4P 1 SR Tin 1mm 4 -25℃~+85℃ 1A Copper Alloy Surface Mount，Right Angle SMD,P=1mm,Surface Mount，Right Angle Wire To Board Connector ROHS"
+		(property "Description" "1x4P 4P 1 SR Tin 1mm 4 -25℃~+85℃ 1A Copper Alloy Surface Mount，Right Angle SMD,P=1mm,Surface Mount，Right Angle Wire To Board Connector ROHS"
 			(at 179.07 122.555 0)
 			(effects

Commit message: add page info
Other:
- company: (none) -> Teapot Laboratories
- title: (none) -> Sensors
Changed lines of the file:
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@@
 	(generator_version "8.0")
 	(paper "A4")
+	(title_block
+		(title "Sensors")
+		(date "2024-05-17")
+		(rev "1")
+		(company "Teapot Laboratories")
+	)
 	(junction
 		(at 200.66 74.93)

Commit message: Update for PCB Layout
Parts:
- J5: renamed from J6; footprint bwlc1a:JST_SH_SM04B-SRSS-TB_1x04-1MP_P1.00mm_Horizontal -> Connector_JST:JST_SH_BM04B-SRSS-TB_1x04-1MP_P1.00mm_Vertical
- renumbered C8 to C34, C9 to C35, C10 to C36, C11 to C37, C12 to C38, R10 to R32, U4 to U10, U5 to U9
Connections:
- net +3V3: now also J5.3 (Pin_3); no longer J5.2 (Pin_2)
- net GND: now also J5.4 (Pin_4); no longer J5.1 (Pin_1)
- net SCL: now also J5.1 (Pin_1); no longer J5.4 (Pin_4)
- net SDA: now also J5.2 (Pin_2); no longer J5.3 (Pin_3)
Other:
- moved on the sheet: J5
