File: hardware/kicad/sensors.kicad_sch (KiCad schematic)
At the start: 9 parts, among them J5 SM04B-SRSS-TB(LF)(SN), U10 LSM6DSOTR, U9 MAX17048G+

Commit message: Finish Manufacturing File
Parts:
- J5: footprint Connector_JST:JST_SH_BM04B-SRSS-TB_1x04-1MP_P1.00mm_Vertical -> bwlc1a:JST_SH_SM04B-SRSS-TB_1x04-1MP_P1.00mm_Horizontal
Connections:
- net +3V3: now also J5.2 (Pin_2); no longer J5.3 (Pin_3)
- net GND: now also J5.1 (Pin_1); no longer J5.4 (Pin_4)
- net SCL: now also J5.4 (Pin_4); no longer J5.1 (Pin_1)
- net SDA: now also J5.3 (Pin_3); no longer J5.2 (Pin_2)

Commit message: Update Production File
Parts:
- renumbered C34 to C36, C35 to C37, C36 to C38, C37 to C39, C38 to C40, R32 to R24, U9 to U10, U10 to U11
Changed lines of the file:
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@@
 		(on_board yes)
 		(dnp no)
-		(property "Reference" "#PWR094"
+		(property "Reference" "#PWR096"
 			(at 85.725 66.04 0)
 			(effects
@@
 			(project "bwlc1a"
 				(path "/388039b1-99cc-430f-bd4a-010573fde798/f0ceb3a9-6c16-45f6-8aec-9ac0bb10996d"
-					(reference "#PWR094")
+					(reference "#PWR096")
 					(unit 1)
 				)
@@
 		(dnp no)
 		(fields_autoplaced yes)
-		(property "Reference" "U10"
+		(property "Reference" "U11"
 			(at 110.5409 120.65 0)
 			(effects
@@
 			(project "bwlc1a"
 				(path "/388039b1-99cc-430f-bd4a-010573fde798/f0ceb3a9-6c16-45f6-8aec-9ac0bb10996d"
-					(reference "U10")
+					(reference "U11")
 					(unit 1)
 				)
@@
 		(on_board yes)
 		(dnp no)
-		(property "Reference" "#PWR097"
+		(property "Reference" "#PWR099"
 			(at 151.13 72.39 0)
 			(effects
@@
 			(project "bwlc1a"
 				(path "/388039b1-99cc-430f-bd4a-010573fde798/f0ceb3a9-6c16-45f6-8aec-9ac0bb10996d"
-					(reference "#PWR097")
+					(reference "#PWR099")
 					(unit 1)
 				)
@@
 		(on_board yes)
 		(dnp no)
-		(property "Reference" "#PWR0101"
+		(property "Reference" "#PWR0103"
 			(at 127 79.375 0)
 			(effects
@@
 			(project "bwlc1a"
 				(path "/388039b1-99cc-430f-bd4a-010573fde798/f0ceb3a9-6c16-45f6-8aec-9ac0bb10996d"
-					(reference "#PWR0101")
+					(reference "#PWR0103")
 					(unit 1)
 				)
@@
 		(dnp no)
 		(fields_autoplaced yes)
-		(property "Reference" "R32"
+		(property "Reference" "R24"
 			(at 86.995 92.71 90)
 			(effects
@@
 			(project "bwlc1a"
 				(path "/388039b1-99cc-430f-bd4a-010573fde798/f0ceb3a9-6c16-45f6-8aec-9ac0bb10996d"
-					(reference "R32")
+					(reference "R24")
 					(unit 1)
 				)
@@
 		(dnp no)
 		(fields_autoplaced yes)
-		(property "Reference" "C35"
+		(property "Reference" "C37"
 			(at 108.585 69.2213 0)
 			(effects
@@
 			(project "bwlc1a"
 				(path "/388039b1-99cc-430f-bd4a-010573fde798/f0ceb3a9-6c16-45f6-8aec-9ac0bb10996d"
-					(reference "C35")
+					(reference "C37")
 					(unit 1)
 				)
@@
 		(on_board yes)
 		(dnp no)
-		(property "Reference" "#PWR0103"
+		(property "Reference" "#PWR0105"
 			(at 200.66 92.71 0)
 			(effects
@@
 			(project "bwlc1a"
 				(path "/388039b1-99cc-430f-bd4a-010573fde798/f0ceb3a9-6c16-45f6-8aec-9ac0bb10996d"
-					(reference "#PWR0103")
+					(reference "#PWR0105")
 					(unit 1)
 				)
@@
 		(on_board yes)
 		(dnp no)
-		(property "Reference" "#PWR0100"
+		(property "Reference" "#PWR0102"
 			(at 116.84 79.375 0)
 			(effects
@@
 			(project "bwlc1a"
 				(path "/388039b1-99cc-430f-bd4a-010573fde798/f0ceb3a9-6c16-45f6-8aec-9ac0bb10996d"
-					(reference "#PWR0100")
+					(reference "#PWR0102")
 					(unit 1)
 				)
@@
 		(dnp no)
 		(fields_autoplaced yes)
-		(property "Reference" "C38"
+		(property "Reference" "C40"
 			(at 203.835 79.3813 0)
 			(effects
@@
 			(project "bwlc1a"
 				(path "/388039b1-99cc-430f-bd4a-010573fde798/f0ceb3a9-6c16-45f6-8aec-9ac0bb10996d"
-					(reference "C38")
+					(reference "C40")
 					(unit 1)
 				)
@@
 		(dnp no)
 		(fields_autoplaced yes)
-		(property "Reference" "C34"
+		(property "Reference" "C36"
 			(at 88.9 69.2213 0)
 			(effects
@@
 			(project "bwlc1a"
 				(path "/388039b1-99cc-430f-bd4a-010573fde798/f0ceb3a9-6c16-45f6-8aec-9ac0bb10996d"
-					(reference "C34")
+					(reference "C36")
 					(unit 1)
 				)
@@
 		(on_board yes)
 		(dnp no)
-		(property "Reference" "#PWR098"
+		(property "Reference" "#PWR0100"
 			(at 85.725 79.375 0)
 			(effects
@@
 			(project "bwlc1a"
 				(path "/388039b1-99cc-430f-bd4a-010573fde798/f0ceb3a9-6c16-45f6-8aec-9ac0bb10996d"
-					(reference "#PWR098")
+					(reference "#PWR0100")
 					(unit 1)
 				)
@@
 		(dnp no)
 		(fields_autoplaced yes)
-		(property "Reference" "C37"
+		(property "Reference" "C39"
 			(at 130.175 69.2213 0)
 			(effects
@@
 			(project "bwlc1a"
 				(path "/388039b1-99cc-430f-bd4a-010573fde798/f0ceb3a9-6c16-45f6-8aec-9ac0bb10996d"
-					(reference "C37")
+					(reference "C39")
 					(unit 1)
 				)
@@
 		(on_board yes)
 		(dnp no)
-		(property "Reference" "#PWR0102"
+		(property "Reference" "#PWR0104"
 			(at 195.58 92.71 0)
 			(effects
@@
 			(project "bwlc1a"
 				(path "/388039b1-99cc-430f-bd4a-010573fde798/f0ceb3a9-6c16-45f6-8aec-9ac0bb10996d"
-					(reference "#PWR0102")
+					(reference "#PWR0104")
 					(unit 1)
 				)
@@
 		(on_board yes)
 		(dnp no)
-		(property "Reference" "#PWR095"
+		(property "Reference" "#PWR097"
 			(at 116.84 66.04 0)
 			(effects
@@
 			(project "bwlc1a"
 				(path "/388039b1-99cc-430f-bd4a-010573fde798/f0ceb3a9-6c16-45f6-8aec-9ac0bb10996d"
-					(reference "#PWR095")
+					(reference "#PWR097")
 					(unit 1)
 				)
@@
 		(dnp no)
 		(fields_autoplaced yes)
-		(property "Reference" "C36"
+		(property "Reference" "C38"
 			(at 120.015 69.2213 0)
 			(effects
@@
 			(project "bwlc1a"
 				(path "/388039b1-99cc-430f-bd4a-010573fde798/f0ceb3a9-6c16-45f6-8aec-9ac0bb10996d"
-					(reference "C36")
+					(reference "C38")
 					(unit 1)
 				)
@@
 		(dnp no)
 		(fields_autoplaced yes)
-		(property "Reference" "#PWR096"
+		(property "Reference" "#PWR098"
 			(at 200.66 68.58 0)
 			(effects
@@
 			(project "bwlc1a"
 				(path "/388039b1-99cc-430f-bd4a-010573fde798/f0ceb3a9-6c16-45f6-8aec-9ac0bb10996d"
-					(reference "#PWR096")
+					(reference "#PWR098")
 					(unit 1)
 				)
@@
 		(on_board yes)
 		(dnp no)
-		(property "Reference" "#PWR099"
+		(property "Reference" "#PWR0101"
 			(at 105.41 79.375 0)
 			(effects
@@
 			(project "bwlc1a"
 				(path "/388039b1-99cc-430f-bd4a-010573fde798/f0ceb3a9-6c16-45f6-8aec-9ac0bb10996d"
-					(reference "#PWR099")
+					(reference "#PWR0101")
 					(unit 1)
 				)
@@
 		(on_board yes)
 		(dnp no)
-		(property "Reference" "#PWR0106"
+		(property "Reference" "#PWR0108"
 			(at 108.585 127 0)
 			(effects
@@
 			(project "bwlc1a"
 				(path "/388039b1-99cc-430f-bd4a-010573fde798/f0ceb3a9-6c16-45f6-8aec-9ac0bb10996d"
-					(reference "#PWR0106")
+					(reference "#PWR0108")
 					(unit 1)
 				)
@@
 		(on_board yes)
 		(dnp no)
-		(property "Reference" "#PWR0104"
+		(property "Reference" "#PWR0106"
 			(at 78.105 110.49 0)
 			(effects
@@
 			(project "bwlc1a"
 				(path "/388039b1-99cc-430f-bd4a-010573fde798/f0ceb3a9-6c16-45f6-8aec-9ac0bb10996d"
-					(reference "#PWR0104")
+					(reference "#PWR0106")
 					(unit 1)
 				)
@@
 		(dnp no)
 		(fields_autoplaced yes)
-		(property "Reference" "U9"
+		(property "Reference" "U10"
 			(at 175.26 63.5 0)
 			(effects
@@
 			(project "bwlc1a"
 				(path "/388039b1-99cc-430f-bd4a-010573fde798/f0ceb3a9-6c16-45f6-8aec-9ac0bb10996d"
-					(reference "U9")
+					(reference "U10")
 					(unit 1)
 				)
@@
 		(dnp no)
 		(fields_autoplaced yes)
-		(property "Reference" "#PWR0107"
+		(property "Reference" "#PWR0109"
 			(at 163.83 133.35 0)
 			(effects
@@
 			(project "bwlc1a"
 				(path "/388039b1-99cc-430f-bd4a-010573fde798/f0ceb3a9-6c16-45f6-8aec-9ac0bb10996d"
-					(reference "#PWR0107")
+					(reference "#PWR0109")
 					(unit 1)
 				)
@@
 		(on_board yes)
 		(dnp no)
-		(property "Reference" "#PWR0105"
+		(property "Reference" "#PWR0107"
 			(at 163.83 123.19 0)
 			(effects
@@
 			(project "bwlc1a"
 				(path "/388039b1-99cc-430f-bd4a-010573fde798/f0ceb3a9-6c16-45f6-8aec-9ac0bb10996d"
-					(reference "#PWR0105")
-					(unit 1)
-				)
+					(reference "#PWR0107")
+					(unit 1)
+				)
